Commit message: feat: add gazebo sim bringup with obstacle world
- add big_bertha_sim_bringup package (worlds, launch, config, rviz, test)
- obstacle_world.sdf: 10x10 m walled arena, boxes + pillars blocking A->B
- simulation.launch.py: headless-capable gz server, robot spawn, ros_gz_bridge, ros2_control spawners
- ros_gz_bridge.yaml bridges /clock /scan /imu /odom /tf
- add gz OdometryPublisher to description gazebo xacro behind publish_odom arg
- thread publish_odom through urdf xacro and rsp launch
- verify_simulation.sh headless gate: rates on /scan /imu /odom /clock, finite ranges, no NaN

File: big_bertha_description/urdf/big_bertha.gazebo.xacro (robot description, xacro)
@@ -11,4 +11,22 @@
 -->
 <robot xmlns:xacro="http://www.ros.org/wiki/xacro">
+  <!-- Emit a gz OdometryPublisher for base_link -> /odom + odom->base_link
+       tf. Enabled in simulation; the real robot fuses wheel/leg odom in the
+       EKF instead, so this stays behind an arg. -->
+  <xacro:arg name="publish_odom" default="true"/>
+  <xacro:property name="publish_odom" value="$(arg publish_odom)"/>
+  <xacro:if value="${publish_odom}">
+    <gazebo>
+      <plugin filename="gz-sim-odometry-publisher-system"
+              name="gz::sim::systems::OdometryPublisher">
+        <odom_frame>odom</odom_frame>
+        <robot_base_frame>base_link</robot_base_frame>
+        <odom_topic>odom</odom_topic>
+        <tf_topic>/tf</tf_topic>
+        <dimensions>3</dimensions>
+        <odom_publish_frequency>50</odom_publish_frequency>
+      </plugin>
+    </gazebo>
+  </xacro:if>
   <!-- ===================== Friction / materials ====================== -->
   <xacro:macro name="bb_surface" params="link color:=Gazebo/Silver mu:=1.0">

File: big_bertha_description/urdf/big_bertha.urdf.xacro (robot description, xacro)
@@ -21,4 +21,6 @@
   <xacro:arg name="ros2_control_config"
              default="$(find big_bertha_description)/config/ros2_control.yaml"/>
+  <!-- Forwarded to the gz OdometryPublisher in big_bertha.gazebo.xacro. -->
+  <xacro:arg name="publish_odom" default="true"/>
   <xacro:property name="use_gz" value="$(arg use_gz)"/>
   <!-- ============================ Materials ============================ -->

Commit message: feat: add robot_localization ekf state estimation
- add config/ekf.yaml fusing /odom (planar vel) + /imu (yaw, yaw rate)
- ekf publishes continuous odom->base_link tf and /odometry/filtered at 50 Hz
- add launch/state_estimation/ekf.launch.py
- add odom_tf xacro arg so the EKF owns odom->base_link (gz tf routed away)
- thread odom_tf through urdf xacro, rsp launch, and simulation launch
- verify_state_estimation.sh gate: tf continuous, covariance bounded, no NaN

File: big_bertha_description/urdf/big_bertha.gazebo.xacro (robot description, xacro)
@@ -13,7 +13,14 @@
   <!-- Emit a gz OdometryPublisher for base_link -> /odom + odom->base_link
        tf. Enabled in simulation; the real robot fuses wheel/leg odom in the
-       EKF instead, so this stays behind an arg. -->
+       EKF instead, so this stays behind an arg.
+       odom_tf controls whether this plugin also publishes the
+       odom->base_link transform. When the robot_localization EKF is running
+       it owns that transform, so the state_estimation bringup sets
+       odom_tf:=false and the plugin's tf is routed to an unused topic
+       (keeping /odom as the EKF input). -->
   <xacro:arg name="publish_odom" default="true"/>
+  <xacro:arg name="odom_tf" default="true"/>
   <xacro:property name="publish_odom" value="$(arg publish_odom)"/>
+  <xacro:property name="odom_tf" value="$(arg odom_tf)"/>
   <xacro:if value="${publish_odom}">
     <gazebo>
@@ -23,5 +30,10 @@
         <robot_base_frame>base_link</robot_base_frame>
         <odom_topic>odom</odom_topic>
-        <tf_topic>/tf</tf_topic>
+        <xacro:if value="${odom_tf}">
+          <tf_topic>/tf</tf_topic>
+        </xacro:if>
+        <xacro:unless value="${odom_tf}">
+          <tf_topic>/odom_tf_unused</tf_topic>
+        </xacro:unless>
         <dimensions>3</dimensions>
         <odom_publish_frequency>50</odom_publish_frequency>

File: big_bertha_description/urdf/big_bertha.urdf.xacro (robot description, xacro)
@@ -23,4 +23,6 @@
   <!-- Forwarded to the gz OdometryPublisher in big_bertha.gazebo.xacro. -->
   <xacro:arg name="publish_odom" default="true"/>
+  <!-- When false, the EKF (state_estimation) owns the odom->base_link tf. -->
+  <xacro:arg name="odom_tf" default="true"/>
   <xacro:property name="use_gz" value="$(arg use_gz)"/>
   <!-- ============================ Materials ============================ -->

Commit message: feat: add slam_toolbox mapping and saved grid
- add config/slam_toolbox.yaml (online async, base_link/odom/scan tuned)
- add launch/mapping/slam.launch.py with nav2_lifecycle_manager autostart
- add sim-only gz VelocityControl kinematic drive (sim_drive arg) + ROS->gz cmd_vel bridge for scripted verification drives
- add test/scripted_drive.sh patrol and test/verify_mapping.sh gate
- save maps/obstacle_world.{yaml,pgm} from a scripted drive (committed directly)
- fix verify scripts: source ROS before set -u
- thread sim_drive through urdf xacro, rsp launch, simulation launch

File: big_bertha_description/urdf/big_bertha.gazebo.xacro (robot description, xacro)
@@ -38,4 +38,21 @@
         <dimensions>3</dimensions>
         <odom_publish_frequency>50</odom_publish_frequency>
+      </plugin>
+    </gazebo>
+  </xacro:if>
+  <!-- Sim-only kinematic drive. When sim_drive:=true a gz VelocityControl
+       system moves base_link directly from a Twist on the gz "cmd_vel"
+       topic, decoupled from the legs. This is a verification aid for the
+       mapping / localization / planning gates: it lets a scripted /cmd_vel
+       drive build a map and run A->B navigation independently of the gait
+       policy (which does not transfer to Gazebo, see issue #5). The real
+       robot and the locomotion demo do not use it (sim_drive defaults off). -->
+  <xacro:arg name="sim_drive" default="false"/>
+  <xacro:property name="sim_drive" value="$(arg sim_drive)"/>
+  <xacro:if value="${sim_drive}">
+    <gazebo>
+      <plugin filename="gz-sim-velocity-control-system"
+              name="gz::sim::systems::VelocityControl">
+        <topic>cmd_vel</topic>
       </plugin>
     </gazebo>

File: big_bertha_description/urdf/big_bertha.urdf.xacro (robot description, xacro)
@@ -25,4 +25,6 @@
   <!-- When false, the EKF (state_estimation) owns the odom->base_link tf. -->
   <xacro:arg name="odom_tf" default="true"/>
+  <!-- Sim-only kinematic drive (gz VelocityControl) for verification gates. -->
+  <xacro:arg name="sim_drive" default="false"/>
   <xacro:property name="use_gz" value="$(arg use_gz)"/>
   <!-- ============================ Materials ============================ -->

Commit message: fix: drive policy controller with effort-pd actuator

File: big_bertha_description/urdf/big_bertha.gazebo.xacro (robot description, xacro)
@@ -64,5 +64,8 @@
       <mu1>${mu}</mu1>
       <mu2>${mu}</mu2>
-      <self_collide>true</self_collide>
+      <!-- Self-collision off: the upper-leg links still use STL-mesh collision,
+           and mesh-mesh self contact injects noisy forces (only the feet are
+           clean spheres). Legs do not overlap in a normal gait. -->
+      <self_collide>false</self_collide>
     </gazebo>
   </xacro:macro>
@@ -72,14 +75,14 @@
   <xacro:bb_surface link="arm_a_1_1"  mu="0.6"/>
   <xacro:bb_surface link="arm_b_1_1"  mu="0.6"/>
-  <xacro:bb_surface link="arm_c_1_1"  mu="1.0"/>
+  <xacro:bb_surface link="arm_c_1_1"  mu="1.5"/>
   <xacro:bb_surface link="arm_a_2_1"  mu="0.6"/>
   <xacro:bb_surface link="arm_b_2_1"  mu="0.6"/>
-  <xacro:bb_surface link="arm_c_2_1"  mu="1.0"/>
+  <xacro:bb_surface link="arm_c_2_1"  mu="1.5"/>
   <xacro:bb_surface link="arm_a_3_1"  mu="0.6"/>
   <xacro:bb_surface link="arm_b_3_1"  mu="0.6"/>
-  <xacro:bb_surface link="arm_c_3_1"  mu="1.0"/>
+  <xacro:bb_surface link="arm_c_3_1"  mu="1.5"/>
   <xacro:bb_surface link="arm_a_4_1"  mu="0.6"/>
   <xacro:bb_surface link="arm_b_4_1"  mu="0.6"/>
-  <xacro:bb_surface link="arm_c_4_1"  mu="1.0"/>
+  <xacro:bb_surface link="arm_c_4_1"  mu="1.5"/>
   <!-- ============================ Lidar ============================== -->
   <!-- YDLidar X2: 360 deg, ~8 m range, 5 Hz. Published on gz topic "scan",
@@ -109,5 +112,10 @@
         </scan>
         <range>
-          <min>0.12</min>
+          <!-- 0.35 m, not 0.12: the body lidar otherwise hits Big Bertha's own
+               legs (~0.14-0.30 m away, ~80 of 360 rays), which marked the
+               robot's own cell as a near-lethal obstacle (cost 99) so Nav2
+               could not plan from its start pose, and fed self-returns into
+               slam. Real obstacles are well beyond 0.35 m. -->
+          <min>0.35</min>
           <max>8.0</max>
           <resolution>0.01</resolution>

File: big_bertha_description/urdf/big_bertha.ros2_control.xacro (robot description, xacro)
@@ -2,9 +2,10 @@
 <!--
   ros2_control hardware description for Big Bertha under gz_ros2_control.
-  All 12 leg joints (Revolute_110 .. Revolute_121) are exposed with a
-  position command interface and position/velocity state interfaces, so the
-  policy controller can stream targets on /position_controller/commands and
-  read /joint_states. The <param>initial_value</param> reproduces the
-  training default pose ([0.0, 0.5, 0.0] per leg).
+  All 12 leg joints (Revolute_110 .. Revolute_121) are exposed with an
+  effort command interface and position/velocity/effort state interfaces, so
+  the policy controller can stream joint torques on
+  /position_controller/commands and read /joint_states. The
+  <param>initial_value</param> reproduces the training default pose
+  ([0.0, 0.5, 0.0] per leg).
 -->
 <robot xmlns:xacro="http://www.ros.org/wiki/xacro">
@@ -12,7 +13,7 @@
   <xacro:macro name="bb_joint" params="name init:=0.0">
     <joint name="${name}">
-      <command_interface name="position">
-        <param name="min">-3.14159</param>
-        <param name="max">3.14159</param>
+      <command_interface name="effort">
+        <param name="min">-12.0</param>
+        <param name="max">12.0</param>
       </command_interface>
       <state_interface name="position">
@@ -45,5 +46,8 @@
   </ros2_control>
   <!-- gz_ros2_control system plugin: loads controller_manager inside gz,
-       parameterised by config/ros2_control.yaml. -->
+       parameterised by config/ros2_control.yaml. The leg joints use an EFFORT
+       command interface (the policy node streams torque tau = kp*(q_des-q) +
+       kd*(0-qd)), which gz_ros2_control applies directly as joint torque, so
+       no position_proportional_gain servo is involved. -->
   <gazebo>
     <plugin filename="gz_ros2_control-system"

File: big_bertha_description/urdf/big_bertha.urdf.xacro (robot description, xacro)
@@ -62,6 +62,8 @@
       <origin xyz="0.0045 0 0.035" rpy="0 0 0"/>
       <mass value="0.126"/>
-      <inertia ixx="1.35942189e-08" iyy="3.17136623e-08" izz="3.50224283e-08"
-               ixy="-4.05791206e-11" ixz="4.26994723e-09" iyz="8.44411878e-11"/>
+      <!-- Plausible solid-puck inertia; the CAD export gave ~1e-8 (degenerate),
+           which DART uses verbatim (PhysX silently regularizes it) and turns
+           the mass matrix near-singular -> solver jitter. -->
+      <inertia ixx="1.2e-04" iyy="1.2e-04" izz="1.0e-04" ixy="0.0" ixz="0.0" iyz="0.0"/>
     </inertial>
     <visual>
@@ -77,6 +79,6 @@
       <origin xyz="0.04 -0.01 0.02" rpy="0 0 0"/>
       <mass value="0.2244"/>
-      <inertia ixx="0.00000006" iyy="0.00000008" izz="0.00000010"
-               ixy="-0.00000000" ixz="0.00000000" iyz="-0.00000000"/>
+      <!-- Plausible battery-pack inertia; CAD export gave ~6e-8 (degenerate). -->
+      <inertia ixx="1.5e-04" iyy="1.5e-04" izz="1.5e-04" ixy="0.0" ixz="0.0" iyz="0.0"/>
     </inertial>
     <visual>
@@ -93,5 +95,5 @@
       <origin xyz="0 0 0" rpy="0 0 0"/>
       <mass value="0.001"/>
-      <inertia ixx="1e-09" iyy="1e-09" izz="1e-09" ixy="0" ixz="0" iyz="0"/>
+      <inertia ixx="1e-06" iyy="1e-06" izz="1e-06" ixy="0" ixz="0" iyz="0"/>
     </inertial>
     <visual>
@@ -107,5 +109,8 @@
       <origin xyz="-0.029329716066216552 -0.02813594305937389 -0.02511915559887622" rpy="0 0 0"/>
       <mass value="0.12"/>
-      <inertia ixx="0.00014066085674721668" iyy="0.0001330984450941405" izz="9.579054760563143e-05" ixy="-1.512482330615233e-05" iyz="-5.041607768717444e-07" ixz="5.041607768717444e-06"/>
+      <!-- Symmetrized to match arm_a_1/2/3 (identical leg part); the CAD export
+           gave this one leg ~2.3x the inertia, which an explicit PD turns into
+           a curved walk (Isaac's implicit PD hides the asymmetry). -->
+      <inertia ixx="5.834254143646408e-05" iyy="6.165745856353591e-05" izz="4.198895027624309e-05" ixy="6.629834254143645e-06" iyz="2.2099447513812153e-06" ixz="2.209944751381215e-07"/>
     </inertial>
     <visual>
@@ -156,8 +161,8 @@
       <material name="silver"/>
     </visual>
-    <collision>
-      <origin xyz="0.124465 0.14848 -0.082982" rpy="0 0 0"/>
-      <geometry>
-        <mesh filename="${mesh_pkg}/arm_c_4_1.stl" scale="0.001 0.001 0.001"/>
+    <collision name="arm_c_4_1_foot">
+      <origin xyz="-0.0691 -0.0439 -0.1215" rpy="0 0 0"/>
+      <geometry>
+        <sphere radius="0.012"/>
       </geometry>
     </collision>
@@ -216,8 +221,13 @@
       <material name="silver"/>
     </visual>
-    <collision>
-      <origin xyz="-0.16378 0.109165 -0.082982" rpy="0 0 0"/>
-      <geometry>
-        <mesh filename="${mesh_pkg}/arm_c_1_1.stl" scale="0.001 0.001 0.001"/>
+    <!-- Foot contact: a sphere at the toe tip, not the STL mesh. DART does
+         literal mesh-plane contact (points jump between triangles -> noisy,
+         non-deterministic footing -> the gait wanders); a sphere gives one
+         clean, stable contact point. PhysX convex-decomposes so Isaac is fine
+         with the mesh. Visual keeps the mesh. -->
+    <collision name="arm_c_1_1_foot">
+      <origin xyz="0.0439 -0.0691 -0.1215" rpy="0 0 0"/>
+      <geometry>
+        <sphere radius="0.012"/>
       </geometry>
     </collision>
@@ -276,8 +286,8 @@
       <material name="silver"/>
     </visual>
-    <collision>
-      <origin xyz="-0.124465 -0.14848 -0.082982" rpy="0 0 0"/>
-      <geometry>
-        <mesh filename="${mesh_pkg}/arm_c_2_1.stl" scale="0.001 0.001 0.001"/>
+    <collision name="arm_c_2_1_foot">
+      <origin xyz="0.0691 0.0439 -0.1215" rpy="0 0 0"/>
+      <geometry>
+        <sphere radius="0.012"/>
       </geometry>
     </collision>
@@ -336,8 +346,8 @@
       <material name="silver"/>
     </visual>
-    <collision>
-      <origin xyz="0.16378 -0.109165 -0.082982" rpy="0 0 0"/>
-      <geometry>
-        <mesh filename="${mesh_pkg}/arm_c_3_1.stl" scale="0.001 0.001 0.001"/>
+    <collision name="arm_c_3_1_foot">
+      <origin xyz="-0.0439 0.0691 -0.1215" rpy="0 0 0"/>
+      <geometry>
+        <sphere radius="0.012"/>
       </geometry>
     </collision>
@@ -350,5 +360,5 @@
     <child link="arm_a_4_1"/>
     <axis xyz="0.0 -0.0 1.0"/>
-    <dynamics damping="0.1" friction="0.0"/>
+    <dynamics damping="0.02" friction="0.0"/>
   </joint>
   <joint name="Revolute_111" type="continuous">
@@ -357,5 +367,5 @@
     <child link="arm_b_4_1"/>
     <axis xyz="0.707107 -0.707107 0.0"/>
-    <dynamics damping="0.1" friction="0.0"/>
+    <dynamics damping="0.02" friction="0.0"/>
   </joint>
   <joint name="Revolute_112" type="continuous">
@@ -364,5 +374,5 @@
     <child link="arm_c_4_1"/>
     <axis xyz="-0.707107 0.707107 -0.0"/>
-    <dynamics damping="0.1" friction="0.0"/>
+    <dynamics damping="0.02" friction="0.0"/>
   </joint>
   <!-- Leg 1 (front-left): Revolute_113/114/115 -->
@@ -372,5 +382,5 @@
     <child link="arm_a_1_1"/>
     <axis xyz="0.0 -0.0 1.0"/>
-    <dynamics damping="0.1" friction="0.0"/>
+    <dynamics damping="0.02" friction="0.0"/>
   </joint>
   <joint name="Revolute_114" type="continuous">
@@ -379,5 +389,5 @@
     <child link="arm_b_1_1"/>
     <axis xyz="0.707107 0.707107 0.0"/>
-    <dynamics damping="0.1" friction="0.0"/>
+    <dynamics damping="0.02" friction="0.0"/>
   </joint>
   <joint name="Revolute_115" type="continuous">
@@ -386,5 +396,5 @@
     <child link="arm_c_1_1"/>
     <axis xyz="-0.707107 -0.707107 -0.0"/>
-    <dynamics damping="0.1" friction="0.0"/>
+    <dynamics damping="0.02" friction="0.0"/>
   </joint>
   <!-- Leg 2 (front-right): Revolute_116/117/118 -->
@@ -394,5 +404,5 @@
     <child link="arm_a_2_1"/>
     <axis xyz="-0.0 0.0 1.0"/>
-    <dynamics damping="0.1" friction="0.0"/>
+    <dynamics damping="0.02" friction="0.0"/>
   </joint>
   <joint name="Revolute_117" type="continuous">
@@ -401,5 +411,5 @@
     <child link="arm_b_2_1"/>
     <axis xyz="-0.707107 0.707107 -0.0"/>
-    <dynamics damping="0.1" friction="0.0"/>
+    <dynamics damping="0.02" friction="0.0"/>
   </joint>
   <joint name="Revolute_118" type="continuous">
@@ -408,5 +418,5 @@
     <child link="arm_c_2_1"/>
     <axis xyz="0.707107 -0.707107 -0.0"/>
-    <dynamics damping="0.1" friction="0.0"/>
+    <dynamics damping="0.02" friction="0.0"/>
   </joint>
   <!-- Leg 3 (back-right): Revolute_119/120/121 -->
@@ -416,5 +426,5 @@
     <child link="arm_a_3_1"/>
     <axis xyz="-0.0 0.0 1.0"/>
-    <dynamics damping="0.1" friction="0.0"/>
+    <dynamics damping="0.02" friction="0.0"/>
   </joint>
   <joint name="Revolute_120" type="continuous">
@@ -423,5 +433,5 @@
     <child link="arm_b_3_1"/>
     <axis xyz="-0.707107 -0.707107 0.0"/>
-    <dynamics damping="0.1" friction="0.0"/>
+    <dynamics damping="0.02" friction="0.0"/>
   </joint>
   <joint name="Revolute_121" type="continuous">
@@ -430,5 +440,5 @@
     <child link="arm_c_3_1"/>
     <axis xyz="0.707107 0.707107 -0.0"/>
-    <dynamics damping="0.1" friction="0.0"/>
+    <dynamics damping="0.02" friction="0.0"/>
   </joint>
   <!-- Fixed sensor / payload frames -->
