Commit message: feat: mshes updated for big_berth_description

File: big_bertha_description/urdf/big_bertha.gazebo.xacro (robot description, xacro)
@@ -3,5 +3,5 @@
   Gazebo Harmonic (gz-sim 8) sensor + surface configuration for Big Bertha.
   Provides:
-    - a 2D lidar (YDLidar X2 class) on lidar_link  -> gz topic "scan"
+    - a 2D lidar (YDLidar X2 class) on ydlidar_link  -> gz topic "scan"
     - an IMU (MPU9250 class) on imu_link           -> gz topic "imu"
     - per-link friction/material surface properties.
@@ -85,12 +85,16 @@
   <xacro:bb_surface link="arm_b_4_1"  mu="0.6"/>
   <xacro:bb_surface link="arm_c_4_1"  mu="1.5"/>
+  <xacro:bb_surface link="battery_link"          mu="0.6"/>
+  <xacro:bb_surface link="circuit_box_base_link" mu="0.6"/>
+  <xacro:bb_surface link="circuit_box_link"      mu="0.6"/>
+  <xacro:bb_surface link="ydlidar_link"          mu="0.6"/>
   <!-- ============================ Lidar ============================== -->
   <!-- YDLidar X2: 360 deg, ~8 m range, 5 Hz. Published on gz topic "scan",
-       frame_id = lidar_link. -->
-  <gazebo reference="lidar_link">
+       frame_id = ydlidar_link. -->
+  <gazebo reference="ydlidar_link">
     <material>Gazebo/DarkGrey</material>
     <sensor name="lidar" type="gpu_lidar">
       <topic>scan</topic>
-      <gz_frame_id>lidar_link</gz_frame_id>
+      <gz_frame_id>ydlidar_link</gz_frame_id>
       <update_rate>10</update_rate>
       <always_on>true</always_on>

File: big_bertha_description/urdf/big_bertha.urdf.xacro (robot description, xacro)
@@ -1,32 +1,11 @@
 <?xml version="1.0" ?>
-<!--
-  Big Bertha quadruped description (ROS 2 Jazzy + Gazebo Harmonic).
-  Links and joints are copied from the source CAD export
-  (assets/URDF/big_bertha/Spyder_mg995_description.urdf) and augmented with:
-    - a gz_ros2_control system plugin,
-    - a 12-joint position ros2_control block,
-    - a gz 2D lidar sensor on lidar_link (YDLidar X2),
-    - a gz IMU sensor on imu_link (MPU9250),
-    - gz friction/material surface properties.
-  Joints Revolute_110 .. Revolute_121 (4 legs x 3 joints) are position
-  controlled by gz_ros2_control. Default per-leg pose is [0.0, 0.5, 0.0]
-  i.e. the middle joint of each leg (111/114/117/120) defaults to 0.5 rad.
--->
 <robot name="big_bertha" xmlns:xacro="http://www.ros.org/wiki/xacro">
-  <!-- ============================ Arguments ============================ -->
-  <!-- Use ros2_control + gz sensors when running in Gazebo; disable for a
-       pure visualisation / check_urdf pass. -->
   <xacro:arg name="use_gz" default="true"/>
-  <!-- ros2_control.yaml passed to the gz_ros2_control plugin. -->
   <xacro:arg name="ros2_control_config"
              default="$(find big_bertha_description)/config/ros2_control.yaml"/>
-  <!-- Forwarded to the gz OdometryPublisher in big_bertha.gazebo.xacro. -->
   <xacro:arg name="publish_odom" default="true"/>
-  <!-- When false, the EKF (state_estimation) owns the odom->base_link tf. -->
   <xacro:arg name="odom_tf" default="true"/>
-  <!-- Sim-only kinematic drive (gz VelocityControl) for verification gates. -->
   <xacro:arg name="sim_drive" default="false"/>
   <xacro:property name="use_gz" value="$(arg use_gz)"/>
-  <!-- ============================ Materials ============================ -->
   <material name="silver">
     <color rgba="0.700 0.700 0.700 1.000"/>
@@ -35,60 +14,175 @@
     <color rgba="0.200 0.200 0.200 1.000"/>
   </material>
-  <!-- ======================= Convenience macros ======================= -->
   <xacro:property name="mesh_pkg" value="package://big_bertha_description/meshes"/>
   <!-- ============================== Links ============================== -->
   <link name="base_link">
     <inertial>
-      <origin xyz="4.0195046385725887e-10 -9.5697371012907e-08 -0.005922558162110875" rpy="0 0 0"/>
-      <mass value="0.35"/>
-      <inertia ixx="0.0008859783497446459" iyy="0.001397362239817623" izz="0.0021187809645138865" ixy="-0.0" iyz="-0.0" ixz="-0.0"/>
-    </inertial>
-    <visual>
-      <origin xyz="0 0 0" rpy="0 0 0"/>
-      <geometry>
-        <mesh filename="${mesh_pkg}/base_link.stl" scale="0.001 0.001 0.001"/>
-      </geometry>
-      <material name="silver"/>
-    </visual>
-    <collision>
-      <origin xyz="0 0 0" rpy="0 0 0"/>
-      <geometry>
-        <mesh filename="${mesh_pkg}/base_link.stl" scale="0.001 0.001 0.001"/>
-      </geometry>
-    </collision>
-  </link>
-  <link name="lidar_link">
-    <inertial>
-      <origin xyz="0.0045 0 0.035" rpy="0 0 0"/>
-      <mass value="0.126"/>
-      <!-- Plausible solid-puck inertia; the CAD export gave ~1e-8 (degenerate),
-           which DART uses verbatim (PhysX silently regularizes it) and turns
-           the mass matrix near-singular -> solver jitter. -->
-      <inertia ixx="1.2e-04" iyy="1.2e-04" izz="1.0e-04" ixy="0.0" ixz="0.0" iyz="0.0"/>
-    </inertial>
-    <visual>
-      <origin xyz="-0.05 -0.01 0.015" rpy="0 0 0"/>
-      <geometry>
-        <mesh filename="${mesh_pkg}/ydlidar.stl" scale="0.0001 0.0001 0.0001"/>
-      </geometry>
-      <material name="dark_grey"/>
-    </visual>
-  </link>
-  <link name="battery_link">
-    <inertial>
-      <origin xyz="0.04 -0.01 0.02" rpy="0 0 0"/>
-      <mass value="0.2244"/>
-      <!-- Plausible battery-pack inertia; CAD export gave ~6e-8 (degenerate). -->
-      <inertia ixx="1.5e-04" iyy="1.5e-04" izz="1.5e-04" ixy="0.0" ixz="0.0" iyz="0.0"/>
-    </inertial>
-    <visual>
-      <origin xyz="0 0 0" rpy="0 0 0"/>
-      <geometry>
-        <mesh filename="${mesh_pkg}/battery_3s2p.stl" scale="0.001 0.001 0.001"/>
-      </geometry>
-      <material name="dark_grey"/>
-    </visual>
-  </link>
-  <!-- IMU frame (MPU9250 on the body). No mesh; small massless frame. -->
+      <mass value="0.263885"/>
+      <origin xyz="0.06489606 -0.06499993 0.02039469" rpy="0 0 0"/>
+      <inertia ixx="0.00116595" ixy="-0.00000226" ixz="0.00000001" iyy="0.00116867" iyz="0.00000004" izz="0.00226074"/>
+    </inertial>
+    <visual>
+      <origin xyz="0 0 0.005" rpy="3.140796 0 0"/>
+      <geometry><mesh filename="${mesh_pkg}/central_perforated_plate.stl" scale="0.001 0.001 0.001"/></geometry>
+      <material name="silver"/>
+    </visual>
+    <collision>
+      <origin xyz="0 0 0.005" rpy="3.140796 0 0"/>
+      <geometry><mesh filename="${mesh_pkg}/central_perforated_plate.stl" scale="0.001 0.001 0.001"/></geometry>
+    </collision>
+    <visual>
+      <origin xyz="0 0 0.035" rpy="3.140796 0 0"/>
+      <geometry><mesh filename="${mesh_pkg}/central_perforated_plate.stl" scale="0.001 0.001 0.001"/></geometry>
+      <material name="silver"/>
+    </visual>
+    <collision>
+      <origin xyz="0 0 0.035" rpy="3.140796 0 0"/>
+      <geometry><mesh filename="${mesh_pkg}/central_perforated_plate.stl" scale="0.001 0.001 0.001"/></geometry>
+    </collision>
+    <visual>
+      <origin xyz="0.001 -0.061 0.03" rpy="3.140796 0 0"/>
+      <geometry><mesh filename="${mesh_pkg}/body_standoffs.stl" scale="0.001 0.001 0.001"/></geometry>
+      <material name="silver"/>
+    </visual>
+    <collision>
+      <origin xyz="0.001 -0.061 0.03" rpy="3.140796 0 0"/>
+      <geometry><mesh filename="${mesh_pkg}/body_standoffs.stl" scale="0.001 0.001 0.001"/></geometry>
+    </collision>
+    <visual>
+      <origin xyz="0.069 -0.001 0.03" rpy="3.140796 0 -1.57"/>
+      <geometry><mesh filename="${mesh_pkg}/body_standoffs.stl" scale="0.001 0.001 0.001"/></geometry>
+      <material name="silver"/>
+    </visual>
+    <collision>
+      <origin xyz="0.069 -0.001 0.03" rpy="3.140796 0 -1.57"/>
+      <geometry><mesh filename="${mesh_pkg}/body_standoffs.stl" scale="0.001 0.001 0.001"/></geometry>
+    </collision>
+    <visual>
+      <origin xyz="0.127 -0.069 0.03" rpy="3.140796 0 3.14"/>
+      <geometry><mesh filename="${mesh_pkg}/body_standoffs.stl" scale="0.001 0.001 0.001"/></geometry>
+      <material name="silver"/>
+    </visual>
+    <collision>
+      <origin xyz="0.127 -0.069 0.03" rpy="3.140796 0 3.14"/>
+      <geometry><mesh filename="${mesh_pkg}/body_standoffs.stl" scale="0.001 0.001 0.001"/></geometry>
+    </collision>
+    <visual>
+      <origin xyz="0.068 -0.127 0.03" rpy="3.140796 0 1.57"/>
+      <geometry><mesh filename="${mesh_pkg}/body_standoffs.stl" scale="0.001 0.001 0.001"/></geometry>
+      <material name="silver"/>
+    </visual>
+    <collision>
+      <origin xyz="0.068 -0.127 0.03" rpy="3.140796 0 1.57"/>
+      <geometry><mesh filename="${mesh_pkg}/body_standoffs.stl" scale="0.001 0.001 0.001"/></geometry>
+    </collision>
+    <visual>
+      <origin xyz="0.0325 0.007 0" rpy="3.140796 0 -1.57"/>
+      <geometry><mesh filename="${mesh_pkg}/arm_perforated_plate_bottom.stl" scale="0.001 0.001 0.001"/></geometry>
+      <material name="silver"/>
+    </visual>
+    <collision>
+      <origin xyz="0.0325 0.007 0" rpy="3.140796 0 -1.57"/>
+      <geometry><mesh filename="${mesh_pkg}/arm_perforated_plate_bottom.stl" scale="0.001 0.001 0.001"/></geometry>
+    </collision>
+    <visual>
+      <origin xyz="0.137 -0.032 0" rpy="3.140796 0 3.14"/>
+      <geometry><mesh filename="${mesh_pkg}/arm_perforated_plate_bottom.stl" scale="0.001 0.001 0.001"/></geometry>
+      <material name="silver"/>
+    </visual>
+    <collision>
+      <origin xyz="0.137 -0.032 0" rpy="3.140796 0 3.14"/>
+      <geometry><mesh filename="${mesh_pkg}/arm_perforated_plate_bottom.stl" scale="0.001 0.001 0.001"/></geometry>
+    </collision>
+    <visual>
+      <origin xyz="-0.007 -0.098 0" rpy="3.140796 0 0"/>
+      <geometry><mesh filename="${mesh_pkg}/arm_perforated_plate_bottom.stl" scale="0.001 0.001 0.001"/></geometry>
+      <material name="silver"/>
+    </visual>
+    <collision>
+      <origin xyz="-0.007 -0.098 0" rpy="3.140796 0 0"/>
+      <geometry><mesh filename="${mesh_pkg}/arm_perforated_plate_bottom.stl" scale="0.001 0.001 0.001"/></geometry>
+    </collision>
+    <visual>
+      <origin xyz="0.097 -0.137 0" rpy="3.140796 0 1.57"/>
+      <geometry><mesh filename="${mesh_pkg}/arm_perforated_plate_bottom.stl" scale="0.001 0.001 0.001"/></geometry>
+      <material name="silver"/>
+    </visual>
+    <collision>
+      <origin xyz="0.097 -0.137 0" rpy="3.140796 0 1.57"/>
+      <geometry><mesh filename="${mesh_pkg}/arm_perforated_plate_bottom.stl" scale="0.001 0.001 0.001"/></geometry>
+    </collision>
+    <visual>
+      <origin xyz="0.155 -0.078 0.03" rpy="3.140796 0 -1.57"/>
+      <geometry><mesh filename="${mesh_pkg}/arm_perforated_plate_top.stl" scale="0.001 0.001 0.001"/></geometry>
+      <material name="silver"/>
+    </visual>
+    <collision>
+      <origin xyz="0.155 -0.078 0.03" rpy="3.140796 0 -1.57"/>
+      <geometry><mesh filename="${mesh_pkg}/arm_perforated_plate_top.stl" scale="0.001 0.001 0.001"/></geometry>
+    </collision>
+    <visual>
+      <origin xyz="0.052 -0.155 0.03" rpy="3.140796 0 -3.14"/>
+      <geometry><mesh filename="${mesh_pkg}/arm_perforated_plate_top.stl" scale="0.001 0.001 0.001"/></geometry>
+      <material name="silver"/>
+    </visual>
+    <collision>
+      <origin xyz="0.052 -0.155 0.03" rpy="3.140796 0 -3.14"/>
+      <geometry><mesh filename="${mesh_pkg}/arm_perforated_plate_top.stl" scale="0.001 0.001 0.001"/></geometry>
+    </collision>
+    <visual>
+      <origin xyz="0.078 0.025 0.03" rpy="3.140796 0 0"/>
+      <geometry><mesh filename="${mesh_pkg}/arm_perforated_plate_top.stl" scale="0.001 0.001 0.001"/></geometry>
+      <material name="silver"/>
+    </visual>
+    <collision>
+      <origin xyz="0.078 0.025 0.03" rpy="3.140796 0 0"/>
+      <geometry><mesh filename="${mesh_pkg}/arm_perforated_plate_top.stl" scale="0.001 0.001 0.001"/></geometry>
+    </collision>
+    <visual>
+      <origin xyz="-0.025 -0.052 0.03" rpy="3.140796 0 1.57"/>
+      <geometry><mesh filename="${mesh_pkg}/arm_perforated_plate_top.stl" scale="0.001 0.001 0.001"/></geometry>
+      <material name="silver"/>
+    </visual>
+    <collision>
+      <origin xyz="-0.025 -0.052 0.03" rpy="3.140796 0 1.57"/>
+      <geometry><mesh filename="${mesh_pkg}/arm_perforated_plate_top.stl" scale="0.001 0.001 0.001"/></geometry>
+    </collision>
+    <visual>
+      <origin xyz="-0.015 -0.0115 0.002" rpy="0.0007963268 0 0"/>
+      <geometry><mesh filename="${mesh_pkg}/servo_mg995.stl" scale="0.001 0.001 0.001"/></geometry>
+      <material name="silver"/>
+    </visual>
+    <collision>
+      <origin xyz="-0.015 -0.0115 0.002" rpy="0.0007963268 0 0"/>
+      <geometry><mesh filename="${mesh_pkg}/servo_mg995.stl" scale="0.001 0.001 0.001"/></geometry>
+    </collision>
+    <visual>
+      <origin xyz="0.011 -0.145 0.002" rpy="0.0007963268 0 1.57"/>
+      <geometry><mesh filename="${mesh_pkg}/servo_mg995.stl" scale="0.001 0.001 0.001"/></geometry>
+      <material name="silver"/>
+    </visual>
+    <collision>
+      <origin xyz="0.011 -0.145 0.002" rpy="0.0007963268 0 1.57"/>
+      <geometry><mesh filename="${mesh_pkg}/servo_mg995.stl" scale="0.001 0.001 0.001"/></geometry>
+    </collision>
+    <visual>
+      <origin xyz="0.145 -0.1185 0.002" rpy="0.0007963268 0 -3.14"/>
+      <geometry><mesh filename="${mesh_pkg}/servo_mg995.stl" scale="0.001 0.001 0.001"/></geometry>
+      <material name="silver"/>
+    </visual>
+    <collision>
+      <origin xyz="0.145 -0.1185 0.002" rpy="0.0007963268 0 -3.14"/>
+      <geometry><mesh filename="${mesh_pkg}/servo_mg995.stl" scale="0.001 0.001 0.001"/></geometry>
+    </collision>
+    <visual>
+      <origin xyz="0.1185 0.015 0.002" rpy="0.0007963268 0 -1.57"/>
+      <geometry><mesh filename="${mesh_pkg}/servo_mg995.stl" scale="0.001 0.001 0.001"/></geometry>
+      <material name="silver"/>
+    </visual>
+    <collision>
+      <origin xyz="0.1185 0.015 0.002" rpy="0.0007963268 0 -1.57"/>
+      <geometry><mesh filename="${mesh_pkg}/servo_mg995.stl" scale="0.001 0.001 0.001"/></geometry>
+    </collision>
+  </link>
   <link name="imu_link">
     <inertial>
@@ -99,368 +193,565 @@
     <visual>
       <origin xyz="0 0 0" rpy="0 0 0"/>
-      <geometry>
-        <box size="0.012 0.016 0.003"/>
-      </geometry>
+      <geometry><box size="0.012 0.016 0.003"/></geometry>
       <material name="dark_grey"/>
     </visual>
   </link>
+  <link name="battery_link">
+    <inertial>
+      <mass value="0.180000"/>
+      <origin xyz="0.00000000 0.00000000 0.01050000" rpy="0 0 0"/>
+      <inertia ixx="0.00002775" ixy="0.00000000" ixz="0.00000000" iyy="0.00018111" iyz="0.00000000" izz="0.00019011"/>
+    </inertial>
+    <visual>
+      <origin xyz="0 0 0.0105" rpy="0 0 0"/>
+      <geometry><box size="0.107 0.035 0.025"/></geometry>
+      <material name="silver"/>
+    </visual>
+    <collision>
+      <origin xyz="0 0 0.0105" rpy="0 0 0"/>
+      <geometry><box size="0.107 0.035 0.025"/></geometry>
+    </collision>
+  </link>
+  <link name="circuit_box_base_link">
+    <inertial>
+      <mass value="0.016044"/>
+      <origin xyz="0.00000000 0.00000000 0.00000000" rpy="0 0 0"/>
+      <inertia ixx="0.00001391" ixy="0.00000001" ixz="0.00000000" iyy="0.00002376" iyz="0.00000000" izz="0.00003767"/>
+    </inertial>
+    <visual>
+      <origin xyz="0 0 0" rpy="0 0 1.57"/>
+      <geometry><box size="0.102 0.1333 0.001"/></geometry>
+      <material name="silver"/>
+    </visual>
+    <collision>
+      <origin xyz="0 0 0" rpy="0 0 1.57"/>
+      <geometry><box size="0.102 0.1333 0.001"/></geometry>
+    </collision>
+  </link>
+  <link name="circuit_box_link">
+    <inertial>
+      <mass value="0.138015"/>
+      <origin xyz="0.02066488 -0.00224629 0.01891372" rpy="0 0 0"/>
+      <inertia ixx="0.00009520" ixy="-0.00001035" ixz="-0.00000298" iyy="0.00023211" iyz="-0.00000273" izz="0.00024761"/>
+    </inertial>
+    <visual>
+      <origin xyz="-0.15 -0.435 -0.01" rpy="0 0 4.71"/>
+      <geometry><mesh filename="${mesh_pkg}/uno_q_simplified.stl" scale="0.001 0.001 0.001"/></geometry>
+    </visual>
+    <collision>
+      <origin xyz="-0.15 -0.435 -0.01" rpy="0 0 4.71"/>
+      <geometry><mesh filename="${mesh_pkg}/uno_q_simplified.stl" scale="0.001 0.001 0.001"/></geometry>
+    </collision>
+    <visual>
+      <origin xyz="0.045 0 0.005" rpy="0 0 -1.57"/>
+      <geometry><mesh filename="${mesh_pkg}/buck_converter_step_down.stl" scale="0.001 0.001 0.001"/></geometry>
+    </visual>
+    <collision>
+      <origin xyz="0.045 0 0.005" rpy="0 0 -1.57"/>
+      <geometry><mesh filename="${mesh_pkg}/buck_converter_step_down.stl" scale="0.001 0.001 0.001"/></geometry>
+    </collision>
+    <visual>
+      <origin xyz="0.025 0.03 0.048" rpy="0 3.14 3.14"/>
+      <geometry><mesh filename="${mesh_pkg}/hw688_layout.stl" scale="0.001 0.001 0.001"/></geometry>
+      <material name="silver"/>
+    </visual>
+    <collision>
+      <origin xyz="0.025 0.03 0.048" rpy="0 3.14 3.14"/>
+      <geometry><mesh filename="${mesh_pkg}/hw688_layout.stl" scale="0.001 0.001 0.001"/></geometry>
+    </collision>
+    <visual>
+      <origin xyz="0.005 -0.025 0.005" rpy="1.57 0 1.57"/>
+      <geometry><mesh filename="${mesh_pkg}/pca9685.stl" scale="0.001 0.001 0.001"/></geometry>
+    </visual>
+    <collision>
+      <origin xyz="0.005 -0.025 0.005" rpy="1.57 0 1.57"/>
+      <geometry><mesh filename="${mesh_pkg}/pca9685.stl" scale="0.001 0.001 0.001"/></geometry>
+    </collision>
+    <visual>
+      <origin xyz="0 0.018 0.012" rpy="0 0 1.57"/>
+      <geometry><mesh filename="${mesh_pkg}/MPU_9265.stl" scale="0.001 0.001 0.001"/></geometry>
+    </visual>
+    <collision>
+      <origin xyz="0 0.018 0.012" rpy="0 0 1.57"/>
+      <geometry><mesh filename="${mesh_pkg}/MPU_9265.stl" scale="0.001 0.001 0.001"/></geometry>
+    </collision>
+    <visual>
+      <origin xyz="-0.065 -0.05 0.0005" rpy="0 0 0"/>
+      <geometry><mesh filename="${mesh_pkg}/body_standoffs.stl" scale="0.001 0.001 0.001"/></geometry>
+      <material name="silver"/>
+    </visual>
+    <collision>
+      <origin xyz="-0.065 -0.05 0.0005" rpy="0 0 0"/>
+      <geometry><mesh filename="${mesh_pkg}/body_standoffs.stl" scale="0.001 0.001 0.001"/></geometry>
+    </collision>
+    <visual>
+      <origin xyz="-0.065 -0.05 0.0255" rpy="0 0 0"/>
+      <geometry><mesh filename="${mesh_pkg}/body_standoffs.stl" scale="0.001 0.001 0.001"/></geometry>
+      <material name="silver"/>
+    </visual>
+    <collision>
+      <origin xyz="-0.065 -0.05 0.0255" rpy="0 0 0"/>
+      <geometry><mesh filename="${mesh_pkg}/body_standoffs.stl" scale="0.001 0.001 0.001"/></geometry>
+    </collision>
+    <visual>
+      <origin xyz="-0.065 0.042 0" rpy="0 0 0"/>
+      <geometry><mesh filename="${mesh_pkg}/body_standoffs.stl" scale="0.001 0.001 0.001"/></geometry>
+      <material name="silver"/>
+    </visual>
+    <collision>
+      <origin xyz="-0.065 0.042 0" rpy="0 0 0"/>
+      <geometry><mesh filename="${mesh_pkg}/body_standoffs.stl" scale="0.001 0.001 0.001"/></geometry>
+    </collision>
+    <visual>
+      <origin xyz="-0.065 0.042 0.0255" rpy="0 0 0"/>
+      <geometry><mesh filename="${mesh_pkg}/body_standoffs.stl" scale="0.001 0.001 0.001"/></geometry>
+      <material name="silver"/>
+    </visual>
+    <collision>
+      <origin xyz="-0.065 0.042 0.0255" rpy="0 0 0"/>
+      <geometry><mesh filename="${mesh_pkg}/body_standoffs.stl" scale="0.001 0.001 0.001"/></geometry>
+    </collision>
+    <visual>
+      <origin xyz="0.065 0.049 0.0005" rpy="0 0 3.14"/>
+      <geometry><mesh filename="${mesh_pkg}/body_standoffs.stl" scale="0.001 0.001 0.001"/></geometry>
+      <material name="silver"/>
+    </visual>
+    <collision>
+      <origin xyz="0.065 0.049 0.0005" rpy="0 0 3.14"/>
+      <geometry><mesh filename="${mesh_pkg}/body_standoffs.stl" scale="0.001 0.001 0.001"/></geometry>
+    </collision>
+    <visual>
+      <origin xyz="0.065 0.049 0.0255" rpy="0 0 3.14"/>
+      <geometry><mesh filename="${mesh_pkg}/body_standoffs.stl" scale="0.001 0.001 0.001"/></geometry>
+      <material name="silver"/>
+    </visual>
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