Commit message: feat: mshes updated for big_berth_description

File: big_bertha_description/urdf/big_bertha.gazebo.xacro (robot description, xacro)
@@ -3,5 +3,5 @@
   Gazebo Harmonic (gz-sim 8) sensor + surface configuration for Big Bertha.
   Provides:
-    - a 2D lidar (YDLidar X2 class) on lidar_link  -> gz topic "scan"
+    - a 2D lidar (YDLidar X2 class) on ydlidar_link  -> gz topic "scan"
     - an IMU (MPU9250 class) on imu_link           -> gz topic "imu"
     - per-link friction/material surface properties.
@@ -103,10 +103,10 @@
   <!-- ============================ Lidar ============================== -->
   <!-- YDLidar X2: 360 deg, ~8 m range, 5 Hz. Published on gz topic "scan",
-       frame_id = lidar_link. -->
-  <gazebo reference="lidar_link">
+       frame_id = ydlidar_link. -->
+  <gazebo reference="ydlidar_link">
     <material>Gazebo/DarkGrey</material>
     <sensor name="lidar" type="gpu_lidar">
       <topic>scan</topic>
-      <gz_frame_id>lidar_link</gz_frame_id>
+      <gz_frame_id>ydlidar_link</gz_frame_id>
       <update_rate>10</update_rate>
       <always_on>true</always_on>

File: big_bertha_description/urdf/big_bertha.urdf.xacro (robot description, xacro)
@@ -20,19 +20,11 @@
 -->
 <robot name="big_bertha" xmlns:xacro="http://www.ros.org/wiki/xacro">
-  <!-- ============================ Arguments ============================ -->
-  <!-- Use ros2_control + gz sensors when running in Gazebo; disable for a
-       pure visualisation / check_urdf pass. -->
   <xacro:arg name="use_gz" default="true"/>
-  <!-- ros2_control.yaml passed to the gz_ros2_control plugin. -->
   <xacro:arg name="ros2_control_config"
              default="$(find big_bertha_description)/config/ros2_control.yaml"/>
-  <!-- Forwarded to the gz OdometryPublisher in big_bertha.gazebo.xacro. -->
   <xacro:arg name="publish_odom" default="true"/>
-  <!-- When false, the EKF (state_estimation) owns the odom->base_link tf. -->
   <xacro:arg name="odom_tf" default="true"/>
-  <!-- Sim-only kinematic drive (gz VelocityControl) for verification gates. -->
   <xacro:arg name="sim_drive" default="false"/>
   <xacro:property name="use_gz" value="$(arg use_gz)"/>
-  <!-- ============================ Materials ============================ -->
   <material name="silver">
     <color rgba="0.700 0.700 0.700 1.000"/>
@@ -41,5 +33,4 @@
     <color rgba="0.200 0.200 0.200 1.000"/>
   </material>
-  <!-- ======================= Convenience macros ======================= -->
   <xacro:property name="mesh_pkg" value="package://big_bertha_description/meshes"/>
   <!-- ============================== Links ============================== -->
@@ -549,11 +540,9 @@
     <visual>
       <origin xyz="0 0 0" rpy="0 0 0"/>
-      <geometry>
-        <box size="0.012 0.016 0.003"/>
-      </geometry>
+      <geometry><box size="0.012 0.016 0.003"/></geometry>
       <material name="dark_grey"/>
     </visual>
   </link>
-  <link name="arm_a_4_1">
+  <link name="battery_link">
     <inertial>
       <origin xyz="-0.00051903 -0.01742240 -0.04805902" rpy="0 0 0"/>
@@ -655,4 +644,5 @@
     </collision>
   </link>
+  <!-- arm_a_1_1 (front-left, leg 1) -->
   <link name="arm_a_1_1">
     <inertial>
@@ -747,4 +737,5 @@
     </collision>
   </link>
+  <!-- arm_a_2_1 (front-right, leg 2) -->
   <link name="arm_a_2_1">
     <inertial>
@@ -830,4 +821,5 @@
     </collision>
   </link>
+  <!-- arm_a_3_1 (back-right, leg 3) -->
   <link name="arm_a_3_1">
     <inertial>
@@ -1061,5 +1053,4 @@
     <child link="imu_link"/>
   </joint>
-  <!-- =================== ros2_control + Gazebo plugins ================= -->
   <xacro:if value="${use_gz}">
     <xacro:include filename="$(find big_bertha_description)/urdf/big_bertha.ros2_control.xacro"/>

Commit message: fix: Stable PD controller + 1000 Hz physics for mass-corrected inertia
The v1.0.0 URDF's real per-link mass/inertia (vs the old placeholders)
pushed JointEffortPdController's explicit-PD stability ratio (kp*dt^2/I)
past the project's own documented ~1.4 ceiling for the calf/foot link,
which chattered at the hardware velocity limit every control tick.

Fixes it two ways:
- Stable PD (Tan, Liu & Turk, "Stable Proportional-Derivative
  Controllers"): the P-term is evaluated against the predicted next-step
  position (q + dt*qd) instead of the current q, which is unconditionally
  stable for kd >= kp*dt (true here by a wide margin).
- Physics/controller_manager rate raised 500 -> 1000 Hz for a comfortable
  margin (ratio ~1.74 -> ~0.43) on top of the algorithmic fix.

Also: ground plane friction raised to match the feet's own mu (1.5) --
Gazebo/DART combines contact friction by MINIMUM of the two surfaces,
unlike Isaac's "multiply" combine, so the old ground mu=1.0 gave the feet
a third less effective grip than training. controller spawner
--switch-timeout raised to 30s: the full-fidelity URDF (all of training's
circuit-box detail meshes) takes gz longer to load/activate than the 5s
default allows.

File: big_bertha_description/urdf/big_bertha.gazebo.xacro (robot description, xacro)
@@ -59,5 +59,5 @@
   </xacro:if>
   <!-- ===================== Friction / materials ====================== -->
-  <xacro:macro name="bb_surface" params="link color:=Gazebo/Silver mu:=1.0">
+  <xacro:macro name="bb_surface" params="link color:=Gazebo/Silver mu:=1.0 soft:=false">
     <gazebo reference="${link}">
       <material>${color}</material>
@@ -68,21 +68,37 @@
            clean spheres). Legs do not overlap in a normal gait. -->
       <self_collide>false</self_collide>
+      <!-- Foot contact softness: DART's default (near-rigid) contact stiffness
+           was tuned implicitly against the old, ~2x-too-heavy foot mass. The
+           v1.0.0 mass correction (0.12 to 0.0637 kg per calf/foot link, see
+           big_bertha.urdf.xacro) halved the foot's mass without softening the
+           contact spring, so the natural contact frequency ~sqrt(kp/m) roughly
+           doubled, observed as joint velocity pinned at the hardware cap
+           (6.54 rad/s) in perfect 4 leg sync every control tick, a genuine
+           physical resonance, not a PD/damping tunable oscillation (confirmed
+           unresponsive to a 12.5x joint PD kd increase). kp/kd here are ODE
+           contact spring stiffness/damping (N/m, Ns/m), not the joint PD gains.
+      -->
+      <xacro:if value="${soft}">
+        <kp>1.0e5</kp>
+        <kd>10.0</kd>
+      </xacro:if>
     </gazebo>
   </xacro:macro>
   <!-- Feet (arm_c_*) get high friction to match the training ground
-       (static/dynamic 1.0); body + upper links a touch lower. -->
+       (static/dynamic 1.0) and softened contact for the lighter foot mass;
+       body + upper links a touch lower friction, default (rigid) contact. -->
   <xacro:bb_surface link="base_link"  mu="0.6"/>
   <xacro:bb_surface link="arm_a_1_1"  mu="0.6"/>
   <xacro:bb_surface link="arm_b_1_1"  mu="0.6"/>
-  <xacro:bb_surface link="arm_c_1_1"  mu="1.5"/>
+  <xacro:bb_surface link="arm_c_1_1"  mu="1.5" soft="true"/>
   <xacro:bb_surface link="arm_a_2_1"  mu="0.6"/>
   <xacro:bb_surface link="arm_b_2_1"  mu="0.6"/>
-  <xacro:bb_surface link="arm_c_2_1"  mu="1.5"/>
+  <xacro:bb_surface link="arm_c_2_1"  mu="1.5" soft="true"/>
   <xacro:bb_surface link="arm_a_3_1"  mu="0.6"/>
   <xacro:bb_surface link="arm_b_3_1"  mu="0.6"/>
-  <xacro:bb_surface link="arm_c_3_1"  mu="1.5"/>
+  <xacro:bb_surface link="arm_c_3_1"  mu="1.5" soft="true"/>
   <xacro:bb_surface link="arm_a_4_1"  mu="0.6"/>
   <xacro:bb_surface link="arm_b_4_1"  mu="0.6"/>
-  <xacro:bb_surface link="arm_c_4_1"  mu="1.5"/>
+  <xacro:bb_surface link="arm_c_4_1"  mu="1.5" soft="true"/>
   <!-- ============================ Lidar ============================== -->
   <!-- YDLidar X2: 360 deg, ~8 m range, 5 Hz. Published on gz topic "scan",
