Commit message: feat(bringup): swap MPU-6500 IMU for BNO055 on-chip fusion
Replace the magnetometer-less MPU-6500 with a BNO055 read in NDOF mode on
the STM32U585 co-processor, giving absolute heading instead of unbounded
yaw drift.

- firmware: BNO055 driver (boot handshake, CONFIG->NDOF, fused quaternion
  + accel/gyro/mag at 100 Hz), IMU sent as a single comma-CSV string to
  stay under the router arg limit; imu_diag now reports chip_id/op_mode/
  calib_* nibbles
- node: publish fused orientation with real covariance, parse CSV payload,
  status key mpu9250_ok -> imu_ok
- remove imu_filter_madgwick node/config/dependency; consumers point at
  /imu (fused) instead of /filtered/imu
- update imu_scanner/i2c_scanner diagnostic apps, configs, scripts, and
  docs/URDF (mesh renamed BNO055.stl)
- IMU axis signs and quaternion convention kept from old mount and flagged
  for bench validation

File: big_bertha_description/urdf/big_bertha.gazebo.xacro (robot description, xacro)
@@ -4,5 +4,5 @@
   Provides:
     - a 2D lidar (YDLidar X2 class) on lidar_link  -> gz topic "scan"
-    - an IMU (MPU9250 class) on imu_link           -> gz topic "imu"
+    - an IMU (BNO055 class) on imu_link           -> gz topic "imu"
     - per-link friction/material surface properties.
   The ros_gz_bridge (simulation module) maps these gz topics onto the ROS 2
@@ -150,5 +150,5 @@
   </gazebo>
   <!-- ============================= IMU =============================== -->
-  <!-- MPU9250 class IMU on imu_link. Published on gz topic "imu",
+  <!-- BNO055 class IMU on imu_link. Published on gz topic "imu",
        frame_id = imu_link. -->
   <gazebo reference="imu_link">

File: big_bertha_description/urdf/big_bertha.urdf.xacro (robot description, xacro)
@@ -12,5 +12,5 @@
     - a 12-joint position ros2_control block,
     - a gz 2D lidar sensor on lidar_link (YDLidar X2),
-    - a gz IMU sensor on imu_link (MPU6050, identity rotation vs base_link,
+    - a gz IMU sensor on imu_link (BNO055, identity rotation vs base_link,
       matching training's ImuCfg convention),
     - gz friction/material surface properties.
@@ -410,5 +410,5 @@
       <origin xyz="0 0.018 0.012" rpy="0 0 1.57"/>
       <geometry>
-        <mesh filename="${mesh_pkg}/MPU_9265.stl" scale="0.001 0.001 0.001"/>
+        <mesh filename="${mesh_pkg}/BNO055.stl" scale="0.001 0.001 0.001"/>
       </geometry>
       <material name="silver"/>
@@ -417,5 +417,5 @@
       <origin xyz="0 0.018 0.012" rpy="0 0 1.57"/>
       <geometry>
-        <mesh filename="${mesh_pkg}/MPU_9265.stl" scale="0.001 0.001 0.001"/>
+        <mesh filename="${mesh_pkg}/BNO055.stl" scale="0.001 0.001 0.001"/>
       </geometry>
     </collision>
@@ -538,7 +538,7 @@
     </collision>
   </link>
-  <!-- IMU frame (MPU6050 on the body; hardware BOM name). No mesh.
+  <!-- IMU frame (BNO055 on the body; hardware BOM name). No mesh.
        Identity rotation vs base_link, matching training's ImuCfg
-       convention (not the MPU_9265 mesh's own cosmetic mount rotation). -->
+       convention (not the BNO055.stl mesh's own cosmetic mount rotation). -->
   <link name="imu_link">
     <inertial>
@@ -1054,6 +1054,6 @@
   <!-- IMU stays a direct base_link child (not chained through circuit_box)
        so its rotation is identity vs base_link, matching training's own
-       ImuCfg convention (rot=(1,0,0,0)) rather than the MPU_9265 mesh's own
-       cosmetic mount rotation inside circuit_box_link. -->
+       ImuCfg convention (rot=(1,0,0,0)) rather than the BNO055.stl mesh's
+       own cosmetic mount rotation inside circuit_box_link. -->
   <joint name="imu_joint" type="fixed">
     <origin xyz="0.0657 -0.0657 0.0614" rpy="0 0 0"/>

Commit message: fix(description): restore MPU_9265.stl mesh and URDF references

File: big_bertha_description/urdf/big_bertha.gazebo.xacro (robot description, xacro)
@@ -4,5 +4,5 @@
   Provides:
     - a 2D lidar (YDLidar X2 class) on lidar_link  -> gz topic "scan"
-    - an IMU (BNO055 class) on imu_link           -> gz topic "imu"
+    - an IMU (MPU9250 class) on imu_link           -> gz topic "imu"
     - per-link friction/material surface properties.
   The ros_gz_bridge (simulation module) maps these gz topics onto the ROS 2
@@ -150,5 +150,5 @@
   </gazebo>
   <!-- ============================= IMU =============================== -->
-  <!-- BNO055 class IMU on imu_link. Published on gz topic "imu",
+  <!-- MPU9250 class IMU on imu_link. Published on gz topic "imu",
        frame_id = imu_link. -->
   <gazebo reference="imu_link">

File: big_bertha_description/urdf/big_bertha.urdf.xacro (robot description, xacro)
@@ -12,5 +12,5 @@
     - a 12-joint position ros2_control block,
     - a gz 2D lidar sensor on lidar_link (YDLidar X2),
-    - a gz IMU sensor on imu_link (BNO055, identity rotation vs base_link,
+    - a gz IMU sensor on imu_link (MPU6050, identity rotation vs base_link,
       matching training's ImuCfg convention),
     - gz friction/material surface properties.
@@ -410,5 +410,5 @@
       <origin xyz="0 0.018 0.012" rpy="0 0 1.57"/>
       <geometry>
-        <mesh filename="${mesh_pkg}/BNO055.stl" scale="0.001 0.001 0.001"/>
+        <mesh filename="${mesh_pkg}/MPU_9265.stl" scale="0.001 0.001 0.001"/>
       </geometry>
       <material name="silver"/>
@@ -417,5 +417,5 @@
       <origin xyz="0 0.018 0.012" rpy="0 0 1.57"/>
       <geometry>
-        <mesh filename="${mesh_pkg}/BNO055.stl" scale="0.001 0.001 0.001"/>
+        <mesh filename="${mesh_pkg}/MPU_9265.stl" scale="0.001 0.001 0.001"/>
       </geometry>
     </collision>
@@ -538,7 +538,7 @@
     </collision>
   </link>
-  <!-- IMU frame (BNO055 on the body; hardware BOM name). No mesh.
+  <!-- IMU frame (MPU6050 on the body; hardware BOM name). No mesh.
        Identity rotation vs base_link, matching training's ImuCfg
-       convention (not the BNO055.stl mesh's own cosmetic mount rotation). -->
+       convention (not the MPU_9265 mesh's own cosmetic mount rotation). -->
   <link name="imu_link">
     <inertial>
@@ -1054,6 +1054,6 @@
   <!-- IMU stays a direct base_link child (not chained through circuit_box)
        so its rotation is identity vs base_link, matching training's own
-       ImuCfg convention (rot=(1,0,0,0)) rather than the BNO055.stl mesh's
-       own cosmetic mount rotation inside circuit_box_link. -->
+       ImuCfg convention (rot=(1,0,0,0)) rather than the MPU_9265 mesh's own
+       cosmetic mount rotation inside circuit_box_link. -->
   <joint name="imu_joint" type="fixed">
     <origin xyz="0.0657 -0.0657 0.0614" rpy="0 0 0"/>
