Commit message: chore: restore main plant, my tuning made the walk lurch
Reverts the base_link centring, rigid foot contact, the trained battery
mass, the hip/knee armature and the friction raise. The description and
world are now byte-identical to main.

I had been optimising net displacement and ignoring how the robot looked.
Measured on the straight walk with the v2.0.0 policy, pitch peak-to-peak
is the number that tracks 'walks well':

  main geometry + main plant     0.081 m/s   pitch  9.3 deg
  centred geometry + main plant  0.066       pitch 10.6
  + my mass and armature         0.072       pitch 15.2
  + my friction raise            0.099       pitch 17.4

My changes nearly doubled the pitching. The friction raise bought speed by
letting the feet catch, which is exactly the lurching and toppling that
made the gif unwatchable. Main's plant is both faster than my tuned plant
and half as violent, so it wins on both counts.

The centred base_link costs 18% of speed and a degree of pitch on its own
with no measured benefit, so it goes too; the frame convention question is
deferred to v2.1 regardless. This PR now ships the v2.0.0 policy and the
demo tooling against main's proven plant.

189 tests pass.

File: big_bertha_description/urdf/big_bertha.gazebo.xacro (robot description, xacro)
@@ -79,14 +79,4 @@
            contact spring stiffness/damping (N/m, Ns/m), not the joint PD gains.
       -->
-      <!-- REGRESSION WARNING: the feet were set soft="true" again at some
-           point after this was first fixed, and it cost ~18% of forward speed
-           (0.084 down to 0.071 m/s, measured on the straight walk). Isaac
-           trains on RIGID foot ground contact; a compliant foot yields under
-           load exactly when push off needs normal force, so the legs cycle on
-           schedule but the body barely moves, which looks like the robot is
-           walking on the spot. Keep soft="false" unless the velocity limit
-           resonance returns, and note the 1000 Hz world physics already holds
-           that at bay: p99 joint velocity measured 3.78 of 7.2 rad/s with
-           rigid contact. -->
       <xacro:if value="${soft}">
         <kp>1.0e5</kp>
@@ -95,12 +85,5 @@
     </gazebo>
   </xacro:macro>
-  <!-- Feet mu 3.0, NOT Isaac's effective 1.5. DART needs roughly double to
-       reach the same grip: measured on the straight walk, 1.5 gives 0.072 m/s
-       with feet sliding 7.4 m per metre of body advance, 3.0 gives 0.099 m/s
-       at 4.9, and 6.0 only reaches 0.106 while pitching worse (18.7 vs 17.4
-       deg) and sagging lower. 3.0 is the knee of that curve. Raising it
-       further does not help because what still slides are feet dragging under
-       near-zero load, which no friction coefficient fixes.
-       Feet (arm_c_*) get high friction to match the training ground
+  <!-- Feet (arm_c_*) get high friction to match the training ground
        (static/dynamic 1.0) and softened contact for the lighter foot mass;
        body + upper links a touch lower friction, default (rigid) contact. -->
@@ -108,14 +91,14 @@
   <xacro:bb_surface link="arm_a_1_1"  mu="0.6"/>
   <xacro:bb_surface link="arm_b_1_1"  mu="0.6"/>
-  <xacro:bb_surface link="arm_c_1_1"  mu="3.0" soft="false"/>
+  <xacro:bb_surface link="arm_c_1_1"  mu="1.5" soft="true"/>
   <xacro:bb_surface link="arm_a_2_1"  mu="0.6"/>
   <xacro:bb_surface link="arm_b_2_1"  mu="0.6"/>
-  <xacro:bb_surface link="arm_c_2_1"  mu="3.0" soft="false"/>
+  <xacro:bb_surface link="arm_c_2_1"  mu="1.5" soft="true"/>
   <xacro:bb_surface link="arm_a_3_1"  mu="0.6"/>
   <xacro:bb_surface link="arm_b_3_1"  mu="0.6"/>
-  <xacro:bb_surface link="arm_c_3_1"  mu="3.0" soft="false"/>
+  <xacro:bb_surface link="arm_c_3_1"  mu="1.5" soft="true"/>
   <xacro:bb_surface link="arm_a_4_1"  mu="0.6"/>
   <xacro:bb_surface link="arm_b_4_1"  mu="0.6"/>
-  <xacro:bb_surface link="arm_c_4_1"  mu="3.0" soft="false"/>
+  <xacro:bb_surface link="arm_c_4_1"  mu="1.5" soft="true"/>
   <xacro:bb_surface link="battery_link"          mu="0.6"/>
   <xacro:bb_surface link="circuit_box_base_link" mu="0.6"/>

File: big_bertha_description/urdf/big_bertha.urdf.xacro (robot description, xacro)
@@ -46,10 +46,10 @@
   <link name="base_link">
     <inertial>
-      <origin xyz="0 0 0.02039469" rpy="0 0 0"/>
+      <origin xyz="0.06489606 -0.06499993 0.02039469" rpy="0 0 0"/>
       <mass value="0.263885"/>
       <inertia ixx="0.00116595" ixy="-0.00000226" ixz="0.00000001" iyy="0.00116867" iyz="0.00000004" izz="0.00226074"/>
     </inertial>
     <visual>
-      <origin xyz="-0.06489606 0.06499993 0.005" rpy="3.140796 -0 0"/>
+      <origin xyz="0 -0 0.005" rpy="3.140796 -0 0"/>
       <geometry>
         <mesh filename="${mesh_pkg}/central_perforated_plate.stl" scale="0.001 0.001 0.001"/>
@@ -58,5 +58,5 @@
     </visual>
     <collision>
-      <origin xyz="-0.06489606 0.06499993 0.005" rpy="3.140796 -0 0"/>
+      <origin xyz="0 -0 0.005" rpy="3.140796 -0 0"/>
       <geometry>
         <mesh filename="${mesh_pkg}/central_perforated_plate.stl" scale="0.001 0.001 0.001"/>
@@ -64,5 +64,5 @@
     </collision>
     <visual>
-      <origin xyz="-0.06489606 0.06499993 0.035" rpy="3.140796 -0 0"/>
+      <origin xyz="0 -0 0.035" rpy="3.140796 -0 0"/>
       <geometry>
         <mesh filename="${mesh_pkg}/central_perforated_plate.stl" scale="0.001 0.001 0.001"/>
@@ -71,5 +71,5 @@
     </visual>
     <collision>
-      <origin xyz="-0.06489606 0.06499993 0.035" rpy="3.140796 -0 0"/>
+      <origin xyz="0 -0 0.035" rpy="3.140796 -0 0"/>
       <geometry>
         <mesh filename="${mesh_pkg}/central_perforated_plate.stl" scale="0.001 0.001 0.001"/>
@@ -77,57 +77,57 @@
     </collision>
     <visual>
-      <origin xyz="-0.06389606 0.00399993 0.03" rpy="3.140796 -0 0"/>
-      <geometry>
-        <mesh filename="${mesh_pkg}/body_standoffs.stl" scale="0.001 0.001 0.001"/>
-      </geometry>
-      <material name="silver"/>
-    </visual>
-    <collision>
-      <origin xyz="-0.06389606 0.00399993 0.03" rpy="3.140796 -0 0"/>
-      <geometry>
-        <mesh filename="${mesh_pkg}/body_standoffs.stl" scale="0.001 0.001 0.001"/>
-      </geometry>
-    </collision>
-    <visual>
-      <origin xyz="0.00410394 0.06399993 0.03" rpy="3.140796 -0 -1.57"/>
-      <geometry>
-        <mesh filename="${mesh_pkg}/body_standoffs.stl" scale="0.001 0.001 0.001"/>
-      </geometry>
-      <material name="silver"/>
-    </visual>
-    <collision>
-      <origin xyz="0.00410394 0.06399993 0.03" rpy="3.140796 -0 -1.57"/>
-      <geometry>
-        <mesh filename="${mesh_pkg}/body_standoffs.stl" scale="0.001 0.001 0.001"/>
-      </geometry>
-    </collision>
-    <visual>
-      <origin xyz="0.06210394 -0.00400007 0.03" rpy="3.140796 -0 3.14"/>
-      <geometry>
-        <mesh filename="${mesh_pkg}/body_standoffs.stl" scale="0.001 0.001 0.001"/>
-      </geometry>
-      <material name="silver"/>
-    </visual>
-    <collision>
-      <origin xyz="0.06210394 -0.00400007 0.03" rpy="3.140796 -0 3.14"/>
-      <geometry>
-        <mesh filename="${mesh_pkg}/body_standoffs.stl" scale="0.001 0.001 0.001"/>
-      </geometry>
-    </collision>
-    <visual>
-      <origin xyz="0.00310394 -0.06200007 0.03" rpy="3.140796 -0 1.57"/>
-      <geometry>
-        <mesh filename="${mesh_pkg}/body_standoffs.stl" scale="0.001 0.001 0.001"/>
-      </geometry>
-      <material name="silver"/>
-    </visual>
-    <collision>
-      <origin xyz="0.00310394 -0.06200007 0.03" rpy="3.140796 -0 1.57"/>
-      <geometry>
-        <mesh filename="${mesh_pkg}/body_standoffs.stl" scale="0.001 0.001 0.001"/>
-      </geometry>
-    </collision>
-    <visual>
-      <origin xyz="-0.03239606 0.07199993 0" rpy="3.140796 -0 -1.57"/>
+      <origin xyz="0.001 -0.061 0.03" rpy="3.140796 -0 0"/>
+      <geometry>
+        <mesh filename="${mesh_pkg}/body_standoffs.stl" scale="0.001 0.001 0.001"/>
+      </geometry>
+      <material name="silver"/>
+    </visual>
+    <collision>
+      <origin xyz="0.001 -0.061 0.03" rpy="3.140796 -0 0"/>
+      <geometry>
+        <mesh filename="${mesh_pkg}/body_standoffs.stl" scale="0.001 0.001 0.001"/>
+      </geometry>
+    </collision>
+    <visual>
+      <origin xyz="0.069 -0.001 0.03" rpy="3.140796 -0 -1.57"/>
+      <geometry>
+        <mesh filename="${mesh_pkg}/body_standoffs.stl" scale="0.001 0.001 0.001"/>
+      </geometry>
+      <material name="silver"/>
+    </visual>
+    <collision>
+      <origin xyz="0.069 -0.001 0.03" rpy="3.140796 -0 -1.57"/>
+      <geometry>
+        <mesh filename="${mesh_pkg}/body_standoffs.stl" scale="0.001 0.001 0.001"/>
+      </geometry>
+    </collision>
+    <visual>
+      <origin xyz="0.127 -0.069 0.03" rpy="3.140796 -0 3.14"/>
+      <geometry>
+        <mesh filename="${mesh_pkg}/body_standoffs.stl" scale="0.001 0.001 0.001"/>
+      </geometry>
+      <material name="silver"/>
+    </visual>
+    <collision>
+      <origin xyz="0.127 -0.069 0.03" rpy="3.140796 -0 3.14"/>
+      <geometry>
+        <mesh filename="${mesh_pkg}/body_standoffs.stl" scale="0.001 0.001 0.001"/>
+      </geometry>
+    </collision>
+    <visual>
+      <origin xyz="0.068 -0.127 0.03" rpy="3.140796 -0 1.57"/>
+      <geometry>
+        <mesh filename="${mesh_pkg}/body_standoffs.stl" scale="0.001 0.001 0.001"/>
+      </geometry>
+      <material name="silver"/>
+    </visual>
+    <collision>
+      <origin xyz="0.068 -0.127 0.03" rpy="3.140796 -0 1.57"/>
+      <geometry>
+        <mesh filename="${mesh_pkg}/body_standoffs.stl" scale="0.001 0.001 0.001"/>
+      </geometry>
+    </collision>
+    <visual>
+      <origin xyz="0.0325 0.007 0" rpy="3.140796 -0 -1.57"/>
       <geometry>
         <mesh filename="${mesh_pkg}/arm_perforated_plate_bottom.stl" scale="0.001 0.001 0.001"/>
@@ -136,5 +136,5 @@
     </visual>
     <collision>
-      <origin xyz="-0.03239606 0.07199993 0" rpy="3.140796 -0 -1.57"/>
+      <origin xyz="0.0325 0.007 0" rpy="3.140796 -0 -1.57"/>
       <geometry>
         <mesh filename="${mesh_pkg}/arm_perforated_plate_bottom.stl" scale="0.001 0.001 0.001"/>
@@ -142,5 +142,5 @@
     </collision>
     <visual>
-      <origin xyz="0.07210394 0.03299993 0" rpy="3.140796 -0 3.14"/>
+      <origin xyz="0.137 -0.032 0" rpy="3.140796 -0 3.14"/>
       <geometry>
         <mesh filename="${mesh_pkg}/arm_perforated_plate_bottom.stl" scale="0.001 0.001 0.001"/>
@@ -149,5 +149,5 @@
     </visual>
     <collision>
-      <origin xyz="0.07210394 0.03299993 0" rpy="3.140796 -0 3.14"/>
+      <origin xyz="0.137 -0.032 0" rpy="3.140796 -0 3.14"/>
       <geometry>
         <mesh filename="${mesh_pkg}/arm_perforated_plate_bottom.stl" scale="0.001 0.001 0.001"/>
@@ -155,5 +155,5 @@
     </collision>
     <visual>
-      <origin xyz="-0.07189606 -0.03300007 0" rpy="3.140796 -0 0"/>
+      <origin xyz="-0.007 -0.098 0" rpy="3.140796 -0 0"/>
       <geometry>
         <mesh filename="${mesh_pkg}/arm_perforated_plate_bottom.stl" scale="0.001 0.001 0.001"/>
@@ -162,5 +162,5 @@
     </visual>
     <collision>
-      <origin xyz="-0.07189606 -0.03300007 0" rpy="3.140796 -0 0"/>
+      <origin xyz="-0.007 -0.098 0" rpy="3.140796 -0 0"/>
       <geometry>
         <mesh filename="${mesh_pkg}/arm_perforated_plate_bottom.stl" scale="0.001 0.001 0.001"/>
@@ -168,5 +168,5 @@
     </collision>
     <visual>
-      <origin xyz="0.03210394 -0.07200007 0" rpy="3.140796 -0 1.57"/>
+      <origin xyz="0.097 -0.137 0" rpy="3.140796 -0 1.57"/>
       <geometry>
         <mesh filename="${mesh_pkg}/arm_perforated_plate_bottom.stl" scale="0.001 0.001 0.001"/>
@@ -175,5 +175,5 @@
     </visual>
     <collision>
-      <origin xyz="0.03210394 -0.07200007 0" rpy="3.140796 -0 1.57"/>
+      <origin xyz="0.097 -0.137 0" rpy="3.140796 -0 1.57"/>
       <geometry>
         <mesh filename="${mesh_pkg}/arm_perforated_plate_bottom.stl" scale="0.001 0.001 0.001"/>
@@ -181,5 +181,5 @@
     </collision>
     <visual>
-      <origin xyz="0.09010394 -0.01300007 0.03" rpy="3.140796 -0 -1.57"/>
+      <origin xyz="0.155 -0.078 0.03" rpy="3.140796 -0 -1.57"/>
       <geometry>
         <mesh filename="${mesh_pkg}/arm_perforated_plate_top.stl" scale="0.001 0.001 0.001"/>
@@ -188,5 +188,5 @@
     </visual>
     <collision>
-      <origin xyz="0.09010394 -0.01300007 0.03" rpy="3.140796 -0 -1.57"/>
+      <origin xyz="0.155 -0.078 0.03" rpy="3.140796 -0 -1.57"/>
       <geometry>
         <mesh filename="${mesh_pkg}/arm_perforated_plate_top.stl" scale="0.001 0.001 0.001"/>
@@ -194,5 +194,5 @@
     </collision>
     <visual>
-      <origin xyz="-0.01289606 -0.09000007 0.03" rpy="3.140796 -0 -3.14"/>
+      <origin xyz="0.052 -0.155 0.03" rpy="3.140796 -0 -3.14"/>
       <geometry>
         <mesh filename="${mesh_pkg}/arm_perforated_plate_top.stl" scale="0.001 0.001 0.001"/>
@@ -201,5 +201,5 @@
     </visual>
     <collision>
-      <origin xyz="-0.01289606 -0.09000007 0.03" rpy="3.140796 -0 -3.14"/>
+      <origin xyz="0.052 -0.155 0.03" rpy="3.140796 -0 -3.14"/>
       <geometry>
         <mesh filename="${mesh_pkg}/arm_perforated_plate_top.stl" scale="0.001 0.001 0.001"/>
@@ -207,5 +207,5 @@
     </collision>
     <visual>
-      <origin xyz="0.01310394 0.08999993 0.03" rpy="3.140796 -0 0"/>
+      <origin xyz="0.078 0.025 0.03" rpy="3.140796 -0 0"/>
       <geometry>
         <mesh filename="${mesh_pkg}/arm_perforated_plate_top.stl" scale="0.001 0.001 0.001"/>
@@ -214,5 +214,5 @@
     </visual>
     <collision>
-      <origin xyz="0.01310394 0.08999993 0.03" rpy="3.140796 -0 0"/>
+      <origin xyz="0.078 0.025 0.03" rpy="3.140796 -0 0"/>
       <geometry>
         <mesh filename="${mesh_pkg}/arm_perforated_plate_top.stl" scale="0.001 0.001 0.001"/>
@@ -220,5 +220,5 @@
     </collision>
     <visual>
-      <origin xyz="-0.08989606 0.01299993 0.03" rpy="3.140796 -0 1.57"/>
+      <origin xyz="-0.025 -0.052 0.03" rpy="3.140796 -0 1.57"/>
       <geometry>
         <mesh filename="${mesh_pkg}/arm_perforated_plate_top.stl" scale="0.001 0.001 0.001"/>
@@ -227,5 +227,5 @@
     </visual>
     <collision>
-      <origin xyz="-0.08989606 0.01299993 0.03" rpy="3.140796 -0 1.57"/>
+      <origin xyz="-0.025 -0.052 0.03" rpy="3.140796 -0 1.57"/>
       <geometry>
         <mesh filename="${mesh_pkg}/arm_perforated_plate_top.stl" scale="0.001 0.001 0.001"/>
@@ -233,51 +233,51 @@
     </collision>
     <visual>
-      <origin xyz="-0.07989606 0.05349993 0.002" rpy="0.0007963268 -0 0"/>
-      <geometry>
-        <mesh filename="${mesh_pkg}/servo_mg995.stl" scale="0.001 0.001 0.001"/>
-      </geometry>
-      <material name="silver"/>
-    </visual>
-    <collision>
-      <origin xyz="-0.07989606 0.05349993 0.002" rpy="0.0007963268 -0 0"/>
-      <geometry>
-        <mesh filename="${mesh_pkg}/servo_mg995.stl" scale="0.001 0.001 0.001"/>
-      </geometry>
-    </collision>
-    <visual>
-      <origin xyz="-0.05389606 -0.08000007 0.002" rpy="0.0007963268 -0 1.57"/>
-      <geometry>
-        <mesh filename="${mesh_pkg}/servo_mg995.stl" scale="0.001 0.001 0.001"/>
-      </geometry>
-      <material name="silver"/>
-    </visual>
-    <collision>
-      <origin xyz="-0.05389606 -0.08000007 0.002" rpy="0.0007963268 -0 1.57"/>
-      <geometry>
-        <mesh filename="${mesh_pkg}/servo_mg995.stl" scale="0.001 0.001 0.001"/>
-      </geometry>
-    </collision>
-    <visual>
-      <origin xyz="0.08010394 -0.05350007 0.002" rpy="0.0007963268 -0 -3.14"/>
-      <geometry>
-        <mesh filename="${mesh_pkg}/servo_mg995.stl" scale="0.001 0.001 0.001"/>
-      </geometry>
-      <material name="silver"/>
-    </visual>
-    <collision>
-      <origin xyz="0.08010394 -0.05350007 0.002" rpy="0.0007963268 -0 -3.14"/>
-      <geometry>
-        <mesh filename="${mesh_pkg}/servo_mg995.stl" scale="0.001 0.001 0.001"/>
-      </geometry>
-    </collision>
-    <visual>
-      <origin xyz="0.05360394 0.07999993 0.002" rpy="0.0007963268 -0 -1.57"/>
-      <geometry>
-        <mesh filename="${mesh_pkg}/servo_mg995.stl" scale="0.001 0.001 0.001"/>
-      </geometry>
-      <material name="silver"/>
-    </visual>
-    <collision>
-      <origin xyz="0.05360394 0.07999993 0.002" rpy="0.0007963268 -0 -1.57"/>
+      <origin xyz="-0.015 -0.0115 0.002" rpy="0.0007963268 -0 0"/>
+      <geometry>
+        <mesh filename="${mesh_pkg}/servo_mg995.stl" scale="0.001 0.001 0.001"/>
+      </geometry>
+      <material name="silver"/>
+    </visual>
+    <collision>
+      <origin xyz="-0.015 -0.0115 0.002" rpy="0.0007963268 -0 0"/>
+      <geometry>
+        <mesh filename="${mesh_pkg}/servo_mg995.stl" scale="0.001 0.001 0.001"/>
+      </geometry>
+    </collision>
+    <visual>
+      <origin xyz="0.011 -0.145 0.002" rpy="0.0007963268 -0 1.57"/>
+      <geometry>
+        <mesh filename="${mesh_pkg}/servo_mg995.stl" scale="0.001 0.001 0.001"/>
+      </geometry>
+      <material name="silver"/>
+    </visual>
+    <collision>
+      <origin xyz="0.011 -0.145 0.002" rpy="0.0007963268 -0 1.57"/>
+      <geometry>
+        <mesh filename="${mesh_pkg}/servo_mg995.stl" scale="0.001 0.001 0.001"/>
+      </geometry>
+    </collision>
+    <visual>
+      <origin xyz="0.145 -0.1185 0.002" rpy="0.0007963268 -0 -3.14"/>
+      <geometry>
+        <mesh filename="${mesh_pkg}/servo_mg995.stl" scale="0.001 0.001 0.001"/>
+      </geometry>
+      <material name="silver"/>
+    </visual>
+    <collision>
+      <origin xyz="0.145 -0.1185 0.002" rpy="0.0007963268 -0 -3.14"/>
+      <geometry>
+        <mesh filename="${mesh_pkg}/servo_mg995.stl" scale="0.001 0.001 0.001"/>
+      </geometry>
+    </collision>
+    <visual>
+      <origin xyz="0.1185 0.015 0.002" rpy="0.0007963268 -0 -1.57"/>
+      <geometry>
+        <mesh filename="${mesh_pkg}/servo_mg995.stl" scale="0.001 0.001 0.001"/>
+      </geometry>
+      <material name="silver"/>
+    </visual>
+    <collision>
+      <origin xyz="0.1185 0.015 0.002" rpy="0.0007963268 -0 -1.57"/>
       <geometry>
         <mesh filename="${mesh_pkg}/servo_mg995.stl" scale="0.001 0.001 0.001"/>
@@ -312,10 +312,6 @@
     <inertial>
       <origin xyz="0 0 0.0105" rpy="0 0 0"/>
-      <!-- 0.5 kg, matching the training URDF. This carried 0.18 kg, which made
-           the deployed robot ~1.13 kg against the ~1.45 kg the policy trained
-           on. Friction is mu*N, so a 22% lighter body has 22% less normal force
-           and the feet skid instead of pushing off. -->
-      <mass value="0.5"/>
-      <inertia ixx="0.00034198" ixy="0.0" ixz="0.0" iyy="0.00058075" iyz="0.0" izz="0.00073864"/>
+      <mass value="0.18"/>
+      <inertia ixx="0.00002775" ixy="0.0" ixz="0.0" iyy="0.00018111" iyz="0.0" izz="0.00019011"/>
     </inertial>
     <visual>
@@ -563,5 +559,5 @@
       <origin xyz="-0.00051903 -0.01742240 -0.04805902" rpy="0 0 0"/>
       <mass value="0.061703"/>
-      <inertia ixx="0.00201630" ixy="-0.00000008" ixz="-0.00000046" iyy="0.00201265" iyz="0.00000033" izz="0.00201841"/>
+      <inertia ixx="0.00001630" ixy="-0.00000008" ixz="-0.00000046" iyy="0.00001265" iyz="0.00000033" izz="0.00001841"/>
     </inertial>
     <visual>
@@ -596,5 +592,5 @@
       <origin xyz="0.04154098 -0.00048149 0.00107965" rpy="0 0 0"/>
       <mass value="0.008137"/>
-      <inertia ixx="0.00200479" ixy="-0.00000000" ixz="-0.00000001" iyy="0.00200378" iyz="0.00000000" izz="0.00200801"/>
+      <inertia ixx="0.00000479" ixy="-0.00000000" ixz="-0.00000001" iyy="0.00000378" iyz="0.00000000" izz="0.00000801"/>
     </inertial>
     <visual>
@@ -659,19 +655,9 @@
     </collision>
   </link>
-  <!-- ARMATURE ON HIPS AND KNEES. Training adds armature to Revolute_.* (ALL
-       twelve joints, 0.005 pinned in clean eval); only the calf links carried
-       it here, so hips and knees ran with none and the legs decoupled. Folding
-       it into link inertia is an approximation: unlike true joint armature it
-       also adds parasitic inertia to the chain, which costs forward speed, so
-       the value here is 0.002 rather than training's 0.005. Measured: ankle
-       amplitude asymmetry (legs 1&4 vs 2&3, Isaac = 1.00) 1.30 -> 1.07 at
-       0.002 and 1.13 at 0.005, with speed 0.086 -> 0.072 and 0.055 m/s.
-       A proper fix needs joint-level armature, which sdformat14 and the
-       dartsim plugin do not expose; that wants a custom gz-sim system plugin. -->
   <link name="arm_a_1_1">
     <inertial>
       <origin xyz="-0.00089507 -0.01742240 -0.05050470" rpy="0 0 0"/>
       <mass value="0.061703"/>
-      <inertia ixx="0.00201640" ixy="-0.00000009" ixz="-0.00000040" iyy="0.00201271" iyz="0.00000034" izz="0.00201836"/>
+      <inertia ixx="0.00001640" ixy="-0.00000009" ixz="-0.00000040" iyy="0.00001271" iyz="0.00000034" izz="0.00001836"/>
     </inertial>
     <visual>
@@ -706,5 +692,5 @@
       <origin xyz="0.04154098 -0.00048149 0.00107965" rpy="0 0 0"/>
       <mass value="0.008137"/>
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