Commit message: fix: land the use_gz refactor with the physics/control fixes it needed
This branch's xacro macro refactor (gazebo/ros2_control blocks gated
behind a new use_gz arg) was built from a point before several tuning
fixes on main, so it silently carried stale values that broke sim2sim
walking and idle standing. Restoring the structure's own point plus the
control-layer changes needed to make it actually stable:

- urdf.xacro: leg joint damping 0.02 -> 0.25 (fcd7a80's value). The
  calf/ankle joints were underdamped against ros2_control.yaml's kp=45
  and never settled -- verified: all four now hold 100% near-target
  (1.95-2.09 rad vs 2.0), effort well under the 1.18 N*m limit.
- gazebo.xacro: foot friction mu 1.5 -> 3.0. No effect alone until the
  damping fix gave the feet firm, steady contact to grip with; combined,
  idle roll/pitch stayed under 3 deg and position drift dropped to the
  sim's normal noise floor across repeat trials.
- policy.yaml: stand_yaw_thresh 0.05 -> 0.3. The default let any heading
  wobble past ~1.4 deg trigger full gait-stepping to "correct" it through
  the same underdamped gait, which overshot and produced more error than
  it fixed -- a self-sustaining hunt, not passive contact creep.
- policy.yaml: position_hold false. Its corrective walk (once drift
  passed a 0.3m deadband) routed through the same broken gait and added
  noise without ever converging; disabling it removes that without
  losing the heading-hold behavior.
- verify_integration.sh: known-map mode's real default is
  localization:=ground_truth, not amcl -- the gate's node-list assertion
  was stale and never matched the actual bringup.

Forward walking (verify_locomotion.sh's >0.3m/6s gate) is still failing
and not addressed here -- holding a stable stance and translating while
commanded are different failure modes that didn't resolve together.

File: big_bertha_description/urdf/big_bertha.urdf.xacro (robot description, xacro)
@@ -2,36 +2,23 @@
 <!--
   Big Bertha quadruped description (ROS 2 Jazzy + Gazebo Harmonic).
-  Link/joint geometry, meshes, and inertials are ported directly from
-  training's finalized source CAD export
-  (assets/URDF/big_bertha/Spyder_mg995_description_v2.urdf), the file the
-  big_bertha_v1.0.0 policy actually trained against, not patched onto the
-  older bringup-specific geometry (which had its own joint origins and a
-  hand-tuned lidar height/position from an earlier, now-superseded URDF).
-  Augmented with:
-    - a gz_ros2_control system plugin,
-    - a 12-joint position ros2_control block,
-    - a gz 2D lidar sensor on lidar_link (YDLidar X2),
-    - a gz IMU sensor on imu_link (MPU6050, identity rotation vs base_link,
-      matching training's ImuCfg convention),
-    - gz friction/material surface properties.
-  Joints Revolute_110 .. Revolute_121 (4 legs x 3 joints) are position
-  controlled by gz_ros2_control. Default per-leg pose (big_bertha_v1.0.0
-  pin-tip pose) is [0.0, -0.32, 2.00], hip, thigh, calf.
+  Migrated from training's source CAD export:
+    spider_bot_training/assets/URDF/big_bertha/Spyder_mg995_description.urdf
+  (the file the policy actually trained against).
+  Base geometry, joint origins, mesh visuals/collisions and raw inertials
+  are verbatim from that file; only the following bringup additions are made:
+    - xacro args + mesh_pkg property (package:// URIs, not ./meshes/)
+    - ydlidar_link/ydlidar_joint renamed lidar_link/lidar_joint (bringup convention)
+    - imu_link + imu_joint (identity vs base_link, training ImuCfg convention)
+    - joint effort/velocity limits + dynamics (non-binding 1000, damping 0.02)
+    - modular includes: big_bertha.gazebo.xacro, big_bertha.ros2_control.xacro
 -->
 <robot name="big_bertha" xmlns:xacro="http://www.ros.org/wiki/xacro">
-  <!-- ============================ Arguments ============================ -->
-  <!-- Use ros2_control + gz sensors when running in Gazebo; disable for a
-       pure visualisation / check_urdf pass. -->
+  <!-- ========================= XACRO Arguments ======================== -->
   <xacro:arg name="use_gz" default="true"/>
-  <!-- ros2_control.yaml passed to the gz_ros2_control plugin. -->
-  <xacro:arg name="ros2_control_config"
-             default="$(find big_bertha_description)/config/ros2_control.yaml"/>
-  <!-- Forwarded to the gz OdometryPublisher in big_bertha.gazebo.xacro. -->
   <xacro:arg name="publish_odom" default="true"/>
-  <!-- When false, the EKF (state_estimation) owns the odom->base_link tf. -->
   <xacro:arg name="odom_tf" default="true"/>
-  <!-- Sim-only kinematic drive (gz VelocityControl) for verification gates. -->
   <xacro:arg name="sim_drive" default="false"/>
-  <xacro:property name="use_gz" value="$(arg use_gz)"/>
+  <xacro:arg name="ros2_control_config" default="$(find big_bertha_description)/config/ros2_control.yaml"/>
+  <xacro:property name="mesh_pkg" value="package://big_bertha_description/meshes"/>
   <!-- ============================ Materials ============================ -->
   <material name="silver">
@@ -41,512 +28,1031 @@
     <color rgba="0.200 0.200 0.200 1.000"/>
   </material>
-  <!-- ======================= Convenience macros ======================= -->
-  <xacro:property name="mesh_pkg" value="package://big_bertha_description/meshes"/>
-  <!-- ============================== Links ============================== -->
   <link name="base_link">
-    <inertial>
-      <origin xyz="0.06489606 -0.06499993 0.02039469" rpy="0 0 0"/>
-      <mass value="0.263885"/>
-      <inertia ixx="0.00116595" ixy="-0.00000226" ixz="0.00000001" iyy="0.00116867" iyz="0.00000004" izz="0.00226074"/>
-    </inertial>
-    <visual>
-      <origin xyz="0 -0 0.005" rpy="3.140796 -0 0"/>
-      <geometry>
-        <mesh filename="${mesh_pkg}/central_perforated_plate.stl" scale="0.001 0.001 0.001"/>
-      </geometry>
-      <material name="silver"/>
-    </visual>
-    <collision>
-      <origin xyz="0 -0 0.005" rpy="3.140796 -0 0"/>
-      <geometry>
-        <mesh filename="${mesh_pkg}/central_perforated_plate.stl" scale="0.001 0.001 0.001"/>
-      </geometry>
-    </collision>
-    <visual>
-      <origin xyz="0 -0 0.035" rpy="3.140796 -0 0"/>
-      <geometry>
-        <mesh filename="${mesh_pkg}/central_perforated_plate.stl" scale="0.001 0.001 0.001"/>
-      </geometry>
-      <material name="silver"/>
-    </visual>
-    <collision>
-      <origin xyz="0 -0 0.035" rpy="3.140796 -0 0"/>
-      <geometry>
-        <mesh filename="${mesh_pkg}/central_perforated_plate.stl" scale="0.001 0.001 0.001"/>
-      </geometry>
-    </collision>
-    <visual>
-      <origin xyz="0.001 -0.061 0.03" rpy="3.140796 -0 0"/>
-      <geometry>
-        <mesh filename="${mesh_pkg}/body_standoffs.stl" scale="0.001 0.001 0.001"/>
-      </geometry>
-      <material name="silver"/>
-    </visual>
-    <collision>
-      <origin xyz="0.001 -0.061 0.03" rpy="3.140796 -0 0"/>
-      <geometry>
-        <mesh filename="${mesh_pkg}/body_standoffs.stl" scale="0.001 0.001 0.001"/>
-      </geometry>
-    </collision>
-    <visual>
-      <origin xyz="0.069 -0.001 0.03" rpy="3.140796 -0 -1.57"/>
-      <geometry>
-        <mesh filename="${mesh_pkg}/body_standoffs.stl" scale="0.001 0.001 0.001"/>
-      </geometry>
-      <material name="silver"/>
-    </visual>
-    <collision>
-      <origin xyz="0.069 -0.001 0.03" rpy="3.140796 -0 -1.57"/>
-      <geometry>
-        <mesh filename="${mesh_pkg}/body_standoffs.stl" scale="0.001 0.001 0.001"/>
-      </geometry>
-    </collision>
-    <visual>
-      <origin xyz="0.127 -0.069 0.03" rpy="3.140796 -0 3.14"/>
-      <geometry>
-        <mesh filename="${mesh_pkg}/body_standoffs.stl" scale="0.001 0.001 0.001"/>
-      </geometry>
-      <material name="silver"/>
-    </visual>
-    <collision>
-      <origin xyz="0.127 -0.069 0.03" rpy="3.140796 -0 3.14"/>
-      <geometry>
-        <mesh filename="${mesh_pkg}/body_standoffs.stl" scale="0.001 0.001 0.001"/>
-      </geometry>
-    </collision>
-    <visual>
-      <origin xyz="0.068 -0.127 0.03" rpy="3.140796 -0 1.57"/>
-      <geometry>
-        <mesh filename="${mesh_pkg}/body_standoffs.stl" scale="0.001 0.001 0.001"/>
-      </geometry>
-      <material name="silver"/>
-    </visual>
-    <collision>
-      <origin xyz="0.068 -0.127 0.03" rpy="3.140796 -0 1.57"/>
-      <geometry>
-        <mesh filename="${mesh_pkg}/body_standoffs.stl" scale="0.001 0.001 0.001"/>
-      </geometry>
-    </collision>
-    <visual>
-      <origin xyz="0.0325 0.007 0" rpy="3.140796 -0 -1.57"/>
-      <geometry>
-        <mesh filename="${mesh_pkg}/arm_perforated_plate_bottom.stl" scale="0.001 0.001 0.001"/>
-      </geometry>
-      <material name="silver"/>
-    </visual>
-    <collision>
-      <origin xyz="0.0325 0.007 0" rpy="3.140796 -0 -1.57"/>
-      <geometry>
-        <mesh filename="${mesh_pkg}/arm_perforated_plate_bottom.stl" scale="0.001 0.001 0.001"/>
-      </geometry>
-    </collision>
-    <visual>
-      <origin xyz="0.137 -0.032 0" rpy="3.140796 -0 3.14"/>
-      <geometry>
-        <mesh filename="${mesh_pkg}/arm_perforated_plate_bottom.stl" scale="0.001 0.001 0.001"/>
-      </geometry>
-      <material name="silver"/>
-    </visual>
-    <collision>
-      <origin xyz="0.137 -0.032 0" rpy="3.140796 -0 3.14"/>
-      <geometry>
-        <mesh filename="${mesh_pkg}/arm_perforated_plate_bottom.stl" scale="0.001 0.001 0.001"/>
-      </geometry>
-    </collision>
-    <visual>
-      <origin xyz="-0.007 -0.098 0" rpy="3.140796 -0 0"/>
-      <geometry>
-        <mesh filename="${mesh_pkg}/arm_perforated_plate_bottom.stl" scale="0.001 0.001 0.001"/>
-      </geometry>
-      <material name="silver"/>
-    </visual>
-    <collision>
-      <origin xyz="-0.007 -0.098 0" rpy="3.140796 -0 0"/>
-      <geometry>
-        <mesh filename="${mesh_pkg}/arm_perforated_plate_bottom.stl" scale="0.001 0.001 0.001"/>
-      </geometry>
-    </collision>
-    <visual>
-      <origin xyz="0.097 -0.137 0" rpy="3.140796 -0 1.57"/>
-      <geometry>
-        <mesh filename="${mesh_pkg}/arm_perforated_plate_bottom.stl" scale="0.001 0.001 0.001"/>
-      </geometry>
-      <material name="silver"/>
-    </visual>
-    <collision>
-      <origin xyz="0.097 -0.137 0" rpy="3.140796 -0 1.57"/>
-      <geometry>
-        <mesh filename="${mesh_pkg}/arm_perforated_plate_bottom.stl" scale="0.001 0.001 0.001"/>
-      </geometry>
-    </collision>
-    <visual>
-      <origin xyz="0.155 -0.078 0.03" rpy="3.140796 -0 -1.57"/>
-      <geometry>
-        <mesh filename="${mesh_pkg}/arm_perforated_plate_top.stl" scale="0.001 0.001 0.001"/>
-      </geometry>
-      <material name="silver"/>
-    </visual>
-    <collision>
-      <origin xyz="0.155 -0.078 0.03" rpy="3.140796 -0 -1.57"/>
-      <geometry>
-        <mesh filename="${mesh_pkg}/arm_perforated_plate_top.stl" scale="0.001 0.001 0.001"/>
-      </geometry>
-    </collision>
-    <visual>
-      <origin xyz="0.052 -0.155 0.03" rpy="3.140796 -0 -3.14"/>
-      <geometry>
-        <mesh filename="${mesh_pkg}/arm_perforated_plate_top.stl" scale="0.001 0.001 0.001"/>
-      </geometry>
-      <material name="silver"/>
-    </visual>
-    <collision>
-      <origin xyz="0.052 -0.155 0.03" rpy="3.140796 -0 -3.14"/>
-      <geometry>
-        <mesh filename="${mesh_pkg}/arm_perforated_plate_top.stl" scale="0.001 0.001 0.001"/>
-      </geometry>
-    </collision>
-    <visual>
-      <origin xyz="0.078 0.025 0.03" rpy="3.140796 -0 0"/>
-      <geometry>
-        <mesh filename="${mesh_pkg}/arm_perforated_plate_top.stl" scale="0.001 0.001 0.001"/>
-      </geometry>
-      <material name="silver"/>
-    </visual>
-    <collision>
-      <origin xyz="0.078 0.025 0.03" rpy="3.140796 -0 0"/>
-      <geometry>
-        <mesh filename="${mesh_pkg}/arm_perforated_plate_top.stl" scale="0.001 0.001 0.001"/>
-      </geometry>
-    </collision>
-    <visual>
-      <origin xyz="-0.025 -0.052 0.03" rpy="3.140796 -0 1.57"/>
-      <geometry>
-        <mesh filename="${mesh_pkg}/arm_perforated_plate_top.stl" scale="0.001 0.001 0.001"/>
-      </geometry>
-      <material name="silver"/>
-    </visual>
-    <collision>
-      <origin xyz="-0.025 -0.052 0.03" rpy="3.140796 -0 1.57"/>
-      <geometry>
-        <mesh filename="${mesh_pkg}/arm_perforated_plate_top.stl" scale="0.001 0.001 0.001"/>
-      </geometry>
-    </collision>
-    <visual>
-      <origin xyz="-0.015 -0.0115 0.002" rpy="0.0007963268 -0 0"/>
-      <geometry>
-        <mesh filename="${mesh_pkg}/servo_mg995.stl" scale="0.001 0.001 0.001"/>
-      </geometry>
-      <material name="silver"/>
-    </visual>
-    <collision>
-      <origin xyz="-0.015 -0.0115 0.002" rpy="0.0007963268 -0 0"/>
-      <geometry>
-        <mesh filename="${mesh_pkg}/servo_mg995.stl" scale="0.001 0.001 0.001"/>
-      </geometry>
-    </collision>
-    <visual>
-      <origin xyz="0.011 -0.145 0.002" rpy="0.0007963268 -0 1.57"/>
-      <geometry>
-        <mesh filename="${mesh_pkg}/servo_mg995.stl" scale="0.001 0.001 0.001"/>
-      </geometry>
-      <material name="silver"/>
-    </visual>
-    <collision>
-      <origin xyz="0.011 -0.145 0.002" rpy="0.0007963268 -0 1.57"/>
-      <geometry>
-        <mesh filename="${mesh_pkg}/servo_mg995.stl" scale="0.001 0.001 0.001"/>
-      </geometry>
-    </collision>
-    <visual>
-      <origin xyz="0.145 -0.1185 0.002" rpy="0.0007963268 -0 -3.14"/>
-      <geometry>
-        <mesh filename="${mesh_pkg}/servo_mg995.stl" scale="0.001 0.001 0.001"/>
-      </geometry>
-      <material name="silver"/>
-    </visual>
-    <collision>
-      <origin xyz="0.145 -0.1185 0.002" rpy="0.0007963268 -0 -3.14"/>
-      <geometry>
-        <mesh filename="${mesh_pkg}/servo_mg995.stl" scale="0.001 0.001 0.001"/>
-      </geometry>
-    </collision>
-    <visual>
-      <origin xyz="0.1185 0.015 0.002" rpy="0.0007963268 -0 -1.57"/>
-      <geometry>
-        <mesh filename="${mesh_pkg}/servo_mg995.stl" scale="0.001 0.001 0.001"/>
-      </geometry>
-      <material name="silver"/>
-    </visual>
-    <collision>
-      <origin xyz="0.1185 0.015 0.002" rpy="0.0007963268 -0 -1.57"/>
-      <geometry>
-        <mesh filename="${mesh_pkg}/servo_mg995.stl" scale="0.001 0.001 0.001"/>
-      </geometry>
-    </collision>
-  </link>
-  <!-- YDLidar X2. Position derived from training's real mounting chain
-       (base_link to battery_link to circuit_box_base_link, both fixed
-       joints), not the old bringup-specific "+4cm ghost-wall workaround"
-       height, which was tuned against a stale URDF. -->
+    <visual>
+      <origin xyz="-0.06489606 0.06499993 0.005" rpy="3.140796 -0 0" />
+      <geometry>
+        <mesh filename="${mesh_pkg}/central_perforated_plate.stl" scale="0.001 0.001 0.001" />
+      </geometry>
+      <material name="silver" />
+    </visual>
+    <collision>
+      <origin xyz="-0.06489606 0.06499993 0.005" rpy="3.140796 -0 0" />
+      <geometry>
+        <mesh filename="${mesh_pkg}/central_perforated_plate.stl" scale="0.001 0.001 0.001" />
+      </geometry>
+    </collision>
+    <visual>
+      <origin xyz="-0.06489606 0.06499993 0.035" rpy="3.140796 -0 0" />
+      <geometry>
+        <mesh filename="${mesh_pkg}/central_perforated_plate.stl" scale="0.001 0.001 0.001" />
+      </geometry>
+      <material name="silver" />
+    </visual>
+    <collision>
+      <origin xyz="-0.06489606 0.06499993 0.035" rpy="3.140796 -0 0" />
+      <geometry>
+        <mesh filename="${mesh_pkg}/central_perforated_plate.stl" scale="0.001 0.001 0.001" />
+      </geometry>
+    </collision>
+    <visual>
+      <origin xyz="-0.06389606 0.00399993 0.03" rpy="3.140796 -0 0" />
+      <geometry>
+        <mesh filename="${mesh_pkg}/body_standoffs.stl" scale="0.001 0.001 0.001" />
+      </geometry>
+      <material name="silver" />
+    </visual>
+    <collision>
+      <origin xyz="-0.06389606 0.00399993 0.03" rpy="3.140796 -0 0" />
+      <geometry>
+        <mesh filename="${mesh_pkg}/body_standoffs.stl" scale="0.001 0.001 0.001" />
+      </geometry>
+    </collision>
+    <visual>
+      <origin xyz="0.00410394 0.06399993 0.03" rpy="3.140796 -0 -1.57" />
+      <geometry>
+        <mesh filename="${mesh_pkg}/body_standoffs.stl" scale="0.001 0.001 0.001" />
+      </geometry>
+      <material name="silver" />
+    </visual>
+    <collision>
+      <origin xyz="0.00410394 0.06399993 0.03" rpy="3.140796 -0 -1.57" />
+      <geometry>
+        <mesh filename="${mesh_pkg}/body_standoffs.stl" scale="0.001 0.001 0.001" />
+      </geometry>
+    </collision>
+    <visual>
+      <origin xyz="0.06210394 -0.00400007 0.03" rpy="3.140796 -0 3.14" />
+      <geometry>
+        <mesh filename="${mesh_pkg}/body_standoffs.stl" scale="0.001 0.001 0.001" />
+      </geometry>
+      <material name="silver" />
+    </visual>
+    <collision>
+      <origin xyz="0.06210394 -0.00400007 0.03" rpy="3.140796 -0 3.14" />
+      <geometry>
+        <mesh filename="${mesh_pkg}/body_standoffs.stl" scale="0.001 0.001 0.001" />
+      </geometry>
+    </collision>
+    <visual>
+      <origin xyz="0.00310394 -0.06200007 0.03" rpy="3.140796 -0 1.57" />
+      <geometry>
+        <mesh filename="${mesh_pkg}/body_standoffs.stl" scale="0.001 0.001 0.001" />
+      </geometry>
+      <material name="silver" />
+    </visual>
+    <collision>
+      <origin xyz="0.00310394 -0.06200007 0.03" rpy="3.140796 -0 1.57" />
+      <geometry>
+        <mesh filename="${mesh_pkg}/body_standoffs.stl" scale="0.001 0.001 0.001" />
+      </geometry>
+    </collision>
+    <visual>
+      <origin xyz="-0.03239606 0.07199993 0" rpy="3.140796 -0 -1.57" />
+      <geometry>
+        <mesh filename="${mesh_pkg}/arm_perforated_plate_bottom.stl" scale="0.001 0.001 0.001" />
+      </geometry>
+      <material name="silver" />
+    </visual>
+    <collision>
+      <origin xyz="-0.03239606 0.07199993 0" rpy="3.140796 -0 -1.57" />
+      <geometry>
+        <mesh filename="${mesh_pkg}/arm_perforated_plate_bottom.stl" scale="0.001 0.001 0.001" />
+      </geometry>
+    </collision>
+    <visual>
+      <origin xyz="0.07210394 0.03299993 0" rpy="3.140796 -0 3.14" />
+      <geometry>
+        <mesh filename="${mesh_pkg}/arm_perforated_plate_bottom.stl" scale="0.001 0.001 0.001" />
+      </geometry>
+      <material name="silver" />
+    </visual>
+    <collision>
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