Commit message: fix: per-foot contact sensing, real-dt gait clock, and hip-bias headroom
Adds per-foot Gazebo contact sensors (ground truth, not a proxy) and a
contact-based landing-assist v3 in the policy controller, shipped
disabled -- the sensor watches each leg's whole primary collision mesh
rather than an isolated toe, so it reads near-constant contact and the
assist never usefully engages. Kept because the sensing pipeline itself
is correct and may be useful once there's an isolated toe collision to
reference.

Adds per-joint-group action scale (hip/knee/ankle), defaulting to
action_scale for exact parity. Every amplitude boost tried on this sim
(knee 0.3-1.0, alone or with ankle/friction) either did nothing or hurt
walking distance, unlike the same technique's real win on the hardware
branch -- shipped unused, parity only.

Fixes a real gait-clock bug: advance_clock() was called with a fixed
1/control_rate_ dt per decimated policy step instead of measured
elapsed time. The underlying sim-time timer fires in bursts under load
(84% of decimated steps logged under 15ms apart, impossible at a
steady 200Hz), so the fixed-dt assumption silently desynced the gait
phase from real elapsed time. Now uses measured dt, capped only on the
high end for a startup/re-enable gap.

Raises steer_max 0.26 -> 0.4 (heading-hold hip-bias authority). Idle
drift is a real, deterministic ~1-1.5cm/s creep -- same direction on
every independent fresh-spawn trial, not solver noise -- traced to
arm_c_2_1/arm_c_3_1 not matching training's URDF (training has them
byte-identical; ours match neither each other nor training). URDF
stays out of scope; this is a measured, non-regressing 17% reduction
in idle drift via the one lever available on the controller side.

Comment corrections in obstacle_world.sdf/policy.yaml reflect what was
actually measured this round, including a correction to an earlier
friction note that was itself based on since-invalidated batch
measurements (verify_locomotion.sh and idle checks don't respawn the
robot between trials, so multi-trial batches without a full respawn
aren't independent samples -- this produced multiple false
conclusions before being caught; see plan doc / project memory).

Walking-gate forward progress remains open. Best measured config
(fresh respawn per trial, proper methodology) reaches ~0.09-0.12m
over 6s @ vx=0.3 against the 0.3m gate -- closer than earlier batch
testing suggested, but not passing.

Co-Authored-By: Claude Sonnet 5 <noreply@anthropic.com>
Claude-Session: https://claude.ai/code/session_01XDLXHfxpPPWwmqHVw2hj3a

File: big_bertha_description/urdf/big_bertha.gazebo.xacro (robot description, xacro)
@@ -128,4 +128,58 @@
       </sensor>
     </gazebo>
+    <!-- ==================== Foot contact sensors ======================= -->
+    <!-- Ground-truth per-foot contact, for the policy controller's landing
+         assist (see big_bertha_policy_controller). References each foot's
+         PRIMARY collision only (arm_c_N_1_collision: the main leg/foot
+         mesh, auto-named by the URDF->SDF collision-ordering convention,
+         confirmed by dry-running `gz sdf -p` on the expanded urdf). This is
+         the same collision the training env treats as "the foot tip" (see
+         big_bertha_env.py's _tip_offset comment), deliberately NOT the
+         secondary servo-housing collision (arm_c_N_1_collision_1), which
+         isn't the ground-contact surface. Requires gz-sim-contact-system,
+         already loaded in obstacle_world.sdf. Additive only: no link,
+         joint, or collision element is moved or added; this just attaches
+         a sensor to existing geometry. -->
+    <!-- NOTE: the contact sensor publishes on the topic nested inside
+         <contact>, NOT the generic sensor-level <topic> that other sensor
+         types (lidar/imu) use: confirmed empirically, the outer <topic>
+         was silently ignored, gz only had a publisher on the
+         auto-generated default topic until this was fixed. -->
+    <gazebo reference="arm_c_1_1">
+      <sensor name="foot_contact" type="contact">
+        <update_rate>200</update_rate>
+        <contact>
+          <collision>arm_c_1_1_collision</collision>
+          <topic>foot_contact/leg1</topic>
+        </contact>
+      </sensor>
+    </gazebo>
+    <gazebo reference="arm_c_2_1">
+      <sensor name="foot_contact" type="contact">
+        <update_rate>200</update_rate>
+        <contact>
+          <collision>arm_c_2_1_collision</collision>
+          <topic>foot_contact/leg2</topic>
+        </contact>
+      </sensor>
+    </gazebo>
+    <gazebo reference="arm_c_3_1">
+      <sensor name="foot_contact" type="contact">
+        <update_rate>200</update_rate>
+        <contact>
+          <collision>arm_c_3_1_collision</collision>
+          <topic>foot_contact/leg3</topic>
+        </contact>
+      </sensor>
+    </gazebo>
+    <gazebo reference="arm_c_4_1">
+      <sensor name="foot_contact" type="contact">
+        <update_rate>200</update_rate>
+        <contact>
+          <collision>arm_c_4_1_collision</collision>
+          <topic>foot_contact/leg4</topic>
+        </contact>
+      </sensor>
+    </gazebo>
   </xacro:macro>
 </robot>
