Commit message: feat: heading_lock for straight demo + lidar +4cm
- heading_lock: hold a fixed world heading (demo_straight uses due-East via the spawn yaw) instead of latching the ~14 deg south heading the robot settles into during the DART warmup drop, so the gait walks a true straight line; off for nav (Nav2 owns heading)
- plumbed through policy_controller.launch.py (heading_lock, heading_lock_yaw) and demo_straight.launch.py
- lidar_joint z 0.041 -> 0.081 (+4 cm)

File: big_bertha_description/urdf/big_bertha.urdf.xacro (robot description, xacro)
@@ -444,5 +444,5 @@
   <!-- Fixed sensor / payload frames -->
   <joint name="lidar_joint" type="fixed">
-    <origin xyz="0.01 0.01 0.041" rpy="0 0 0"/>
+    <origin xyz="0.01 0.01 0.081" rpy="0 0 0"/>
     <parent link="base_link"/>
     <child link="lidar_link"/>

Commit message: feat: IMU scan filter + in-place turns end ghost-wall obstacle stall
- scan_ground_filter (rclcpp): rotate each lidar ray by the IMU orientation
  and drop returns whose 3D endpoint lands at/below the floor, removing the
  ghost walls the tilting body lidar painted (EKF two_d_mode -> flat TF)
- costmaps + collision monitor now consume /scan_filtered
- nav2: use_rotate_to_heading for hard turns to escape obstacles; revert the
  collision lookahead 0.4->1.0 (0.4 clipped obstacles)
- raise lidar +4 cm (0.081->0.121) for a geometric ghost-wall margin
- deploy flatter+turn policy: reaches the diagonal goal with 0 recoveries

File: big_bertha_description/urdf/big_bertha.urdf.xacro (robot description, xacro)
@@ -444,5 +444,9 @@
   <!-- Fixed sensor / payload frames -->
   <joint name="lidar_joint" type="fixed">
-    <origin xyz="0.01 0.01 0.081" rpy="0 0 0"/>
+    <!-- z 0.081 to 0.121 (+4 cm): a higher body lidar needs more body pitch
+         before its beam reaches the floor, so the gait's tilt produces fewer,
+         farther ground hits (the geometric half of the ghost-wall fix; the
+         scan_ground_filter node is the perception half). -->
+    <origin xyz="0.01 0.01 0.121" rpy="0 0 0"/>
     <parent link="base_link"/>
     <child link="lidar_link"/>
