Commit message: feat(isaac): Isaac Sim bringup with lidar ghost-scan mitigations
Adds the Isaac Sim bringup path (isaac_bringup.launch.py, isaac_simulation
.launch.py, scripts/isaac/) alongside the existing Gazebo bringup, plus a
run of fixes for lidar ghost scans discovered while validating it:

- scripts/isaac/launch_isaac.py: real obstacle_world.sdf-mirrored room
  geometry (was a 3-box placeholder), rotation_rate left at Gazebo-matching
  10.0 after a rotation_rate=0 experiment measured worse, and lidar_joint
  raised +0.02m in big_bertha.urdf.xacro (untested against a re-tuned
  floor_margin yet).
- isaac_bringup.launch.py: scan_ground_filter's floor_margin raised to 0.07
  for Isaac (Gazebo's 0.4 default untouched), obstacle_markers node so
  RViz can render the scene's collision-only geometry, slam_toolbox_isaac
  .yaml with occupancy_threshold raised to 0.7 so the residual ghost rate
  stops baking into /map's static_layer permanently.
- select_nav2_params.py: Humble/Jazzy Nav2 param and BT xml selection.
- nav2_params.yaml, integration.rviz: footprint re-derivation for the
  recentered base_link, obstacle_markers display.

Root cause of the ghost scans: this gait's asymmetric leg-phase offsets
produce a persistent, direction-biased lean while walking straight, which
scan_ground_filter's single-IMU-sample-per-scan design doesn't fully
correct for on the more-tilted side. Measured and verified with
scripts/measure_scan.py plus a geometric reprojection of surviving points
against known obstacle positions, not just eyeballed. Not fully resolved;
still investigating.

Co-Authored-By: Claude Sonnet 5 <noreply@anthropic.com>
Claude-Session: https://claude.ai/code/session_016ve9vrsGykjRBYxkCx6Xt9

File: big_bertha_description/urdf/big_bertha.urdf.xacro (robot description, xacro)
@@ -8,4 +8,38 @@
   older bringup-specific geometry (which had its own joint origins and a
   hand-tuned lidar height/position from an earlier, now-superseded URDF).
+  Refreshed 2026-08-28 against a newer hardware-revision CAD export
+  (big_bertha_description/urdf/Spyder_mg995_description.urdf, no _v2 suffix,
+  a raw, non-xacro URDF dump, base_link-relative coordinates only, no
+  ros2_control/gazebo scaffolding). base_link now uses that export's raw CAD
+  origin directly, verified as the true geometric center of the chassis: the
+  4 leg-mount points on both the bottom and top perforated plates average to
+  (0,0) in this frame to within 1e-4 m. An earlier pass at this transfer
+  preserved an inherited offset from the older xacro (+0.06489606,
+  -0.06499993 relative to this frame) under the mistaken assumption that
+  matching nav2_params.yaml's already-tuned footprint polygon meant that
+  offset was the correct/centered choice, it wasn't actually centered, it
+  was just wherever one CAD sub-part's own local mesh origin happened to
+  land. Corrected: base_link, the 4 hip joints, battery_joint, and imu_joint
+  (a bringup-synthetic frame with no CAD source of its own, but still
+  base_link-relative so it moves too) all use the raw/true-centered frame
+  now; nav2_params.yaml's footprint polygon has been re-derived into this
+  frame to match (see that file's own note). The actual hardware delta the
+  new export carries is real: a bigger/heavier battery (0.18kg
+  0.107x0.035x0.025m to 0.5kg 0.1083x0.07745x0.047m), which pushed
+  circuit_box_base_joint's mount point down accordingly, plus small
+  CAD-refinement updates to circuit_box_link's inertia and the MPU_9265
+  chip's mesh placement. Joint topology (names, parent/child, axes, limits)
+  is unchanged, so ros2_control.yaml's joint list and ordering remain valid
+  untouched.
+  arm_c_2_1/arm_c_3_1 (2026-08-28, later same day): the CAD export gave
+  these two links different inertia despite both using arm_c_left.stl,
+  the same physical part as each other, mounted at different corners. That
+  has no legitimate hardware explanation and matched a transcription-
+  artifact pattern already diagnosed once before on a different branch
+  (see memory: project_sim2sim_walking_regression), confirmed here too by
+  an A/B test (symmetrizing cut an 8s straight-walk yaw veer from +0.043
+  rad to +0.015 rad). Re-symmetrized to the arithmetic mean of the two CAD
+  readings (no independent/training reference was available to pick one
+  as correct), see each link's own inertial comment.
   Augmented with:
     - a gz_ros2_control system plugin,
@@ -44,12 +78,23 @@
   <xacro:property name="mesh_pkg" value="package://big_bertha_description/meshes"/>
   <!-- ============================== Links ============================== -->
+  <!-- base_link origin is the raw CAD origin from Spyder_mg995_description.urdf
+       (the 2026-08-28 hardware CAD refresh), verified as the true geometric
+       center of the chassis: the 4 leg-mount points on both the bottom and
+       top perforated plates average to (0,0) in this frame to within 1e-4 m.
+       An earlier pass at this transfer preserved an inherited offset from
+       the older xacro (+0.06489606, -0.06499993 relative to this frame)
+       under the mistaken assumption that "already matches nav2's footprint
+       tuning" meant "correct/centered", it wasn't actually centered, it
+       was just wherever one CAD sub-part's own local mesh origin happened to
+       land. Corrected here; nav2_params.yaml's footprint polygon has been
+       re-derived into this frame to match (see that file). -->
   <link name="base_link">
     <inertial>
-      <origin xyz="0.06489606 -0.06499993 0.02039469" rpy="0 0 0"/>
+      <origin xyz="0 0 0.02039469" rpy="0 0 0"/>
       <mass value="0.263885"/>
       <inertia ixx="0.00116595" ixy="-0.00000226" ixz="0.00000001" iyy="0.00116867" iyz="0.00000004" izz="0.00226074"/>
     </inertial>
     <visual>
-      <origin xyz="0 -0 0.005" rpy="3.140796 -0 0"/>
+      <origin xyz="-0.06489606 0.06499993 0.005" rpy="3.140796 -0 0"/>
       <geometry>
         <mesh filename="${mesh_pkg}/central_perforated_plate.stl" scale="0.001 0.001 0.001"/>
@@ -58,5 +103,5 @@
     </visual>
     <collision>
-      <origin xyz="0 -0 0.005" rpy="3.140796 -0 0"/>
+      <origin xyz="-0.06489606 0.06499993 0.005" rpy="3.140796 -0 0"/>
       <geometry>
         <mesh filename="${mesh_pkg}/central_perforated_plate.stl" scale="0.001 0.001 0.001"/>
@@ -64,5 +109,5 @@
     </collision>
     <visual>
-      <origin xyz="0 -0 0.035" rpy="3.140796 -0 0"/>
+      <origin xyz="-0.06489606 0.06499993 0.035" rpy="3.140796 -0 0"/>
       <geometry>
         <mesh filename="${mesh_pkg}/central_perforated_plate.stl" scale="0.001 0.001 0.001"/>
@@ -71,5 +116,5 @@
     </visual>
     <collision>
-      <origin xyz="0 -0 0.035" rpy="3.140796 -0 0"/>
+      <origin xyz="-0.06489606 0.06499993 0.035" rpy="3.140796 -0 0"/>
       <geometry>
         <mesh filename="${mesh_pkg}/central_perforated_plate.stl" scale="0.001 0.001 0.001"/>
@@ -77,57 +122,57 @@
     </collision>
     <visual>
-      <origin xyz="0.001 -0.061 0.03" rpy="3.140796 -0 0"/>
-      <geometry>
-        <mesh filename="${mesh_pkg}/body_standoffs.stl" scale="0.001 0.001 0.001"/>
-      </geometry>
-      <material name="silver"/>
-    </visual>
-    <collision>
-      <origin xyz="0.001 -0.061 0.03" rpy="3.140796 -0 0"/>
-      <geometry>
-        <mesh filename="${mesh_pkg}/body_standoffs.stl" scale="0.001 0.001 0.001"/>
-      </geometry>
-    </collision>
-    <visual>
-      <origin xyz="0.069 -0.001 0.03" rpy="3.140796 -0 -1.57"/>
-      <geometry>
-        <mesh filename="${mesh_pkg}/body_standoffs.stl" scale="0.001 0.001 0.001"/>
-      </geometry>
-      <material name="silver"/>
-    </visual>
-    <collision>
-      <origin xyz="0.069 -0.001 0.03" rpy="3.140796 -0 -1.57"/>
-      <geometry>
-        <mesh filename="${mesh_pkg}/body_standoffs.stl" scale="0.001 0.001 0.001"/>
-      </geometry>
-    </collision>
-    <visual>
-      <origin xyz="0.127 -0.069 0.03" rpy="3.140796 -0 3.14"/>
-      <geometry>
-        <mesh filename="${mesh_pkg}/body_standoffs.stl" scale="0.001 0.001 0.001"/>
-      </geometry>
-      <material name="silver"/>
-    </visual>
-    <collision>
-      <origin xyz="0.127 -0.069 0.03" rpy="3.140796 -0 3.14"/>
-      <geometry>
-        <mesh filename="${mesh_pkg}/body_standoffs.stl" scale="0.001 0.001 0.001"/>
-      </geometry>
-    </collision>
-    <visual>
-      <origin xyz="0.068 -0.127 0.03" rpy="3.140796 -0 1.57"/>
-      <geometry>
-        <mesh filename="${mesh_pkg}/body_standoffs.stl" scale="0.001 0.001 0.001"/>
-      </geometry>
-      <material name="silver"/>
-    </visual>
-    <collision>
-      <origin xyz="0.068 -0.127 0.03" rpy="3.140796 -0 1.57"/>
-      <geometry>
-        <mesh filename="${mesh_pkg}/body_standoffs.stl" scale="0.001 0.001 0.001"/>
-      </geometry>
-    </collision>
-    <visual>
-      <origin xyz="0.0325 0.007 0" rpy="3.140796 -0 -1.57"/>
+      <origin xyz="-0.06389606 0.00399993 0.03" rpy="3.140796 -0 0"/>
+      <geometry>
+        <mesh filename="${mesh_pkg}/body_standoffs.stl" scale="0.001 0.001 0.001"/>
+      </geometry>
+      <material name="silver"/>
+    </visual>
+    <collision>
+      <origin xyz="-0.06389606 0.00399993 0.03" rpy="3.140796 -0 0"/>
+      <geometry>
+        <mesh filename="${mesh_pkg}/body_standoffs.stl" scale="0.001 0.001 0.001"/>
+      </geometry>
+    </collision>
+    <visual>
+      <origin xyz="0.00410394 0.06399993 0.03" rpy="3.140796 -0 -1.57"/>
+      <geometry>
+        <mesh filename="${mesh_pkg}/body_standoffs.stl" scale="0.001 0.001 0.001"/>
+      </geometry>
+      <material name="silver"/>
+    </visual>
+    <collision>
+      <origin xyz="0.00410394 0.06399993 0.03" rpy="3.140796 -0 -1.57"/>
+      <geometry>
+        <mesh filename="${mesh_pkg}/body_standoffs.stl" scale="0.001 0.001 0.001"/>
+      </geometry>
+    </collision>
+    <visual>
+      <origin xyz="0.06210394 -0.00400007 0.03" rpy="3.140796 -0 3.14"/>
+      <geometry>
+        <mesh filename="${mesh_pkg}/body_standoffs.stl" scale="0.001 0.001 0.001"/>
+      </geometry>
+      <material name="silver"/>
+    </visual>
+    <collision>
+      <origin xyz="0.06210394 -0.00400007 0.03" rpy="3.140796 -0 3.14"/>
+      <geometry>
+        <mesh filename="${mesh_pkg}/body_standoffs.stl" scale="0.001 0.001 0.001"/>
+      </geometry>
+    </collision>
+    <visual>
+      <origin xyz="0.00310394 -0.06200007 0.03" rpy="3.140796 -0 1.57"/>
+      <geometry>
+        <mesh filename="${mesh_pkg}/body_standoffs.stl" scale="0.001 0.001 0.001"/>
+      </geometry>
+      <material name="silver"/>
+    </visual>
+    <collision>
+      <origin xyz="0.00310394 -0.06200007 0.03" rpy="3.140796 -0 1.57"/>
+      <geometry>
+        <mesh filename="${mesh_pkg}/body_standoffs.stl" scale="0.001 0.001 0.001"/>
+      </geometry>
+    </collision>
+    <visual>
+      <origin xyz="-0.03239606 0.07199993 0" rpy="3.140796 -0 -1.57"/>
       <geometry>
         <mesh filename="${mesh_pkg}/arm_perforated_plate_bottom.stl" scale="0.001 0.001 0.001"/>
@@ -136,5 +181,5 @@
     </visual>
     <collision>
-      <origin xyz="0.0325 0.007 0" rpy="3.140796 -0 -1.57"/>
+      <origin xyz="-0.03239606 0.07199993 0" rpy="3.140796 -0 -1.57"/>
       <geometry>
         <mesh filename="${mesh_pkg}/arm_perforated_plate_bottom.stl" scale="0.001 0.001 0.001"/>
@@ -142,5 +187,5 @@
     </collision>
     <visual>
-      <origin xyz="0.137 -0.032 0" rpy="3.140796 -0 3.14"/>
+      <origin xyz="0.07210394 0.03299993 0" rpy="3.140796 -0 3.14"/>
       <geometry>
         <mesh filename="${mesh_pkg}/arm_perforated_plate_bottom.stl" scale="0.001 0.001 0.001"/>
@@ -149,5 +194,5 @@
     </visual>
     <collision>
-      <origin xyz="0.137 -0.032 0" rpy="3.140796 -0 3.14"/>
+      <origin xyz="0.07210394 0.03299993 0" rpy="3.140796 -0 3.14"/>
       <geometry>
         <mesh filename="${mesh_pkg}/arm_perforated_plate_bottom.stl" scale="0.001 0.001 0.001"/>
@@ -155,5 +200,5 @@
     </collision>
     <visual>
-      <origin xyz="-0.007 -0.098 0" rpy="3.140796 -0 0"/>
+      <origin xyz="-0.07189606 -0.03300007 0" rpy="3.140796 -0 0"/>
       <geometry>
         <mesh filename="${mesh_pkg}/arm_perforated_plate_bottom.stl" scale="0.001 0.001 0.001"/>
@@ -162,5 +207,5 @@
     </visual>
     <collision>
-      <origin xyz="-0.007 -0.098 0" rpy="3.140796 -0 0"/>
+      <origin xyz="-0.07189606 -0.03300007 0" rpy="3.140796 -0 0"/>
       <geometry>
         <mesh filename="${mesh_pkg}/arm_perforated_plate_bottom.stl" scale="0.001 0.001 0.001"/>
@@ -168,5 +213,5 @@
     </collision>
     <visual>
-      <origin xyz="0.097 -0.137 0" rpy="3.140796 -0 1.57"/>
+      <origin xyz="0.03210394 -0.07200007 0" rpy="3.140796 -0 1.57"/>
       <geometry>
         <mesh filename="${mesh_pkg}/arm_perforated_plate_bottom.stl" scale="0.001 0.001 0.001"/>
@@ -175,5 +220,5 @@
     </visual>
     <collision>
-      <origin xyz="0.097 -0.137 0" rpy="3.140796 -0 1.57"/>
+      <origin xyz="0.03210394 -0.07200007 0" rpy="3.140796 -0 1.57"/>
       <geometry>
         <mesh filename="${mesh_pkg}/arm_perforated_plate_bottom.stl" scale="0.001 0.001 0.001"/>
@@ -181,5 +226,5 @@
     </collision>
     <visual>
-      <origin xyz="0.155 -0.078 0.03" rpy="3.140796 -0 -1.57"/>
+      <origin xyz="0.09010394 -0.01300007 0.03" rpy="3.140796 -0 -1.57"/>
       <geometry>
         <mesh filename="${mesh_pkg}/arm_perforated_plate_top.stl" scale="0.001 0.001 0.001"/>
@@ -188,5 +233,5 @@
     </visual>
     <collision>
-      <origin xyz="0.155 -0.078 0.03" rpy="3.140796 -0 -1.57"/>
+      <origin xyz="0.09010394 -0.01300007 0.03" rpy="3.140796 -0 -1.57"/>
       <geometry>
         <mesh filename="${mesh_pkg}/arm_perforated_plate_top.stl" scale="0.001 0.001 0.001"/>
@@ -194,5 +239,5 @@
     </collision>
     <visual>
-      <origin xyz="0.052 -0.155 0.03" rpy="3.140796 -0 -3.14"/>
+      <origin xyz="-0.01289606 -0.09000007 0.03" rpy="3.140796 -0 -3.14"/>
       <geometry>
         <mesh filename="${mesh_pkg}/arm_perforated_plate_top.stl" scale="0.001 0.001 0.001"/>
@@ -201,5 +246,5 @@
     </visual>
     <collision>
-      <origin xyz="0.052 -0.155 0.03" rpy="3.140796 -0 -3.14"/>
+      <origin xyz="-0.01289606 -0.09000007 0.03" rpy="3.140796 -0 -3.14"/>
       <geometry>
         <mesh filename="${mesh_pkg}/arm_perforated_plate_top.stl" scale="0.001 0.001 0.001"/>
@@ -207,5 +252,5 @@
     </collision>
     <visual>
-      <origin xyz="0.078 0.025 0.03" rpy="3.140796 -0 0"/>
+      <origin xyz="0.01310394 0.08999993 0.03" rpy="3.140796 -0 0"/>
       <geometry>
         <mesh filename="${mesh_pkg}/arm_perforated_plate_top.stl" scale="0.001 0.001 0.001"/>
@@ -214,5 +259,5 @@
     </visual>
     <collision>
-      <origin xyz="0.078 0.025 0.03" rpy="3.140796 -0 0"/>
+      <origin xyz="0.01310394 0.08999993 0.03" rpy="3.140796 -0 0"/>
       <geometry>
         <mesh filename="${mesh_pkg}/arm_perforated_plate_top.stl" scale="0.001 0.001 0.001"/>
@@ -220,5 +265,5 @@
     </collision>
     <visual>
-      <origin xyz="-0.025 -0.052 0.03" rpy="3.140796 -0 1.57"/>
+      <origin xyz="-0.08989606 0.01299993 0.03" rpy="3.140796 -0 1.57"/>
       <geometry>
         <mesh filename="${mesh_pkg}/arm_perforated_plate_top.stl" scale="0.001 0.001 0.001"/>
@@ -227,5 +272,5 @@
     </visual>
     <collision>
-      <origin xyz="-0.025 -0.052 0.03" rpy="3.140796 -0 1.57"/>
+      <origin xyz="-0.08989606 0.01299993 0.03" rpy="3.140796 -0 1.57"/>
       <geometry>
         <mesh filename="${mesh_pkg}/arm_perforated_plate_top.stl" scale="0.001 0.001 0.001"/>
@@ -233,51 +278,51 @@
     </collision>
     <visual>
-      <origin xyz="-0.015 -0.0115 0.002" rpy="0.0007963268 -0 0"/>
-      <geometry>
-        <mesh filename="${mesh_pkg}/servo_mg995.stl" scale="0.001 0.001 0.001"/>
-      </geometry>
-      <material name="silver"/>
-    </visual>
-    <collision>
-      <origin xyz="-0.015 -0.0115 0.002" rpy="0.0007963268 -0 0"/>
-      <geometry>
-        <mesh filename="${mesh_pkg}/servo_mg995.stl" scale="0.001 0.001 0.001"/>
-      </geometry>
-    </collision>
-    <visual>
-      <origin xyz="0.011 -0.145 0.002" rpy="0.0007963268 -0 1.57"/>
-      <geometry>
-        <mesh filename="${mesh_pkg}/servo_mg995.stl" scale="0.001 0.001 0.001"/>
-      </geometry>
-      <material name="silver"/>
-    </visual>
-    <collision>
-      <origin xyz="0.011 -0.145 0.002" rpy="0.0007963268 -0 1.57"/>
-      <geometry>
-        <mesh filename="${mesh_pkg}/servo_mg995.stl" scale="0.001 0.001 0.001"/>
-      </geometry>
-    </collision>
-    <visual>
-      <origin xyz="0.145 -0.1185 0.002" rpy="0.0007963268 -0 -3.14"/>
-      <geometry>
-        <mesh filename="${mesh_pkg}/servo_mg995.stl" scale="0.001 0.001 0.001"/>
-      </geometry>
-      <material name="silver"/>
-    </visual>
-    <collision>
-      <origin xyz="0.145 -0.1185 0.002" rpy="0.0007963268 -0 -3.14"/>
-      <geometry>
-        <mesh filename="${mesh_pkg}/servo_mg995.stl" scale="0.001 0.001 0.001"/>
-      </geometry>
-    </collision>
-    <visual>
-      <origin xyz="0.1185 0.015 0.002" rpy="0.0007963268 -0 -1.57"/>
-      <geometry>
-        <mesh filename="${mesh_pkg}/servo_mg995.stl" scale="0.001 0.001 0.001"/>
-      </geometry>
-      <material name="silver"/>
-    </visual>
-    <collision>
-      <origin xyz="0.1185 0.015 0.002" rpy="0.0007963268 -0 -1.57"/>
+      <origin xyz="-0.07989606 0.05349993 0.002" rpy="0.0007963268 -0 0"/>
+      <geometry>
+        <mesh filename="${mesh_pkg}/servo_mg995.stl" scale="0.001 0.001 0.001"/>
+      </geometry>
+      <material name="silver"/>
+    </visual>
+    <collision>
+      <origin xyz="-0.07989606 0.05349993 0.002" rpy="0.0007963268 -0 0"/>
+      <geometry>
+        <mesh filename="${mesh_pkg}/servo_mg995.stl" scale="0.001 0.001 0.001"/>
+      </geometry>
+    </collision>
+    <visual>
+      <origin xyz="-0.05389606 -0.08000007 0.002" rpy="0.0007963268 -0 1.57"/>
+      <geometry>
+        <mesh filename="${mesh_pkg}/servo_mg995.stl" scale="0.001 0.001 0.001"/>
+      </geometry>
+      <material name="silver"/>
+    </visual>
+    <collision>
+      <origin xyz="-0.05389606 -0.08000007 0.002" rpy="0.0007963268 -0 1.57"/>
+      <geometry>
+        <mesh filename="${mesh_pkg}/servo_mg995.stl" scale="0.001 0.001 0.001"/>
+      </geometry>
+    </collision>
+    <visual>
+      <origin xyz="0.08010394 -0.05350007 0.002" rpy="0.0007963268 -0 -3.14"/>
+      <geometry>
+        <mesh filename="${mesh_pkg}/servo_mg995.stl" scale="0.001 0.001 0.001"/>
+      </geometry>
+      <material name="silver"/>
+    </visual>
+    <collision>
+      <origin xyz="0.08010394 -0.05350007 0.002" rpy="0.0007963268 -0 -3.14"/>
+      <geometry>
+        <mesh filename="${mesh_pkg}/servo_mg995.stl" scale="0.001 0.001 0.001"/>
+      </geometry>
+    </collision>
+    <visual>
+      <origin xyz="0.05360394 0.07999993 0.002" rpy="0.0007963268 -0 -1.57"/>
+      <geometry>
+        <mesh filename="${mesh_pkg}/servo_mg995.stl" scale="0.001 0.001 0.001"/>
+      </geometry>
+      <material name="silver"/>
+    </visual>
+    <collision>
+      <origin xyz="0.05360394 0.07999993 0.002" rpy="0.0007963268 -0 -1.57"/>
       <geometry>
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