Commit message: fix(imu): correct 180 flipped MPU6050 orientation

File: big_bertha_description/urdf/big_bertha.urdf.xacro (robot description, xacro)
@@ -458,5 +458,5 @@
   </joint>
   <joint name="imu_joint" type="fixed">
-    <origin xyz="0.0 0.0 0.01" rpy="0 0 0"/>
+    <origin xyz="0.0 0.0 0.01" rpy="0 0 3.141592653589793"/>
     <parent link="base_link"/>
     <child link="imu_link"/>

Commit message: fix: HUD panel and urdf joint limits

File: big_bertha_description/urdf/big_bertha.urdf.xacro (robot description, xacro)
@@ -634,5 +634,5 @@
     <child link="arm_a_4_1"/>
     <axis xyz="0 1.0 0"/>
-    <limit lower="-1.57" upper="1.57"/>
+    <limit lower="-1.57" upper="1.57" effort="1.0" velocity="6.28"/>
     <dynamics damping="0.02" friction="0.0"/>
   </joint>
@@ -642,5 +642,5 @@
     <child link="arm_b_4_1"/>
     <axis xyz="0 1.0 0"/>
-    <limit lower="-1.57" upper="0.96"/>
+    <limit lower="-1.57" upper="0.96" effort="1.0" velocity="6.28"/>
     <dynamics damping="0.02" friction="0.0"/>
   </joint>
@@ -650,5 +650,5 @@
     <child link="arm_c_4_1"/>
     <axis xyz="0 0 1"/>
-    <limit lower="0" upper="2.355"/>
+    <limit lower="0" upper="2.355" effort="1.0" velocity="6.28"/>
     <dynamics damping="0.02" friction="0.0"/>
   </joint>
@@ -659,5 +659,5 @@
     <child link="arm_a_1_1"/>
     <axis xyz="0 1.0 0"/>
-    <limit lower="-1.57" upper="1.57"/>
+    <limit lower="-1.57" upper="1.57" effort="1.0" velocity="6.28"/>
     <dynamics damping="0.02" friction="0.0"/>
   </joint>
@@ -667,5 +667,5 @@
     <child link="arm_b_1_1"/>
     <axis xyz="0 1.0 0"/>
-    <limit lower="-1.57" upper="0.96"/>
+    <limit lower="-1.57" upper="0.96" effort="1.0" velocity="6.28"/>
     <dynamics damping="0.02" friction="0.0"/>
   </joint>
@@ -675,5 +675,5 @@
     <child link="arm_c_1_1"/>
     <axis xyz="0 0 1"/>
-    <limit lower="0" upper="2.355"/>
+    <limit lower="0" upper="2.355" effort="1.0" velocity="6.28"/>
     <dynamics damping="0.02" friction="0.0"/>
   </joint>
@@ -684,5 +684,5 @@
     <child link="arm_a_2_1"/>
     <axis xyz="0 1.0 0"/>
-    <limit lower="-1.57" upper="1.57"/>
+    <limit lower="-1.57" upper="1.57" effort="1.0" velocity="6.28"/>
     <dynamics damping="0.02" friction="0.0"/>
   </joint>
@@ -692,5 +692,5 @@
     <child link="arm_b_2_1"/>
     <axis xyz="0 1.0 0"/>
-    <limit lower="-1.57" upper="0.96"/>
+    <limit lower="-1.57" upper="0.96" effort="1.0" velocity="6.28"/>
     <dynamics damping="0.02" friction="0.0"/>
   </joint>
@@ -700,5 +700,5 @@
     <child link="arm_c_2_1"/>
     <axis xyz="0 0 1"/>
-    <limit lower="0" upper="2.355"/>
+    <limit lower="0" upper="2.355" effort="1.0" velocity="6.28"/>
     <dynamics damping="0.02" friction="0.0"/>
   </joint>
@@ -709,5 +709,5 @@
     <child link="arm_a_3_1"/>
     <axis xyz="0 1.0 0"/>
-    <limit lower="-1.57" upper="1.57"/>
+    <limit lower="-1.57" upper="1.57" effort="1.0" velocity="6.28"/>
     <dynamics damping="0.02" friction="0.0"/>
   </joint>
@@ -717,5 +717,5 @@
     <child link="arm_b_3_1"/>
     <axis xyz="0 1.0 0"/>
-    <limit lower="-1.57" upper="0.96"/>
+    <limit lower="-1.57" upper="0.96" effort="1.0" velocity="6.28"/>
     <dynamics damping="0.02" friction="0.0"/>
   </joint>
@@ -725,5 +725,5 @@
     <child link="arm_c_3_1"/>
     <axis xyz="0 0 1"/>
-    <limit lower="0" upper="2.355"/>
+    <limit lower="0" upper="2.355" effort="1.0" velocity="6.28"/>
     <dynamics damping="0.02" friction="0.0"/>
   </joint>

Commit message: fix: trying to fix big_bertha_description

File: big_bertha_description/urdf/big_bertha.urdf.xacro (robot description, xacro)
@@ -36,4 +36,166 @@
   <!-- ============================== Links ============================== -->
   <link name="base_link">
+    <visual>
+      <origin xyz="0 0 0.005" rpy="3.140796 0 0"/>
+      <geometry><mesh filename="${mesh_pkg}/central_perforated_plate.stl" scale="0.001 0.001 0.001"/></geometry>
+      <material name="silver"/>
+    </visual>
+    <collision>
+      <origin xyz="0 0 0.005" rpy="3.140796 0 0"/>
+      <geometry><mesh filename="${mesh_pkg}/central_perforated_plate.stl" scale="0.001 0.001 0.001"/></geometry>
+    </collision>
+    <visual>
+      <origin xyz="0 0 0.035" rpy="3.140796 0 0"/>
+      <geometry><mesh filename="${mesh_pkg}/central_perforated_plate.stl" scale="0.001 0.001 0.001"/></geometry>
+      <material name="silver"/>
+    </visual>
+    <collision>
+      <origin xyz="0 0 0.035" rpy="3.140796 0 0"/>
+      <geometry><mesh filename="${mesh_pkg}/central_perforated_plate.stl" scale="0.001 0.001 0.001"/></geometry>
+    </collision>
+    <visual>
+      <origin xyz="0.001 -0.061 0.03" rpy="3.140796 0 0"/>
+      <geometry><mesh filename="${mesh_pkg}/body_standoffs.stl" scale="0.001 0.001 0.001"/></geometry>
+      <material name="silver"/>
+    </visual>
+    <collision>
+      <origin xyz="0.001 -0.061 0.03" rpy="3.140796 0 0"/>
+      <geometry><mesh filename="${mesh_pkg}/body_standoffs.stl" scale="0.001 0.001 0.001"/></geometry>
+    </collision>
+    <visual>
+      <origin xyz="0.069 -0.001 0.03" rpy="3.140796 0 -1.57"/>
+      <geometry><mesh filename="${mesh_pkg}/body_standoffs.stl" scale="0.001 0.001 0.001"/></geometry>
+      <material name="silver"/>
+    </visual>
+    <collision>
+      <origin xyz="0.069 -0.001 0.03" rpy="3.140796 0 -1.57"/>
+      <geometry><mesh filename="${mesh_pkg}/body_standoffs.stl" scale="0.001 0.001 0.001"/></geometry>
+    </collision>
+    <visual>
+      <origin xyz="0.127 -0.069 0.03" rpy="3.140796 0 3.14"/>
+      <geometry><mesh filename="${mesh_pkg}/body_standoffs.stl" scale="0.001 0.001 0.001"/></geometry>
+      <material name="silver"/>
+    </visual>
+    <collision>
+      <origin xyz="0.127 -0.069 0.03" rpy="3.140796 0 3.14"/>
+      <geometry><mesh filename="${mesh_pkg}/body_standoffs.stl" scale="0.001 0.001 0.001"/></geometry>
+    </collision>
+    <visual>
+      <origin xyz="0.068 -0.127 0.03" rpy="3.140796 0 1.57"/>
+      <geometry><mesh filename="${mesh_pkg}/body_standoffs.stl" scale="0.001 0.001 0.001"/></geometry>
+      <material name="silver"/>
+    </visual>
+    <collision>
+      <origin xyz="0.068 -0.127 0.03" rpy="3.140796 0 1.57"/>
+      <geometry><mesh filename="${mesh_pkg}/body_standoffs.stl" scale="0.001 0.001 0.001"/></geometry>
+    </collision>
+    <visual>
+      <origin xyz="0.0325 0.007 0" rpy="3.140796 0 -1.57"/>
+      <geometry><mesh filename="${mesh_pkg}/arm_perforated_plate_bottom.stl" scale="0.001 0.001 0.001"/></geometry>
+      <material name="silver"/>
+    </visual>
+    <collision>
+      <origin xyz="0.0325 0.007 0" rpy="3.140796 0 -1.57"/>
+      <geometry><mesh filename="${mesh_pkg}/arm_perforated_plate_bottom.stl" scale="0.001 0.001 0.001"/></geometry>
+    </collision>
+    <visual>
+      <origin xyz="0.137 -0.032 0" rpy="3.140796 0 3.14"/>
+      <geometry><mesh filename="${mesh_pkg}/arm_perforated_plate_bottom.stl" scale="0.001 0.001 0.001"/></geometry>
+      <material name="silver"/>
+    </visual>
+    <collision>
+      <origin xyz="0.137 -0.032 0" rpy="3.140796 0 3.14"/>
+      <geometry><mesh filename="${mesh_pkg}/arm_perforated_plate_bottom.stl" scale="0.001 0.001 0.001"/></geometry>
+    </collision>
+    <visual>
+      <origin xyz="-0.007 -0.098 0" rpy="3.140796 0 0"/>
+      <geometry><mesh filename="${mesh_pkg}/arm_perforated_plate_bottom.stl" scale="0.001 0.001 0.001"/></geometry>
+      <material name="silver"/>
+    </visual>
+    <collision>
+      <origin xyz="-0.007 -0.098 0" rpy="3.140796 0 0"/>
+      <geometry><mesh filename="${mesh_pkg}/arm_perforated_plate_bottom.stl" scale="0.001 0.001 0.001"/></geometry>
+    </collision>
+    <visual>
+      <origin xyz="0.097 -0.137 0" rpy="3.140796 0 1.57"/>
+      <geometry><mesh filename="${mesh_pkg}/arm_perforated_plate_bottom.stl" scale="0.001 0.001 0.001"/></geometry>
+      <material name="silver"/>
+    </visual>
+    <collision>
+      <origin xyz="0.097 -0.137 0" rpy="3.140796 0 1.57"/>
+      <geometry><mesh filename="${mesh_pkg}/arm_perforated_plate_bottom.stl" scale="0.001 0.001 0.001"/></geometry>
+    </collision>
+    <visual>
+      <origin xyz="0.155 -0.078 0.03" rpy="3.140796 0 -1.57"/>
+      <geometry><mesh filename="${mesh_pkg}/arm_perforated_plate_top.stl" scale="0.001 0.001 0.001"/></geometry>
+      <material name="silver"/>
+    </visual>
+    <collision>
+      <origin xyz="0.155 -0.078 0.03" rpy="3.140796 0 -1.57"/>
+      <geometry><mesh filename="${mesh_pkg}/arm_perforated_plate_top.stl" scale="0.001 0.001 0.001"/></geometry>
+    </collision>
+    <visual>
+      <origin xyz="0.052 -0.155 0.03" rpy="3.140796 0 -3.14"/>
+      <geometry><mesh filename="${mesh_pkg}/arm_perforated_plate_top.stl" scale="0.001 0.001 0.001"/></geometry>
+      <material name="silver"/>
+    </visual>
+    <collision>
+      <origin xyz="0.052 -0.155 0.03" rpy="3.140796 0 -3.14"/>
+      <geometry><mesh filename="${mesh_pkg}/arm_perforated_plate_top.stl" scale="0.001 0.001 0.001"/></geometry>
+    </collision>
+    <visual>
+      <origin xyz="0.078 0.025 0.03" rpy="3.140796 0 0"/>
+      <geometry><mesh filename="${mesh_pkg}/arm_perforated_plate_top.stl" scale="0.001 0.001 0.001"/></geometry>
+      <material name="silver"/>
+    </visual>
+    <collision>
+      <origin xyz="0.078 0.025 0.03" rpy="3.140796 0 0"/>
+      <geometry><mesh filename="${mesh_pkg}/arm_perforated_plate_top.stl" scale="0.001 0.001 0.001"/></geometry>
+    </collision>
+    <visual>
+      <origin xyz="-0.025 -0.052 0.03" rpy="3.140796 0 1.57"/>
+      <geometry><mesh filename="${mesh_pkg}/arm_perforated_plate_top.stl" scale="0.001 0.001 0.001"/></geometry>
+      <material name="silver"/>
+    </visual>
+    <collision>
+      <origin xyz="-0.025 -0.052 0.03" rpy="3.140796 0 1.57"/>
+      <geometry><mesh filename="${mesh_pkg}/arm_perforated_plate_top.stl" scale="0.001 0.001 0.001"/></geometry>
+    </collision>
+    <visual>
+      <origin xyz="-0.015 -0.0115 0.002" rpy="0.0007963268 0 0"/>
+      <geometry><mesh filename="${mesh_pkg}/servo_mg995.stl" scale="0.001 0.001 0.001"/></geometry>
+      <material name="silver"/>
+    </visual>
+    <collision>
+      <origin xyz="-0.015 -0.0115 0.002" rpy="0.0007963268 0 0"/>
+      <geometry><mesh filename="${mesh_pkg}/servo_mg995.stl" scale="0.001 0.001 0.001"/></geometry>
+    </collision>
+    <visual>
+      <origin xyz="0.011 -0.145 0.002" rpy="0.0007963268 0 1.57"/>
+      <geometry><mesh filename="${mesh_pkg}/servo_mg995.stl" scale="0.001 0.001 0.001"/></geometry>
+      <material name="silver"/>
+    </visual>
+    <collision>
+      <origin xyz="0.011 -0.145 0.002" rpy="0.0007963268 0 1.57"/>
+      <geometry><mesh filename="${mesh_pkg}/servo_mg995.stl" scale="0.001 0.001 0.001"/></geometry>
+    </collision>
+    <visual>
+      <origin xyz="0.145 -0.1185 0.002" rpy="0.0007963268 0 -3.14"/>
+      <geometry><mesh filename="${mesh_pkg}/servo_mg995.stl" scale="0.001 0.001 0.001"/></geometry>
+      <material name="silver"/>
+    </visual>
+    <collision>
+      <origin xyz="0.145 -0.1185 0.002" rpy="0.0007963268 0 -3.14"/>
+      <geometry><mesh filename="${mesh_pkg}/servo_mg995.stl" scale="0.001 0.001 0.001"/></geometry>
+    </collision>
+    <visual>
+      <origin xyz="0.1185 0.015 0.002" rpy="0.0007963268 0 -1.57"/>
+      <geometry><mesh filename="${mesh_pkg}/servo_mg995.stl" scale="0.001 0.001 0.001"/></geometry>
+      <material name="silver"/>
+    </visual>
+    <collision>
+      <origin xyz="0.1185 0.015 0.002" rpy="0.0007963268 0 -1.57"/>
+      <geometry><mesh filename="${mesh_pkg}/servo_mg995.stl" scale="0.001 0.001 0.001"/></geometry>
+    </collision>
     <inertial>
       <origin xyz="0.06489606 -0.06499993 0.02039469" rpy="0 0 0"/>
@@ -534,6 +696,6 @@
   <link name="imu_link">
     <inertial>
+      <mass value="0.001"/>
       <origin xyz="0 0 0" rpy="0 0 0"/>
-      <mass value="0.001"/>
       <inertia ixx="1e-06" iyy="1e-06" izz="1e-06" ixy="0" ixz="0" iyz="0"/>
     </inertial>
@@ -545,4 +707,13 @@
   </link>
   <link name="battery_link">
+    <visual>
+      <origin xyz="0 0 0.0105" rpy="0 0 0"/>
+      <geometry><box size="0.107 0.035 0.025"/></geometry>
+      <material name="silver"/>
+    </visual>
+    <collision>
+      <origin xyz="0 0 0.0105" rpy="0 0 0"/>
+      <geometry><box size="0.107 0.035 0.025"/></geometry>
+    </collision>
     <inertial>
       <origin xyz="-0.00051903 -0.01742240 -0.04805902" rpy="0 0 0"/>
@@ -646,4 +817,22 @@
   <!-- arm_a_1_1 (front-left, leg 1) -->
   <link name="arm_a_1_1">
+    <visual>
+      <origin xyz="0.025 0.012 0.008" rpy="3.14 0 -1.57"/>
+      <geometry><mesh filename="${mesh_pkg}/arm_a_right.stl" scale="0.001 0.001 0.001"/></geometry>
+      <material name="silver"/>
+    </visual>
+    <collision>
+      <origin xyz="0.025 0.012 0.008" rpy="3.14 0 -1.57"/>
+      <geometry><mesh filename="${mesh_pkg}/arm_a_right.stl" scale="0.001 0.001 0.001"/></geometry>
+    </collision>
+    <visual>
+      <origin xyz="0.0177 -0.0175 -0.0525" rpy="0 -1.57 0"/>
+      <geometry><mesh filename="${mesh_pkg}/servo_mg995.stl" scale="0.001 0.001 0.001"/></geometry>
+      <material name="silver"/>
+    </visual>
+    <collision>
+      <origin xyz="0.0177 -0.0175 -0.0525" rpy="0 -1.57 0"/>
+      <geometry><mesh filename="${mesh_pkg}/servo_mg995.stl" scale="0.001 0.001 0.001"/></geometry>
+    </collision>
     <inertial>
       <origin xyz="-0.00089507 -0.01742240 -0.05050470" rpy="0 0 0"/>
@@ -723,4 +912,8 @@
       <material name="silver"/>
     </visual>
+    <collision>
+      <origin xyz="0.01 -0.145 -0.053" rpy="1.57 0 -3.14"/>
+      <geometry><mesh filename="${mesh_pkg}/arm_c_right.stl" scale="0.001 0.001 0.001"/></geometry>
+    </collision>
     <visual>
       <origin xyz="0 -0.01 -0.045" rpy="0 0 0"/>
@@ -736,7 +929,46 @@
       </geometry>
     </collision>
+    <inertial>
+      <mass value="0.063687"/>
+      <origin xyz="-0.00152686 -0.01416578 -0.02679160" rpy="0 0 0"/>
+      <inertia ixx="0.00003866" ixy="-0.00000290" ixz="-0.00000068" iyy="0.00001100" iyz="-0.00000123" izz="0.00003408"/>
+    </inertial>
+  </link>
+  <link name="arm_b_1_1">
+    <visual>
+      <origin xyz="-0.0085 -0.032 0.011" rpy="3.14 0 1.57"/>
+      <geometry><mesh filename="${mesh_pkg}/arm_b.stl" scale="0.001 0.001 0.001"/></geometry>
+      <material name="silver"/>
+    </visual>
+    <collision>
+      <origin xyz="-0.0085 -0.032 0.011" rpy="3.14 0 1.57"/>
+      <geometry><mesh filename="${mesh_pkg}/arm_b.stl" scale="0.001 0.001 0.001"/></geometry>
+    </collision>
+    <inertial>
+      <mass value="0.008137"/>
+      <origin xyz="0.04154098 -0.00048149 0.00107965" rpy="0 0 0"/>
+      <inertia ixx="0.00000479" ixy="-0.00000000" ixz="-0.00000001" iyy="0.00000378" iyz="0.00000000" izz="0.00000801"/>
+    </inertial>
   </link>
   <!-- arm_a_2_1 (front-right, leg 2) -->
   <link name="arm_a_2_1">
+    <visual>
+      <origin xyz="0.012 0.012 0.01" rpy="3.14 0 -1.57"/>
+      <geometry><mesh filename="${mesh_pkg}/arm_a_left.stl" scale="0.001 0.001 0.001"/></geometry>
+      <material name="silver"/>
+    </visual>
+    <collision>
+      <origin xyz="0.012 0.012 0.01" rpy="3.14 0 -1.57"/>
+      <geometry><mesh filename="${mesh_pkg}/arm_a_left.stl" scale="0.001 0.001 0.001"/></geometry>
+    </collision>
+    <visual>
+      <origin xyz="-0.016 -0.0175 -0.050" rpy="0 1.57 0"/>
+      <geometry><mesh filename="${mesh_pkg}/servo_mg995.stl" scale="0.001 0.001 0.001"/></geometry>
+      <material name="silver"/>
+    </visual>
+    <collision>
+      <origin xyz="-0.016 -0.0175 -0.050" rpy="0 1.57 0"/>
+      <geometry><mesh filename="${mesh_pkg}/servo_mg995.stl" scale="0.001 0.001 0.001"/></geometry>
+    </collision>
     <inertial>
       <origin xyz="0.00261850 -0.01742175 -0.04806032" rpy="0 0 0"/>
@@ -807,4 +1039,8 @@
       <material name="silver"/>
     </visual>
+    <collision>
+      <origin xyz="0.012 -0.1455 -0.040" rpy="1.57 0 -3.14"/>
+      <geometry><mesh filename="${mesh_pkg}/arm_c_left.stl" scale="0.001 0.001 0.001"/></geometry>
+    </collision>
     <visual>
       <origin xyz="0 -0.011 -0.014" rpy="0 3.14 0"/>
@@ -820,7 +1056,113 @@
       </geometry>
     </collision>
+    <inertial>
+      <mass value="0.063687"/>
+      <origin xyz="-0.00122772 -0.01509700 -0.03204975" rpy="0 0 0"/>
+      <inertia ixx="0.00003854" ixy="-0.00000238" ixz="0.00000067" iyy="0.00001083" iyz="0.00000147" izz="0.00003352"/>
+    </inertial>
+  </link>
+  <link name="arm_b_2_1">
+    <visual>
+      <origin xyz="0.088 0.032 0.011" rpy="0 3.14 1.57"/>
+      <geometry><mesh filename="${mesh_pkg}/arm_b.stl" scale="0.001 0.001 0.001"/></geometry>
+      <material name="silver"/>
+    </visual>
+    <collision>
+      <origin xyz="0.088 0.032 0.011" rpy="0 3.14 1.57"/>
+      <geometry><mesh filename="${mesh_pkg}/arm_b.stl" scale="0.001 0.001 0.001"/></geometry>
+    </collision>
+    <inertial>
+      <mass value="0.008137"/>
+      <origin xyz="0.03797490 0.00049744 0.00094975" rpy="0 0 0"/>
+      <inertia ixx="0.00000479" ixy="-0.00000000" ixz="-0.00000000" iyy="0.00000378" iyz="-0.00000001" izz="0.00000801"/>
+    </inertial>
+  </link>
+  <!-- arm_a_4_1 (back-left, leg 4) -->
+  <link name="arm_a_4_1">
+    <visual>
+      <origin xyz="0.026 0.012 0.01" rpy="3.14 0 -1.57"/>
+      <geometry><mesh filename="${mesh_pkg}/arm_a_right.stl" scale="0.001 0.001 0.001"/></geometry>
+      <material name="silver"/>
+    </visual>
+    <collision>
+      <origin xyz="0.026 0.012 0.01" rpy="3.14 0 -1.57"/>
+      <geometry><mesh filename="${mesh_pkg}/arm_a_right.stl" scale="0.001 0.001 0.001"/></geometry>
+    </collision>
+    <visual>
+      <origin xyz="0.018 -0.0175 -0.050" rpy="0 -1.57 0"/>
+      <geometry><mesh filename="${mesh_pkg}/servo_mg995.stl" scale="0.001 0.001 0.001"/></geometry>
+      <material name="silver"/>
+    </visual>
+    <collision>
+      <origin xyz="0.018 -0.0175 -0.050" rpy="0 -1.57 0"/>
+      <geometry><mesh filename="${mesh_pkg}/servo_mg995.stl" scale="0.001 0.001 0.001"/></geometry>
+    </collision>
+    <inertial>
+      <mass value="0.061703"/>
+      <origin xyz="-0.00051903 -0.01742240 -0.04805902" rpy="0 0 0"/>
+      <inertia ixx="0.00001630" ixy="-0.00000008" ixz="-0.00000046" iyy="0.00001265" iyz="0.00000033" izz="0.00001841"/>
+    </inertial>
+  </link>
+  <link name="arm_c_4_1">
+    <visual>
+      <origin xyz="0.01 -0.145 -0.053" rpy="1.57 0 -3.14"/>
+      <geometry><mesh filename="${mesh_pkg}/arm_c_right.stl" scale="0.001 0.001 0.001"/></geometry>
+      <material name="silver"/>
+    </visual>
+    <collision>
+      <origin xyz="0.01 -0.145 -0.053" rpy="1.57 0 -3.14"/>
+      <geometry><mesh filename="${mesh_pkg}/arm_c_right.stl" scale="0.001 0.001 0.001"/></geometry>
+    </collision>
+    <visual>
+      <origin xyz="0 -0.01 -0.045" rpy="0 0 0"/>
+      <geometry><mesh filename="${mesh_pkg}/servo_mg995.stl" scale="0.001 0.001 0.001"/></geometry>
+      <material name="silver"/>
+    </visual>
+    <collision>
+      <origin xyz="0 -0.01 -0.045" rpy="0 0 0"/>
+      <geometry><mesh filename="${mesh_pkg}/servo_mg995.stl" scale="0.001 0.001 0.001"/></geometry>
+    </collision>
+    <inertial>
+      <mass value="0.063687"/>
+      <origin xyz="-0.00152686 -0.01416578 -0.02679160" rpy="0 0 0"/>
+      <inertia ixx="0.00003866" ixy="-0.00000290" ixz="-0.00000068" iyy="0.00001100" iyz="-0.00000123" izz="0.00003408"/>
+    </inertial>
+  </link>
+  <link name="arm_b_4_1">
+    <visual>
+      <origin xyz="-0.0085 -0.032 0.011" rpy="3.14 0 1.57"/>
+      <geometry><mesh filename="${mesh_pkg}/arm_b.stl" scale="0.001 0.001 0.001"/></geometry>
+      <material name="silver"/>
+    </visual>
+    <collision>
+      <origin xyz="-0.0085 -0.032 0.011" rpy="3.14 0 1.57"/>
+      <geometry><mesh filename="${mesh_pkg}/arm_b.stl" scale="0.001 0.001 0.001"/></geometry>
+    </collision>
+    <inertial>
+      <mass value="0.008137"/>
+      <origin xyz="0.04154098 -0.00048149 0.00107965" rpy="0 0 0"/>
+      <inertia ixx="0.00000479" ixy="-0.00000000" ixz="-0.00000001" iyy="0.00000378" iyz="0.00000000" izz="0.00000801"/>
+    </inertial>
   </link>
   <!-- arm_a_3_1 (back-right, leg 3) -->
   <link name="arm_a_3_1">
+    <visual>
+      <origin xyz="0.012 0.012 0.01" rpy="3.14 0 -1.57"/>
+      <geometry><mesh filename="${mesh_pkg}/arm_a_left.stl" scale="0.001 0.001 0.001"/></geometry>
+      <material name="silver"/>
+    </visual>
+    <collision>
+      <origin xyz="0.012 0.012 0.01" rpy="3.14 0 -1.57"/>
+      <geometry><mesh filename="${mesh_pkg}/arm_a_left.stl" scale="0.001 0.001 0.001"/></geometry>
+    </collision>
+    <visual>
+      <origin xyz="-0.016 -0.0175 -0.050" rpy="0 1.57 0"/>
+      <geometry><mesh filename="${mesh_pkg}/servo_mg995.stl" scale="0.001 0.001 0.001"/></geometry>
+      <material name="silver"/>
+    </visual>
+    <collision>
+      <origin xyz="-0.016 -0.0175 -0.050" rpy="0 1.57 0"/>
+      <geometry><mesh filename="${mesh_pkg}/servo_mg995.stl" scale="0.001 0.001 0.001"/></geometry>
+    </collision>
     <inertial>
       <origin xyz="0.00261850 -0.01742175 -0.04806032" rpy="0 0 0"/>
@@ -891,4 +1233,8 @@
       <material name="silver"/>
     </visual>
+    <collision>
+      <origin xyz="0.012 -0.1455 -0.040" rpy="1.57 0 -3.14"/>
+      <geometry><mesh filename="${mesh_pkg}/arm_c_left.stl" scale="0.001 0.001 0.001"/></geometry>
+    </collision>
     <visual>
       <origin xyz="0 -0.011 -0.014" rpy="0 3.14 0"/>
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