Commit message: fix: trying to fix big_bertha_description

File: big_bertha_description/urdf/big_bertha.urdf.xacro (robot description, xacro)
@@ -17,4 +17,166 @@
   <!-- ============================== Links ============================== -->
   <link name="base_link">
+    <visual>
+      <origin xyz="0 0 0.005" rpy="3.140796 0 0"/>
+      <geometry><mesh filename="${mesh_pkg}/central_perforated_plate.stl" scale="0.001 0.001 0.001"/></geometry>
+      <material name="silver"/>
+    </visual>
+    <collision>
+      <origin xyz="0 0 0.005" rpy="3.140796 0 0"/>
+      <geometry><mesh filename="${mesh_pkg}/central_perforated_plate.stl" scale="0.001 0.001 0.001"/></geometry>
+    </collision>
+    <visual>
+      <origin xyz="0 0 0.035" rpy="3.140796 0 0"/>
+      <geometry><mesh filename="${mesh_pkg}/central_perforated_plate.stl" scale="0.001 0.001 0.001"/></geometry>
+      <material name="silver"/>
+    </visual>
+    <collision>
+      <origin xyz="0 0 0.035" rpy="3.140796 0 0"/>
+      <geometry><mesh filename="${mesh_pkg}/central_perforated_plate.stl" scale="0.001 0.001 0.001"/></geometry>
+    </collision>
+    <visual>
+      <origin xyz="0.001 -0.061 0.03" rpy="3.140796 0 0"/>
+      <geometry><mesh filename="${mesh_pkg}/body_standoffs.stl" scale="0.001 0.001 0.001"/></geometry>
+      <material name="silver"/>
+    </visual>
+    <collision>
+      <origin xyz="0.001 -0.061 0.03" rpy="3.140796 0 0"/>
+      <geometry><mesh filename="${mesh_pkg}/body_standoffs.stl" scale="0.001 0.001 0.001"/></geometry>
+    </collision>
+    <visual>
+      <origin xyz="0.069 -0.001 0.03" rpy="3.140796 0 -1.57"/>
+      <geometry><mesh filename="${mesh_pkg}/body_standoffs.stl" scale="0.001 0.001 0.001"/></geometry>
+      <material name="silver"/>
+    </visual>
+    <collision>
+      <origin xyz="0.069 -0.001 0.03" rpy="3.140796 0 -1.57"/>
+      <geometry><mesh filename="${mesh_pkg}/body_standoffs.stl" scale="0.001 0.001 0.001"/></geometry>
+    </collision>
+    <visual>
+      <origin xyz="0.127 -0.069 0.03" rpy="3.140796 0 3.14"/>
+      <geometry><mesh filename="${mesh_pkg}/body_standoffs.stl" scale="0.001 0.001 0.001"/></geometry>
+      <material name="silver"/>
+    </visual>
+    <collision>
+      <origin xyz="0.127 -0.069 0.03" rpy="3.140796 0 3.14"/>
+      <geometry><mesh filename="${mesh_pkg}/body_standoffs.stl" scale="0.001 0.001 0.001"/></geometry>
+    </collision>
+    <visual>
+      <origin xyz="0.068 -0.127 0.03" rpy="3.140796 0 1.57"/>
+      <geometry><mesh filename="${mesh_pkg}/body_standoffs.stl" scale="0.001 0.001 0.001"/></geometry>
+      <material name="silver"/>
+    </visual>
+    <collision>
+      <origin xyz="0.068 -0.127 0.03" rpy="3.140796 0 1.57"/>
+      <geometry><mesh filename="${mesh_pkg}/body_standoffs.stl" scale="0.001 0.001 0.001"/></geometry>
+    </collision>
+    <visual>
+      <origin xyz="0.0325 0.007 0" rpy="3.140796 0 -1.57"/>
+      <geometry><mesh filename="${mesh_pkg}/arm_perforated_plate_bottom.stl" scale="0.001 0.001 0.001"/></geometry>
+      <material name="silver"/>
+    </visual>
+    <collision>
+      <origin xyz="0.0325 0.007 0" rpy="3.140796 0 -1.57"/>
+      <geometry><mesh filename="${mesh_pkg}/arm_perforated_plate_bottom.stl" scale="0.001 0.001 0.001"/></geometry>
+    </collision>
+    <visual>
+      <origin xyz="0.137 -0.032 0" rpy="3.140796 0 3.14"/>
+      <geometry><mesh filename="${mesh_pkg}/arm_perforated_plate_bottom.stl" scale="0.001 0.001 0.001"/></geometry>
+      <material name="silver"/>
+    </visual>
+    <collision>
+      <origin xyz="0.137 -0.032 0" rpy="3.140796 0 3.14"/>
+      <geometry><mesh filename="${mesh_pkg}/arm_perforated_plate_bottom.stl" scale="0.001 0.001 0.001"/></geometry>
+    </collision>
+    <visual>
+      <origin xyz="-0.007 -0.098 0" rpy="3.140796 0 0"/>
+      <geometry><mesh filename="${mesh_pkg}/arm_perforated_plate_bottom.stl" scale="0.001 0.001 0.001"/></geometry>
+      <material name="silver"/>
+    </visual>
+    <collision>
+      <origin xyz="-0.007 -0.098 0" rpy="3.140796 0 0"/>
+      <geometry><mesh filename="${mesh_pkg}/arm_perforated_plate_bottom.stl" scale="0.001 0.001 0.001"/></geometry>
+    </collision>
+    <visual>
+      <origin xyz="0.097 -0.137 0" rpy="3.140796 0 1.57"/>
+      <geometry><mesh filename="${mesh_pkg}/arm_perforated_plate_bottom.stl" scale="0.001 0.001 0.001"/></geometry>
+      <material name="silver"/>
+    </visual>
+    <collision>
+      <origin xyz="0.097 -0.137 0" rpy="3.140796 0 1.57"/>
+      <geometry><mesh filename="${mesh_pkg}/arm_perforated_plate_bottom.stl" scale="0.001 0.001 0.001"/></geometry>
+    </collision>
+    <visual>
+      <origin xyz="0.155 -0.078 0.03" rpy="3.140796 0 -1.57"/>
+      <geometry><mesh filename="${mesh_pkg}/arm_perforated_plate_top.stl" scale="0.001 0.001 0.001"/></geometry>
+      <material name="silver"/>
+    </visual>
+    <collision>
+      <origin xyz="0.155 -0.078 0.03" rpy="3.140796 0 -1.57"/>
+      <geometry><mesh filename="${mesh_pkg}/arm_perforated_plate_top.stl" scale="0.001 0.001 0.001"/></geometry>
+    </collision>
+    <visual>
+      <origin xyz="0.052 -0.155 0.03" rpy="3.140796 0 -3.14"/>
+      <geometry><mesh filename="${mesh_pkg}/arm_perforated_plate_top.stl" scale="0.001 0.001 0.001"/></geometry>
+      <material name="silver"/>
+    </visual>
+    <collision>
+      <origin xyz="0.052 -0.155 0.03" rpy="3.140796 0 -3.14"/>
+      <geometry><mesh filename="${mesh_pkg}/arm_perforated_plate_top.stl" scale="0.001 0.001 0.001"/></geometry>
+    </collision>
+    <visual>
+      <origin xyz="0.078 0.025 0.03" rpy="3.140796 0 0"/>
+      <geometry><mesh filename="${mesh_pkg}/arm_perforated_plate_top.stl" scale="0.001 0.001 0.001"/></geometry>
+      <material name="silver"/>
+    </visual>
+    <collision>
+      <origin xyz="0.078 0.025 0.03" rpy="3.140796 0 0"/>
+      <geometry><mesh filename="${mesh_pkg}/arm_perforated_plate_top.stl" scale="0.001 0.001 0.001"/></geometry>
+    </collision>
+    <visual>
+      <origin xyz="-0.025 -0.052 0.03" rpy="3.140796 0 1.57"/>
+      <geometry><mesh filename="${mesh_pkg}/arm_perforated_plate_top.stl" scale="0.001 0.001 0.001"/></geometry>
+      <material name="silver"/>
+    </visual>
+    <collision>
+      <origin xyz="-0.025 -0.052 0.03" rpy="3.140796 0 1.57"/>
+      <geometry><mesh filename="${mesh_pkg}/arm_perforated_plate_top.stl" scale="0.001 0.001 0.001"/></geometry>
+    </collision>
+    <visual>
+      <origin xyz="-0.015 -0.0115 0.002" rpy="0.0007963268 0 0"/>
+      <geometry><mesh filename="${mesh_pkg}/servo_mg995.stl" scale="0.001 0.001 0.001"/></geometry>
+      <material name="silver"/>
+    </visual>
+    <collision>
+      <origin xyz="-0.015 -0.0115 0.002" rpy="0.0007963268 0 0"/>
+      <geometry><mesh filename="${mesh_pkg}/servo_mg995.stl" scale="0.001 0.001 0.001"/></geometry>
+    </collision>
+    <visual>
+      <origin xyz="0.011 -0.145 0.002" rpy="0.0007963268 0 1.57"/>
+      <geometry><mesh filename="${mesh_pkg}/servo_mg995.stl" scale="0.001 0.001 0.001"/></geometry>
+      <material name="silver"/>
+    </visual>
+    <collision>
+      <origin xyz="0.011 -0.145 0.002" rpy="0.0007963268 0 1.57"/>
+      <geometry><mesh filename="${mesh_pkg}/servo_mg995.stl" scale="0.001 0.001 0.001"/></geometry>
+    </collision>
+    <visual>
+      <origin xyz="0.145 -0.1185 0.002" rpy="0.0007963268 0 -3.14"/>
+      <geometry><mesh filename="${mesh_pkg}/servo_mg995.stl" scale="0.001 0.001 0.001"/></geometry>
+      <material name="silver"/>
+    </visual>
+    <collision>
+      <origin xyz="0.145 -0.1185 0.002" rpy="0.0007963268 0 -3.14"/>
+      <geometry><mesh filename="${mesh_pkg}/servo_mg995.stl" scale="0.001 0.001 0.001"/></geometry>
+    </collision>
+    <visual>
+      <origin xyz="0.1185 0.015 0.002" rpy="0.0007963268 0 -1.57"/>
+      <geometry><mesh filename="${mesh_pkg}/servo_mg995.stl" scale="0.001 0.001 0.001"/></geometry>
+      <material name="silver"/>
+    </visual>
+    <collision>
+      <origin xyz="0.1185 0.015 0.002" rpy="0.0007963268 0 -1.57"/>
+      <geometry><mesh filename="${mesh_pkg}/servo_mg995.stl" scale="0.001 0.001 0.001"/></geometry>
+    </collision>
     <inertial>
       <mass value="0.263885"/>
@@ -22,171 +184,9 @@
       <inertia ixx="0.00116595" ixy="-0.00000226" ixz="0.00000001" iyy="0.00116867" iyz="0.00000004" izz="0.00226074"/>
     </inertial>
-    <visual>
-      <origin xyz="0 0 0.005" rpy="3.140796 0 0"/>
-      <geometry><mesh filename="${mesh_pkg}/central_perforated_plate.stl" scale="0.001 0.001 0.001"/></geometry>
-      <material name="silver"/>
-    </visual>
-    <collision>
-      <origin xyz="0 0 0.005" rpy="3.140796 0 0"/>
-      <geometry><mesh filename="${mesh_pkg}/central_perforated_plate.stl" scale="0.001 0.001 0.001"/></geometry>
-    </collision>
-    <visual>
-      <origin xyz="0 0 0.035" rpy="3.140796 0 0"/>
-      <geometry><mesh filename="${mesh_pkg}/central_perforated_plate.stl" scale="0.001 0.001 0.001"/></geometry>
-      <material name="silver"/>
-    </visual>
-    <collision>
-      <origin xyz="0 0 0.035" rpy="3.140796 0 0"/>
-      <geometry><mesh filename="${mesh_pkg}/central_perforated_plate.stl" scale="0.001 0.001 0.001"/></geometry>
-    </collision>
-    <visual>
-      <origin xyz="0.001 -0.061 0.03" rpy="3.140796 0 0"/>
-      <geometry><mesh filename="${mesh_pkg}/body_standoffs.stl" scale="0.001 0.001 0.001"/></geometry>
-      <material name="silver"/>
-    </visual>
-    <collision>
-      <origin xyz="0.001 -0.061 0.03" rpy="3.140796 0 0"/>
-      <geometry><mesh filename="${mesh_pkg}/body_standoffs.stl" scale="0.001 0.001 0.001"/></geometry>
-    </collision>
-    <visual>
-      <origin xyz="0.069 -0.001 0.03" rpy="3.140796 0 -1.57"/>
-      <geometry><mesh filename="${mesh_pkg}/body_standoffs.stl" scale="0.001 0.001 0.001"/></geometry>
-      <material name="silver"/>
-    </visual>
-    <collision>
-      <origin xyz="0.069 -0.001 0.03" rpy="3.140796 0 -1.57"/>
-      <geometry><mesh filename="${mesh_pkg}/body_standoffs.stl" scale="0.001 0.001 0.001"/></geometry>
-    </collision>
-    <visual>
-      <origin xyz="0.127 -0.069 0.03" rpy="3.140796 0 3.14"/>
-      <geometry><mesh filename="${mesh_pkg}/body_standoffs.stl" scale="0.001 0.001 0.001"/></geometry>
-      <material name="silver"/>
-    </visual>
-    <collision>
-      <origin xyz="0.127 -0.069 0.03" rpy="3.140796 0 3.14"/>
-      <geometry><mesh filename="${mesh_pkg}/body_standoffs.stl" scale="0.001 0.001 0.001"/></geometry>
-    </collision>
-    <visual>
-      <origin xyz="0.068 -0.127 0.03" rpy="3.140796 0 1.57"/>
-      <geometry><mesh filename="${mesh_pkg}/body_standoffs.stl" scale="0.001 0.001 0.001"/></geometry>
-      <material name="silver"/>
-    </visual>
-    <collision>
-      <origin xyz="0.068 -0.127 0.03" rpy="3.140796 0 1.57"/>
-      <geometry><mesh filename="${mesh_pkg}/body_standoffs.stl" scale="0.001 0.001 0.001"/></geometry>
-    </collision>
-    <visual>
-      <origin xyz="0.0325 0.007 0" rpy="3.140796 0 -1.57"/>
-      <geometry><mesh filename="${mesh_pkg}/arm_perforated_plate_bottom.stl" scale="0.001 0.001 0.001"/></geometry>
-      <material name="silver"/>
-    </visual>
-    <collision>
-      <origin xyz="0.0325 0.007 0" rpy="3.140796 0 -1.57"/>
-      <geometry><mesh filename="${mesh_pkg}/arm_perforated_plate_bottom.stl" scale="0.001 0.001 0.001"/></geometry>
-    </collision>
-    <visual>
-      <origin xyz="0.137 -0.032 0" rpy="3.140796 0 3.14"/>
-      <geometry><mesh filename="${mesh_pkg}/arm_perforated_plate_bottom.stl" scale="0.001 0.001 0.001"/></geometry>
-      <material name="silver"/>
-    </visual>
-    <collision>
-      <origin xyz="0.137 -0.032 0" rpy="3.140796 0 3.14"/>
-      <geometry><mesh filename="${mesh_pkg}/arm_perforated_plate_bottom.stl" scale="0.001 0.001 0.001"/></geometry>
-    </collision>
-    <visual>
-      <origin xyz="-0.007 -0.098 0" rpy="3.140796 0 0"/>
-      <geometry><mesh filename="${mesh_pkg}/arm_perforated_plate_bottom.stl" scale="0.001 0.001 0.001"/></geometry>
-      <material name="silver"/>
-    </visual>
-    <collision>
-      <origin xyz="-0.007 -0.098 0" rpy="3.140796 0 0"/>
-      <geometry><mesh filename="${mesh_pkg}/arm_perforated_plate_bottom.stl" scale="0.001 0.001 0.001"/></geometry>
-    </collision>
-    <visual>
-      <origin xyz="0.097 -0.137 0" rpy="3.140796 0 1.57"/>
-      <geometry><mesh filename="${mesh_pkg}/arm_perforated_plate_bottom.stl" scale="0.001 0.001 0.001"/></geometry>
-      <material name="silver"/>
-    </visual>
-    <collision>
-      <origin xyz="0.097 -0.137 0" rpy="3.140796 0 1.57"/>
-      <geometry><mesh filename="${mesh_pkg}/arm_perforated_plate_bottom.stl" scale="0.001 0.001 0.001"/></geometry>
-    </collision>
-    <visual>
-      <origin xyz="0.155 -0.078 0.03" rpy="3.140796 0 -1.57"/>
-      <geometry><mesh filename="${mesh_pkg}/arm_perforated_plate_top.stl" scale="0.001 0.001 0.001"/></geometry>
-      <material name="silver"/>
-    </visual>
-    <collision>
-      <origin xyz="0.155 -0.078 0.03" rpy="3.140796 0 -1.57"/>
-      <geometry><mesh filename="${mesh_pkg}/arm_perforated_plate_top.stl" scale="0.001 0.001 0.001"/></geometry>
-    </collision>
-    <visual>
-      <origin xyz="0.052 -0.155 0.03" rpy="3.140796 0 -3.14"/>
-      <geometry><mesh filename="${mesh_pkg}/arm_perforated_plate_top.stl" scale="0.001 0.001 0.001"/></geometry>
-      <material name="silver"/>
-    </visual>
-    <collision>
-      <origin xyz="0.052 -0.155 0.03" rpy="3.140796 0 -3.14"/>
-      <geometry><mesh filename="${mesh_pkg}/arm_perforated_plate_top.stl" scale="0.001 0.001 0.001"/></geometry>
-    </collision>
-    <visual>
-      <origin xyz="0.078 0.025 0.03" rpy="3.140796 0 0"/>
-      <geometry><mesh filename="${mesh_pkg}/arm_perforated_plate_top.stl" scale="0.001 0.001 0.001"/></geometry>
-      <material name="silver"/>
-    </visual>
-    <collision>
-      <origin xyz="0.078 0.025 0.03" rpy="3.140796 0 0"/>
-      <geometry><mesh filename="${mesh_pkg}/arm_perforated_plate_top.stl" scale="0.001 0.001 0.001"/></geometry>
-    </collision>
-    <visual>
-      <origin xyz="-0.025 -0.052 0.03" rpy="3.140796 0 1.57"/>
-      <geometry><mesh filename="${mesh_pkg}/arm_perforated_plate_top.stl" scale="0.001 0.001 0.001"/></geometry>
-      <material name="silver"/>
-    </visual>
-    <collision>
-      <origin xyz="-0.025 -0.052 0.03" rpy="3.140796 0 1.57"/>
-      <geometry><mesh filename="${mesh_pkg}/arm_perforated_plate_top.stl" scale="0.001 0.001 0.001"/></geometry>
-    </collision>
-    <visual>
-      <origin xyz="-0.015 -0.0115 0.002" rpy="0.0007963268 0 0"/>
-      <geometry><mesh filename="${mesh_pkg}/servo_mg995.stl" scale="0.001 0.001 0.001"/></geometry>
-      <material name="silver"/>
-    </visual>
-    <collision>
-      <origin xyz="-0.015 -0.0115 0.002" rpy="0.0007963268 0 0"/>
-      <geometry><mesh filename="${mesh_pkg}/servo_mg995.stl" scale="0.001 0.001 0.001"/></geometry>
-    </collision>
-    <visual>
-      <origin xyz="0.011 -0.145 0.002" rpy="0.0007963268 0 1.57"/>
-      <geometry><mesh filename="${mesh_pkg}/servo_mg995.stl" scale="0.001 0.001 0.001"/></geometry>
-      <material name="silver"/>
-    </visual>
-    <collision>
-      <origin xyz="0.011 -0.145 0.002" rpy="0.0007963268 0 1.57"/>
-      <geometry><mesh filename="${mesh_pkg}/servo_mg995.stl" scale="0.001 0.001 0.001"/></geometry>
-    </collision>
-    <visual>
-      <origin xyz="0.145 -0.1185 0.002" rpy="0.0007963268 0 -3.14"/>
-      <geometry><mesh filename="${mesh_pkg}/servo_mg995.stl" scale="0.001 0.001 0.001"/></geometry>
-      <material name="silver"/>
-    </visual>
-    <collision>
-      <origin xyz="0.145 -0.1185 0.002" rpy="0.0007963268 0 -3.14"/>
-      <geometry><mesh filename="${mesh_pkg}/servo_mg995.stl" scale="0.001 0.001 0.001"/></geometry>
-    </collision>
-    <visual>
-      <origin xyz="0.1185 0.015 0.002" rpy="0.0007963268 0 -1.57"/>
-      <geometry><mesh filename="${mesh_pkg}/servo_mg995.stl" scale="0.001 0.001 0.001"/></geometry>
-      <material name="silver"/>
-    </visual>
-    <collision>
-      <origin xyz="0.1185 0.015 0.002" rpy="0.0007963268 0 -1.57"/>
-      <geometry><mesh filename="${mesh_pkg}/servo_mg995.stl" scale="0.001 0.001 0.001"/></geometry>
-    </collision>
   </link>
   <link name="imu_link">
     <inertial>
+      <mass value="0.001"/>
       <origin xyz="0 0 0" rpy="0 0 0"/>
-      <mass value="0.001"/>
       <inertia ixx="1e-06" iyy="1e-06" izz="1e-06" ixy="0" ixz="0" iyz="0"/>
     </inertial>
@@ -198,4 +198,13 @@
   </link>
   <link name="battery_link">
+    <visual>
+      <origin xyz="0 0 0.0105" rpy="0 0 0"/>
+      <geometry><box size="0.107 0.035 0.025"/></geometry>
+      <material name="silver"/>
+    </visual>
+    <collision>
+      <origin xyz="0 0 0.0105" rpy="0 0 0"/>
+      <geometry><box size="0.107 0.035 0.025"/></geometry>
+    </collision>
     <inertial>
       <mass value="0.180000"/>
@@ -203,15 +212,15 @@
       <inertia ixx="0.00002775" ixy="0.00000000" ixz="0.00000000" iyy="0.00018111" iyz="0.00000000" izz="0.00019011"/>
     </inertial>
-    <visual>
-      <origin xyz="0 0 0.0105" rpy="0 0 0"/>
-      <geometry><box size="0.107 0.035 0.025"/></geometry>
-      <material name="silver"/>
-    </visual>
-    <collision>
-      <origin xyz="0 0 0.0105" rpy="0 0 0"/>
-      <geometry><box size="0.107 0.035 0.025"/></geometry>
-    </collision>
   </link>
   <link name="circuit_box_base_link">
+    <visual>
+      <origin xyz="0 0 0" rpy="0 0 1.57"/>
+      <geometry><box size="0.102 0.1333 0.001"/></geometry>
+      <material name="silver"/>
+    </visual>
+    <collision>
+      <origin xyz="0 0 0" rpy="0 0 1.57"/>
+      <geometry><box size="0.102 0.1333 0.001"/></geometry>
+    </collision>
     <inertial>
       <mass value="0.016044"/>
@@ -219,15 +228,128 @@
       <inertia ixx="0.00001391" ixy="0.00000001" ixz="0.00000000" iyy="0.00002376" iyz="0.00000000" izz="0.00003767"/>
     </inertial>
-    <visual>
-      <origin xyz="0 0 0" rpy="0 0 1.57"/>
+  </link>
+  <link name="circuit_box_link">
+    <visual>
+      <origin xyz="-0.15 -0.435 -0.01" rpy="0 0 4.71"/>
+      <geometry><mesh filename="${mesh_pkg}/uno_q_simplified.stl" scale="0.001 0.001 0.001"/></geometry>
+    </visual>
+    <collision>
+      <origin xyz="-0.15 -0.435 -0.01" rpy="0 0 4.71"/>
+      <geometry><mesh filename="${mesh_pkg}/uno_q_simplified.stl" scale="0.001 0.001 0.001"/></geometry>
+    </collision>
+    <visual>
+      <origin xyz="0.045 0 0.005" rpy="0 0 -1.57"/>
+      <geometry><mesh filename="${mesh_pkg}/buck_converter_step_down.stl" scale="0.001 0.001 0.001"/></geometry>
+    </visual>
+    <collision>
+      <origin xyz="0.045 0 0.005" rpy="0 0 -1.57"/>
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
Commit message: fix: imu orientation fix

File: big_bertha_description/urdf/big_bertha.urdf.xacro (robot description, xacro)
@@ -754,5 +754,5 @@
   </joint>
   <joint name="imu_joint" type="fixed">
-    <origin xyz="0.063460 -0.064057 0.072712" rpy="0 0 0"/>
+    <origin xyz="0.063460 -0.064057 0.072712" rpy="3.14159265 0 3.14159265"/>
     <parent link="base_link"/>
     <child link="imu_link"/>

Commit message: Revert "fix: imu orientation fix"
This reverts commit ecccf5eb38d4a1fb50e1648c1a1c6e3c7de57932.

File: big_bertha_description/urdf/big_bertha.urdf.xacro (robot description, xacro)
@@ -754,5 +754,5 @@
   </joint>
   <joint name="imu_joint" type="fixed">
-    <origin xyz="0.063460 -0.064057 0.072712" rpy="3.14159265 0 3.14159265"/>
+    <origin xyz="0.063460 -0.064057 0.072712" rpy="0 0 0"/>
     <parent link="base_link"/>
     <child link="imu_link"/>
