Commit message: fix: refactor inertia params to individual attributes for XML well-formedness
Replace combined inertia string params (e.g. arm_a_inertial_inertia='ixx=...') with individual attribute params (arm_a_ixx, arm_a_ixy, etc.) in leg xacro macro. This fixes the XML parsing error 'not well-formed (invalid token)' when xacro encounters ${...} in raw attribute position.

File: big_bertha_description/urdf/big_bertha.urdf.xacro (robot description, xacro)
@@ -15,4 +15,5 @@
   </material>
   <xacro:property name="mesh_pkg" value="package://big_bertha_description/meshes"/>
+  <xacro:include filename="$(find big_bertha_description)/urdf/leg_macros.xacro"/>
   <!-- ============================== Links ============================== -->
   <link name="base_link">
@@ -374,362 +375,69 @@
     </inertial>
   </link>
-  <!-- ======================== Leg links ============================== -->
-  <!-- arm_a_1_1 (front-left, leg 1) -->
-  <link name="arm_a_1_1">
-    <visual>
-      <origin xyz="0.025 0.012 0.008" rpy="3.14 0 -1.57"/>
-      <geometry><mesh filename="${mesh_pkg}/arm_a_right.stl" scale="0.001 0.001 0.001"/></geometry>
-      <material name="silver"/>
-    </visual>
-    <collision>
-      <origin xyz="0.025 0.012 0.008" rpy="3.14 0 -1.57"/>
-      <geometry><mesh filename="${mesh_pkg}/arm_a_right.stl" scale="0.001 0.001 0.001"/></geometry>
-    </collision>
-    <visual>
-      <origin xyz="0.0177 -0.0175 -0.0525" rpy="0 -1.57 0"/>
-      <geometry><mesh filename="${mesh_pkg}/servo_mg995.stl" scale="0.001 0.001 0.001"/></geometry>
-      <material name="silver"/>
-    </visual>
-    <collision>
-      <origin xyz="0.0177 -0.0175 -0.0525" rpy="0 -1.57 0"/>
-      <geometry><mesh filename="${mesh_pkg}/servo_mg995.stl" scale="0.001 0.001 0.001"/></geometry>
-    </collision>
-    <inertial>
-      <mass value="0.061703"/>
-      <origin xyz="-0.00089507 -0.01742240 -0.05050470" rpy="0 0 0"/>
-      <inertia ixx="0.00001640" ixy="-0.00000009" ixz="-0.00000040" iyy="0.00001271" iyz="0.00000034" izz="0.00001836"/>
-    </inertial>
-  </link>
-  <link name="arm_c_1_1">
-    <visual>
-      <origin xyz="0.01 -0.145 -0.053" rpy="1.57 0 -3.14"/>
-      <geometry><mesh filename="${mesh_pkg}/arm_c_right.stl" scale="0.001 0.001 0.001"/></geometry>
-      <material name="silver"/>
-    </visual>
-    <collision>
-      <origin xyz="0.01 -0.145 -0.053" rpy="1.57 0 -3.14"/>
-      <geometry><mesh filename="${mesh_pkg}/arm_c_right.stl" scale="0.001 0.001 0.001"/></geometry>
-    </collision>
-    <visual>
-      <origin xyz="0 -0.01 -0.045" rpy="0 0 0"/>
-      <geometry><mesh filename="${mesh_pkg}/servo_mg995.stl" scale="0.001 0.001 0.001"/></geometry>
-      <material name="silver"/>
-    </visual>
-    <collision>
-      <origin xyz="0 -0.01 -0.045" rpy="0 0 0"/>
-      <geometry><mesh filename="${mesh_pkg}/servo_mg995.stl" scale="0.001 0.001 0.001"/></geometry>
-    </collision>
-    <inertial>
-      <mass value="0.063687"/>
-      <origin xyz="-0.00152686 -0.01416578 -0.02679160" rpy="0 0 0"/>
-      <inertia ixx="0.00003866" ixy="-0.00000290" ixz="-0.00000068" iyy="0.00001100" iyz="-0.00000123" izz="0.00003408"/>
-    </inertial>
-  </link>
-  <link name="arm_b_1_1">
-    <visual>
-      <origin xyz="-0.0085 -0.032 0.011" rpy="3.14 0 1.57"/>
-      <geometry><mesh filename="${mesh_pkg}/arm_b.stl" scale="0.001 0.001 0.001"/></geometry>
-      <material name="silver"/>
-    </visual>
-    <collision>
-      <origin xyz="-0.0085 -0.032 0.011" rpy="3.14 0 1.57"/>
-      <geometry><mesh filename="${mesh_pkg}/arm_b.stl" scale="0.001 0.001 0.001"/></geometry>
-    </collision>
-    <inertial>
-      <mass value="0.008137"/>
-      <origin xyz="0.04154098 -0.00048149 0.00107965" rpy="0 0 0"/>
-      <inertia ixx="0.00000479" ixy="-0.00000000" ixz="-0.00000001" iyy="0.00000378" iyz="0.00000000" izz="0.00000801"/>
-    </inertial>
-  </link>
-  <!-- arm_a_2_1 (front-right, leg 2) -->
-  <link name="arm_a_2_1">
-    <visual>
-      <origin xyz="0.012 0.012 0.01" rpy="3.14 0 -1.57"/>
-      <geometry><mesh filename="${mesh_pkg}/arm_a_left.stl" scale="0.001 0.001 0.001"/></geometry>
-      <material name="silver"/>
-    </visual>
-    <collision>
-      <origin xyz="0.012 0.012 0.01" rpy="3.14 0 -1.57"/>
-      <geometry><mesh filename="${mesh_pkg}/arm_a_left.stl" scale="0.001 0.001 0.001"/></geometry>
-    </collision>
-    <visual>
-      <origin xyz="-0.016 -0.0175 -0.050" rpy="0 1.57 0"/>
-      <geometry><mesh filename="${mesh_pkg}/servo_mg995.stl" scale="0.001 0.001 0.001"/></geometry>
-      <material name="silver"/>
-    </visual>
-    <collision>
-      <origin xyz="-0.016 -0.0175 -0.050" rpy="0 1.57 0"/>
-      <geometry><mesh filename="${mesh_pkg}/servo_mg995.stl" scale="0.001 0.001 0.001"/></geometry>
-    </collision>
-    <inertial>
-      <mass value="0.061703"/>
-      <origin xyz="0.00261850 -0.01742175 -0.04806032" rpy="0 0 0"/>
-      <inertia ixx="0.00001629" ixy="0.00000010" ixz="0.00000036" iyy="0.00001259" iyz="0.00000033" izz="0.00001835"/>
-    </inertial>
-  </link>
-  <link name="arm_c_2_1">
-    <visual>
-      <origin xyz="0.012 -0.1455 -0.040" rpy="1.57 0 -3.14"/>
-      <geometry><mesh filename="${mesh_pkg}/arm_c_left.stl" scale="0.001 0.001 0.001"/></geometry>
-      <material name="silver"/>
-    </visual>
-    <collision>
-      <origin xyz="0.012 -0.1455 -0.040" rpy="1.57 0 -3.14"/>
-      <geometry><mesh filename="${mesh_pkg}/arm_c_left.stl" scale="0.001 0.001 0.001"/></geometry>
-    </collision>
-    <visual>
-      <origin xyz="0 -0.011 -0.014" rpy="0 3.14 0"/>
-      <geometry><mesh filename="${mesh_pkg}/servo_mg995.stl" scale="0.001 0.001 0.001"/></geometry>
-      <material name="silver"/>
-    </visual>
-    <collision>
-      <origin xyz="0 -0.011 -0.0135" rpy="0 3.14 0"/>
-      <geometry><mesh filename="${mesh_pkg}/servo_mg995.stl" scale="0.001 0.001 0.001"/></geometry>
-    </collision>
-    <inertial>
-      <mass value="0.063687"/>
-      <origin xyz="-0.00122772 -0.01509700 -0.03204975" rpy="0 0 0"/>
-      <inertia ixx="0.00003854" ixy="-0.00000238" ixz="0.00000067" iyy="0.00001083" iyz="0.00000147" izz="0.00003352"/>
-    </inertial>
-  </link>
-  <link name="arm_b_2_1">
-    <visual>
-      <origin xyz="0.088 0.032 0.011" rpy="0 3.14 1.57"/>
-      <geometry><mesh filename="${mesh_pkg}/arm_b.stl" scale="0.001 0.001 0.001"/></geometry>
-      <material name="silver"/>
-    </visual>
-    <collision>
-      <origin xyz="0.088 0.032 0.011" rpy="0 3.14 1.57"/>
-      <geometry><mesh filename="${mesh_pkg}/arm_b.stl" scale="0.001 0.001 0.001"/></geometry>
-    </collision>
-    <inertial>
-      <mass value="0.008137"/>
-      <origin xyz="0.03797490 0.00049744 0.00094975" rpy="0 0 0"/>
-      <inertia ixx="0.00000479" ixy="-0.00000000" ixz="-0.00000000" iyy="0.00000378" iyz="-0.00000001" izz="0.00000801"/>
-    </inertial>
-  </link>
-  <!-- arm_a_4_1 (back-left, leg 4) -->
-  <link name="arm_a_4_1">
-    <visual>
-      <origin xyz="0.026 0.012 0.01" rpy="3.14 0 -1.57"/>
-      <geometry><mesh filename="${mesh_pkg}/arm_a_right.stl" scale="0.001 0.001 0.001"/></geometry>
-      <material name="silver"/>
-    </visual>
-    <collision>
-      <origin xyz="0.026 0.012 0.01" rpy="3.14 0 -1.57"/>
-      <geometry><mesh filename="${mesh_pkg}/arm_a_right.stl" scale="0.001 0.001 0.001"/></geometry>
-    </collision>
-    <visual>
-      <origin xyz="0.018 -0.0175 -0.050" rpy="0 -1.57 0"/>
-      <geometry><mesh filename="${mesh_pkg}/servo_mg995.stl" scale="0.001 0.001 0.001"/></geometry>
-      <material name="silver"/>
-    </visual>
-    <collision>
-      <origin xyz="0.018 -0.0175 -0.050" rpy="0 -1.57 0"/>
-      <geometry><mesh filename="${mesh_pkg}/servo_mg995.stl" scale="0.001 0.001 0.001"/></geometry>
-    </collision>
-    <inertial>
-      <mass value="0.061703"/>
-      <origin xyz="-0.00051903 -0.01742240 -0.04805902" rpy="0 0 0"/>
-      <inertia ixx="0.00001630" ixy="-0.00000008" ixz="-0.00000046" iyy="0.00001265" iyz="0.00000033" izz="0.00001841"/>
-    </inertial>
-  </link>
-  <link name="arm_c_4_1">
-    <visual>
-      <origin xyz="0.01 -0.145 -0.053" rpy="1.57 0 -3.14"/>
-      <geometry><mesh filename="${mesh_pkg}/arm_c_right.stl" scale="0.001 0.001 0.001"/></geometry>
-      <material name="silver"/>
-    </visual>
-    <collision>
-      <origin xyz="0.01 -0.145 -0.053" rpy="1.57 0 -3.14"/>
-      <geometry><mesh filename="${mesh_pkg}/arm_c_right.stl" scale="0.001 0.001 0.001"/></geometry>
-    </collision>
-    <visual>
-      <origin xyz="0 -0.01 -0.045" rpy="0 0 0"/>
-      <geometry><mesh filename="${mesh_pkg}/servo_mg995.stl" scale="0.001 0.001 0.001"/></geometry>
-      <material name="silver"/>
-    </visual>
-    <collision>
-      <origin xyz="0 -0.01 -0.045" rpy="0 0 0"/>
-      <geometry><mesh filename="${mesh_pkg}/servo_mg995.stl" scale="0.001 0.001 0.001"/></geometry>
-    </collision>
-    <inertial>
-      <mass value="0.063687"/>
-      <origin xyz="-0.00152686 -0.01416578 -0.02679160" rpy="0 0 0"/>
-      <inertia ixx="0.00003866" ixy="-0.00000290" ixz="-0.00000068" iyy="0.00001100" iyz="-0.00000123" izz="0.00003408"/>
-    </inertial>
-  </link>
-  <link name="arm_b_4_1">
-    <visual>
-      <origin xyz="-0.0085 -0.032 0.011" rpy="3.14 0 1.57"/>
-      <geometry><mesh filename="${mesh_pkg}/arm_b.stl" scale="0.001 0.001 0.001"/></geometry>
-      <material name="silver"/>
-    </visual>
-    <collision>
-      <origin xyz="-0.0085 -0.032 0.011" rpy="3.14 0 1.57"/>
-      <geometry><mesh filename="${mesh_pkg}/arm_b.stl" scale="0.001 0.001 0.001"/></geometry>
-    </collision>
-    <inertial>
-      <mass value="0.008137"/>
-      <origin xyz="0.04154098 -0.00048149 0.00107965" rpy="0 0 0"/>
-      <inertia ixx="0.00000479" ixy="-0.00000000" ixz="-0.00000001" iyy="0.00000378" iyz="0.00000000" izz="0.00000801"/>
-    </inertial>
-  </link>
-  <!-- arm_a_3_1 (back-right, leg 3) -->
-  <link name="arm_a_3_1">
-    <visual>
-      <origin xyz="0.012 0.012 0.01" rpy="3.14 0 -1.57"/>
-      <geometry><mesh filename="${mesh_pkg}/arm_a_left.stl" scale="0.001 0.001 0.001"/></geometry>
-      <material name="silver"/>
-    </visual>
-    <collision>
-      <origin xyz="0.012 0.012 0.01" rpy="3.14 0 -1.57"/>
-      <geometry><mesh filename="${mesh_pkg}/arm_a_left.stl" scale="0.001 0.001 0.001"/></geometry>
-    </collision>
-    <visual>
-      <origin xyz="-0.016 -0.0175 -0.050" rpy="0 1.57 0"/>
-      <geometry><mesh filename="${mesh_pkg}/servo_mg995.stl" scale="0.001 0.001 0.001"/></geometry>
-      <material name="silver"/>
-    </visual>
-    <collision>
-      <origin xyz="-0.016 -0.0175 -0.050" rpy="0 1.57 0"/>
-      <geometry><mesh filename="${mesh_pkg}/servo_mg995.stl" scale="0.001 0.001 0.001"/></geometry>
-    </collision>
-    <inertial>
-      <mass value="0.061703"/>
-      <origin xyz="0.00261850 -0.01742175 -0.04806032" rpy="0 0 0"/>
-      <inertia ixx="0.00001629" ixy="0.00000010" ixz="0.00000036" iyy="0.00001259" iyz="0.00000033" izz="0.00001835"/>
-    </inertial>
-  </link>
-  <link name="arm_c_3_1">
-    <visual>
-      <origin xyz="0.012 -0.1455 -0.040" rpy="1.57 0 -3.14"/>
-      <geometry><mesh filename="${mesh_pkg}/arm_c_left.stl" scale="0.001 0.001 0.001"/></geometry>
-      <material name="silver"/>
-    </visual>
-    <collision>
-      <origin xyz="0.012 -0.1455 -0.040" rpy="1.57 0 -3.14"/>
-      <geometry><mesh filename="${mesh_pkg}/arm_c_left.stl" scale="0.001 0.001 0.001"/></geometry>
-    </collision>
-    <visual>
-      <origin xyz="0 -0.011 -0.014" rpy="0 3.14 0"/>
-      <geometry><mesh filename="${mesh_pkg}/servo_mg995.stl" scale="0.001 0.001 0.001"/></geometry>
-      <material name="silver"/>
-    </visual>
-    <collision>
-      <origin xyz="0 -0.011 -0.0135" rpy="0 3.14 0"/>
-      <geometry><mesh filename="${mesh_pkg}/servo_mg995.stl" scale="0.001 0.001 0.001"/></geometry>
-    </collision>
-    <inertial>
-      <mass value="0.063687"/>
-      <origin xyz="-0.00122772 -0.01509700 -0.03204975" rpy="0 0 0"/>
-      <inertia ixx="0.00003854" ixy="-0.00000238" ixz="0.00000067" iyy="0.00001083" iyz="0.00000147" izz="0.00003352"/>
-    </inertial>
-  </link>
-  <link name="arm_b_3_1">
-    <visual>
-      <origin xyz="0.088 0.032 0.011" rpy="0 3.14 1.57"/>
-      <geometry><mesh filename="${mesh_pkg}/arm_b.stl" scale="0.001 0.001 0.001"/></geometry>
-      <material name="silver"/>
-    </visual>
-    <collision>
-      <origin xyz="0.088 0.032 0.011" rpy="0 3.14 1.57"/>
-      <geometry><mesh filename="${mesh_pkg}/arm_b.stl" scale="0.001 0.001 0.001"/></geometry>
-    </collision>
-    <inertial>
-      <mass value="0.008137"/>
-      <origin xyz="0.03797490 0.00049744 0.00094975" rpy="0 0 0"/>
-      <inertia ixx="0.00000479" ixy="-0.00000000" ixz="-0.00000000" iyy="0.00000378" iyz="-0.00000001" izz="0.00000801"/>
-    </inertial>
-  </link>
-  <!-- ============================== Joints ============================= -->
-  <!-- Leg 1 (front-left): Revolute_113/114/115 -->
-  <joint name="Revolute_113" type="revolute">
-    <origin xyz="-0.015 -0.002 0.04" rpy="1.570796 0 0.785"/>
-    <parent link="base_link"/>
-    <child link="arm_a_1_1"/>
-    <axis xyz="0 1.0 0"/>
-    <limit lower="-1.57" upper="1.57" effort="1.0" velocity="6.28"/>
-  </joint>
-  <joint name="Revolute_114" type="revolute">
-    <origin xyz="0 -0.008 -0.052" rpy="0 1.57 1.57"/>
-    <parent link="arm_a_1_1"/>
-    <child link="arm_b_1_1"/>
-    <axis xyz="0 1.0 0"/>
-    <limit lower="-1.57" upper="0.96" effort="1.0" velocity="6.28"/>
-  </joint>
-  <joint name="Revolute_115" type="revolute">
-    <origin xyz="0.08 0.03 0" rpy="0 1.57 1.57"/>
-    <parent link="arm_b_1_1"/>
-    <child link="arm_c_1_1"/>
-    <axis xyz="0 0 1"/>
-    <limit lower="0" upper="2.355" effort="1.0" velocity="6.28"/>
-  </joint>
-  <!-- Leg 2 (front-right): Revolute_116/117/118 -->
-  <joint name="Revolute_116" type="revolute">
-    <origin xyz="0.0027 -0.145 0.04" rpy="1.570796 0 2.355"/>
-    <parent link="base_link"/>
-    <child link="arm_a_2_1"/>
-    <axis xyz="0 1.0 0"/>
-    <limit lower="-1.57" upper="1.57" effort="1.0" velocity="6.28"/>
-  </joint>
-  <joint name="Revolute_117" type="revolute">
-    <origin xyz="0 -0.008 -0.052" rpy="0 1.57 1.57"/>
-    <parent link="arm_a_2_1"/>
-    <child link="arm_b_2_1"/>
-    <axis xyz="0 1.0 0"/>
-    <limit lower="-1.57" upper="0.96" effort="1.0" velocity="6.28"/>
-  </joint>
-  <joint name="Revolute_118" type="revolute">
-    <origin xyz="0.08 0.03 0" rpy="0 1.57 1.57"/>
-    <parent link="arm_b_2_1"/>
-    <child link="arm_c_2_1"/>
-    <axis xyz="0 0 1"/>
-    <limit lower="0" upper="2.355" effort="1.0" velocity="6.28"/>
-  </joint>
-  <!-- Leg 4 (back-left): Revolute_110/111/112 -->
-  <joint name="Revolute_110" type="revolute">
-    <origin xyz="0.129 0.015 0.04" rpy="1.570796 0 -0.785"/>
-    <parent link="base_link"/>
-    <child link="arm_a_4_1"/>
-    <axis xyz="0 1.0 0"/>
-    <limit lower="-1.57" upper="1.57" effort="1.0" velocity="6.28"/>
-  </joint>
-  <joint name="Revolute_111" type="revolute">
-    <origin xyz="0 -0.008 -0.052" rpy="0 1.57 1.57"/>
-    <parent link="arm_a_4_1"/>
-    <child link="arm_b_4_1"/>
-    <axis xyz="0 1.0 0"/>
-    <limit lower="-1.57" upper="0.96" effort="1.0" velocity="6.28"/>
-  </joint>
-  <joint name="Revolute_112" type="revolute">
-    <origin xyz="0.08 0.03 0" rpy="0 1.57 1.57"/>
-    <parent link="arm_b_4_1"/>
-    <child link="arm_c_4_1"/>
-    <axis xyz="0 0 1"/>
-    <limit lower="0" upper="2.355" effort="1.0" velocity="6.28"/>
-  </joint>
-  <!-- Leg 3 (back-right): Revolute_119/120/121 -->
-  <joint name="Revolute_119" type="revolute">
-    <origin xyz="0.145 -0.128 0.04" rpy="1.570796 0 -2.355"/>
-    <parent link="base_link"/>
-    <child link="arm_a_3_1"/>
-    <axis xyz="0 1.0 0"/>
-    <limit lower="-1.57" upper="1.57" effort="1.0" velocity="6.28"/>
-  </joint>
-  <joint name="Revolute_120" type="revolute">
-    <origin xyz="0 -0.008 -0.052" rpy="0 1.57 1.57"/>
-    <parent link="arm_a_3_1"/>
-    <child link="arm_b_3_1"/>
-    <axis xyz="0 1.0 0"/>
-    <limit lower="-1.57" upper="0.96" effort="1.0" velocity="6.28"/>
-  </joint>
-  <joint name="Revolute_121" type="revolute">
-    <origin xyz="0.0775 0.03 0.001" rpy="0 1.57 1.57"/>
-    <parent link="arm_b_3_1"/>
-    <child link="arm_c_3_1"/>
-    <axis xyz="0 0 1"/>
-    <limit lower="0" upper="2.355" effort="1.0" velocity="6.28"/>
-  </joint>
+  <!-- ======================== Legs =================================== -->
+  <!-- Leg 1 (front-left, right-side meshes) -->
+  <xacro:leg prefix="1_1" side="right"
+    arm_a_vis_xyz="0.025 0.012 0.008" arm_a_vis_rpy="3.14 0 -1.57"
+    arm_a_servo_xyz="0.0177 -0.0175 -0.0525" arm_a_servo_rpy="0 -1.57 0"
+    arm_a_inertial_origin="-0.00089507 -0.01742240 -0.05050470"
+    arm_a_ixx="0.00001640" arm_a_ixy="-0.00000009" arm_a_ixz="-0.00000040" arm_a_iyy="0.00001271" arm_a_iyz="0.00000034" arm_a_izz="0.00001836"
+    arm_c_vis_xyz="0.01 -0.145 -0.053" arm_c_vis_rpy="1.57 0 -3.14"
+    arm_c_servo_xyz="0 -0.01 -0.045" arm_c_servo_rpy="0 0 0"
+    arm_c_inertial_origin="-0.00152686 -0.01416578 -0.02679160"
+    arm_c_ixx="0.00003866" arm_c_ixy="-0.00000290" arm_c_ixz="-0.00000068" arm_c_iyy="0.00001100" arm_c_iyz="-0.00000123" arm_c_izz="0.00003408"
+    arm_b_vis_xyz="-0.0085 -0.032 0.011" arm_b_vis_rpy="3.14 0 1.57"
+    arm_b_inertial_origin="0.04154098 -0.00048149 0.00107965"
+    arm_b_ixx="0.00000479" arm_b_ixy="-0.00000000" arm_b_ixz="-0.00000001" arm_b_iyy="0.00000378" arm_b_iyz="0.00000000" arm_b_izz="0.00000801"
+    joint_hip_name="Revolute_113" joint_hip_xyz="-0.015 -0.002 0.04" joint_hip_rpy="1.570796 0 0.785"
+    joint_knee_name="Revolute_114" joint_knee_xyz="0 -0.008 -0.052" joint_knee_rpy="0 1.57 1.57"
+    joint_ankle_name="Revolute_115" joint_ankle_xyz="0.08 0.03 0" joint_ankle_rpy="0 1.57 1.57"/>
+  <!-- Leg 2 (front-right, left-side meshes) -->
+  <xacro:leg prefix="2_1" side="left"
+    arm_a_vis_xyz="0.012 0.012 0.01" arm_a_vis_rpy="3.14 0 -1.57"
+    arm_a_servo_xyz="-0.016 -0.0175 -0.050" arm_a_servo_rpy="0 1.57 0"
+    arm_a_inertial_origin="0.00261850 -0.01742175 -0.04806032"
+    arm_a_ixx="0.00001629" arm_a_ixy="0.00000010" arm_a_ixz="0.00000036" arm_a_iyy="0.00001259" arm_a_iyz="0.00000033" arm_a_izz="0.00001835"
+    arm_c_vis_xyz="0.012 -0.1455 -0.040" arm_c_vis_rpy="1.57 0 -3.14"
+    arm_c_servo_xyz="0 -0.011 -0.014" arm_c_servo_rpy="0 3.14 0"
+    arm_c_inertial_origin="-0.00122772 -0.01509700 -0.03204975"
+    arm_c_ixx="0.00003854" arm_c_ixy="-0.00000238" arm_c_ixz="0.00000067" arm_c_iyy="0.00001083" arm_c_iyz="0.00000147" arm_c_izz="0.00003352"
+    arm_b_vis_xyz="0.088 0.032 0.011" arm_b_vis_rpy="0 3.14 1.57"
+    arm_b_inertial_origin="0.03797490 0.00049744 0.00094975"
+    arm_b_ixx="0.00000479" arm_b_ixy="-0.00000000" arm_b_ixz="-0.00000000" arm_b_iyy="0.00000378" arm_b_iyz="-0.00000001" arm_b_izz="0.00000801"
+    joint_hip_name="Revolute_116" joint_hip_xyz="0.0027 -0.145 0.04" joint_hip_rpy="1.570796 0 2.355"
+    joint_knee_name="Revolute_117" joint_knee_xyz="0 -0.008 -0.052" joint_knee_rpy="0 1.57 1.57"
+    joint_ankle_name="Revolute_118" joint_ankle_xyz="0.08 0.03 0" joint_ankle_rpy="0 1.57 1.57"/>
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
Commit message: fix: refactor inertia params to individual attributes for XML well-formedness

File: big_bertha_description/urdf/big_bertha.urdf.xacro (robot description, xacro)
@@ -34,4 +34,5 @@
   </material>
   <xacro:property name="mesh_pkg" value="package://big_bertha_description/meshes"/>
+  <xacro:include filename="$(find big_bertha_description)/urdf/leg_macros.xacro"/>
   <!-- ============================== Links ============================== -->
   <link name="base_link">
@@ -935,20 +936,20 @@
     </inertial>
   </link>
-  <link name="arm_b_1_1">
-    <visual>
-      <origin xyz="-0.0085 -0.032 0.011" rpy="3.14 0 1.57"/>
-      <geometry><mesh filename="${mesh_pkg}/arm_b.stl" scale="0.001 0.001 0.001"/></geometry>
-      <material name="silver"/>
-    </visual>
-    <collision>
-      <origin xyz="-0.0085 -0.032 0.011" rpy="3.14 0 1.57"/>
-      <geometry><mesh filename="${mesh_pkg}/arm_b.stl" scale="0.001 0.001 0.001"/></geometry>
-    </collision>
-    <inertial>
-      <mass value="0.008137"/>
-      <origin xyz="0.04154098 -0.00048149 0.00107965" rpy="0 0 0"/>
-      <inertia ixx="0.00000479" ixy="-0.00000000" ixz="-0.00000001" iyy="0.00000378" iyz="0.00000000" izz="0.00000801"/>
-    </inertial>
-  </link>
+  <!-- Leg 4 (back-left, right-side meshes) -->
+  <xacro:leg prefix="4_1" side="right"
+    arm_a_vis_xyz="0.026 0.012 0.01" arm_a_vis_rpy="3.14 0 -1.57"
+    arm_a_servo_xyz="0.018 -0.0175 -0.050" arm_a_servo_rpy="0 -1.57 0"
+    arm_a_inertial_origin="-0.00051903 -0.01742240 -0.04805902"
+    arm_a_ixx="0.00001630" arm_a_ixy="-0.00000008" arm_a_ixz="-0.00000046" arm_a_iyy="0.00001265" arm_a_iyz="0.00000033" arm_a_izz="0.00001841"
+    arm_c_vis_xyz="0.01 -0.145 -0.053" arm_c_vis_rpy="1.57 0 -3.14"
+    arm_c_servo_xyz="0 -0.01 -0.045" arm_c_servo_rpy="0 0 0"
+    arm_c_inertial_origin="-0.00152686 -0.01416578 -0.02679160"
+    arm_c_ixx="0.00003866" arm_c_ixy="-0.00000290" arm_c_ixz="-0.00000068" arm_c_iyy="0.00001100" arm_c_iyz="-0.00000123" arm_c_izz="0.00003408"
+    arm_b_vis_xyz="-0.0085 -0.032 0.011" arm_b_vis_rpy="3.14 0 1.57"
+    arm_b_inertial_origin="0.04154098 -0.00048149 0.00107965"
+    arm_b_ixx="0.00000479" arm_b_ixy="-0.00000000" arm_b_ixz="-0.00000001" arm_b_iyy="0.00000378" arm_b_iyz="0.00000000" arm_b_izz="0.00000801"
+    joint_hip_name="Revolute_110" joint_hip_xyz="0.129 0.015 0.04" joint_hip_rpy="1.570796 0 -0.785"
+    joint_knee_name="Revolute_111" joint_knee_xyz="0 -0.008 -0.052" joint_knee_rpy="0 1.57 1.57"
+    joint_ankle_name="Revolute_112" joint_ankle_xyz="0.08 0.03 0" joint_ankle_rpy="0 1.57 1.57"/>
   <!-- arm_a_2_1 (front-right, leg 2) -->
   <link name="arm_a_2_1">
