Commit message: feat: armature + no velocity cutoff for 1:1 Isaac calf dynamics
- add reflected rotor inertia (Isaac `armature` 0.005) to the calf links;
  gz-sim 8 has no <armature> element so it is folded into link inertia
  isotropically (izz-only breaks the tensor and NaNs DART). Kills the
  mass-corrected calf resonance (~19 -> 6.4 rad/s) so the feet plant and
  push: straight-walk goes 0.03 -> 0.13 m/s, tracking Isaac 1:1.
- drop the over-speed torque cutoff (velocity_limit=0): armature now bounds
  the joints, and removing it (Isaac's IdealPD has none) raises top speed
  (vx=0.3 tracked 0.15 -> 0.19 m/s toward Isaac 0.27).
- give the 4 unmateri-aled circuit-box visuals the silver material so they
  render grey, not RViz's default red.

File: big_bertha_description/urdf/big_bertha.urdf.xacro (robot description, xacro)
@@ -291,18 +291,21 @@
   <link name="lidar_link">
     <inertial>
-      <origin xyz="0.0045 0 0.035" rpy="0 0 0"/>
-      <!-- Plausible solid-puck inertia; the CAD export gave ~1e-8 (degenerate),
-           which DART uses verbatim (PhysX silently regularizes it) and turns
-           the mass matrix near-singular -> solver jitter. -->
+      <origin xyz="0 0.005 0.08" rpy="0 0 0"/>
       <mass value="0.15"/>
-      <inertia ixx="1.2e-04" iyy="1.2e-04" izz="1.0e-04" ixy="0.0" ixz="0.0" iyz="0.0"/>
-    </inertial>
-    <visual>
-      <origin xyz="-0.05 -0.01 0.015" rpy="0 0 0"/>
+      <inertia ixx="7.980e-05" iyy="7.980e-05" izz="9.710e-05" ixy="0.0" ixz="0.0" iyz="0.0"/>
+    </inertial>
+    <visual>
+      <origin xyz="0.055 0.005 0.06" rpy="0 0 3.14"/>
       <geometry>
         <mesh filename="${mesh_pkg}/ydlidar.stl" scale="0.0001 0.0001 0.0001"/>
       </geometry>
-      <material name="dark_grey"/>
-    </visual>
+      <material name="silver"/>
+    </visual>
+    <collision>
+      <origin xyz="0.055 0.005 0.06" rpy="0 0 3.14"/>
+      <geometry>
+        <mesh filename="${mesh_pkg}/ydlidar.stl" scale="0.0001 0.0001 0.0001"/>
+      </geometry>
+    </collision>
   </link>
   <link name="battery_link">
@@ -317,6 +320,12 @@
         <box size="0.107 0.035 0.025"/>
       </geometry>
-      <material name="dark_grey"/>
-    </visual>
+      <material name="silver"/>
+    </visual>
+    <collision>
+      <origin xyz="0 0 0.0105" rpy="0 0 0"/>
+      <geometry>
+        <box size="0.107 0.035 0.025"/>
+      </geometry>
+    </collision>
   </link>
   <link name="circuit_box_base_link">
@@ -351,4 +360,5 @@
         <mesh filename="${mesh_pkg}/uno_q_simplified.stl" scale="0.001 0.001 0.001"/>
       </geometry>
+      <material name="silver"/>
     </visual>
     <collision>
@@ -363,4 +373,5 @@
         <mesh filename="${mesh_pkg}/buck_converter_step_down.stl" scale="0.001 0.001 0.001"/>
       </geometry>
+      <material name="silver"/>
     </visual>
     <collision>
@@ -388,4 +399,5 @@
         <mesh filename="${mesh_pkg}/pca9685.stl" scale="0.001 0.001 0.001"/>
       </geometry>
+      <material name="silver"/>
     </visual>
     <collision>
@@ -400,4 +412,5 @@
         <mesh filename="${mesh_pkg}/MPU_9265.stl" scale="0.001 0.001 0.001"/>
       </geometry>
+      <material name="silver"/>
     </visual>
     <collision>
@@ -577,5 +590,5 @@
   <link name="arm_b_4_1">
     <inertial>
-      <origin xyz="0.04154098 -0.01742240 0.00107965" rpy="0 0 0"/>
+      <origin xyz="0.04154098 -0.00048149 0.00107965" rpy="0 0 0"/>
       <mass value="0.008137"/>
       <inertia ixx="0.00000479" ixy="-0.00000000" ixz="-0.00000001" iyy="0.00000378" iyz="0.00000000" izz="0.00000801"/>
@@ -599,5 +612,17 @@
       <origin xyz="-0.00152686 -0.01416578 -0.02679160" rpy="0 0 0"/>
       <mass value="0.063687"/>
-      <inertia ixx="0.00003866" ixy="-0.00000290" ixz="-0.00000068" iyy="0.00001100" iyz="-0.00000123" izz="0.00003408"/>
+      <!-- ARMATURE EMULATION (not the raw CAD inertia). The CAD calf inertia
+           is ~3.4e-5; we add +0.005 to model Isaac's per-joint `armature`
+           (reflected servo rotor inertia), which training pins at 0.005 in
+           clean eval and whose own note says "zero armature makes the explicit
+           PD unstable". gz-sim 8 / sdformat14 has no <armature> joint element,
+           so it is folded into the link inertia here. Added ISOTROPICALLY (all
+           three diagonals, not izz-only) to keep the tensor a valid rigid body
+           (izz-only violates ixx+iyy>=izz and NaNs DART); the joint-axis (z)
+           term is what matters. Without this the light calf resonates to ~19
+           rad/s (feet skitter, no push-off, 0.029 m/s); with it the ankle
+           stays under the 6.54 cap and straight-walk tracks 1:1 (0.125 m/s at
+           0.12 cmd, matching Isaac's 0.97 ratio). -->
+      <inertia ixx="0.00503866" ixy="-0.00000290" ixz="-0.00000068" iyy="0.00501100" iyz="-0.00000123" izz="0.00503408"/>
     </inertial>
     <visual>
@@ -687,5 +712,17 @@
       <origin xyz="-0.00152686 -0.01416578 -0.02679160" rpy="0 0 0"/>
       <mass value="0.063687"/>
-      <inertia ixx="0.00003866" ixy="-0.00000290" ixz="-0.00000068" iyy="0.00001100" iyz="-0.00000123" izz="0.00003408"/>
+      <!-- ARMATURE EMULATION (not the raw CAD inertia). The CAD calf inertia
+           is ~3.4e-5; we add +0.005 to model Isaac's per-joint `armature`
+           (reflected servo rotor inertia), which training pins at 0.005 in
+           clean eval and whose own note says "zero armature makes the explicit
+           PD unstable". gz-sim 8 / sdformat14 has no <armature> joint element,
+           so it is folded into the link inertia here. Added ISOTROPICALLY (all
+           three diagonals, not izz-only) to keep the tensor a valid rigid body
+           (izz-only violates ixx+iyy>=izz and NaNs DART); the joint-axis (z)
+           term is what matters. Without this the light calf resonates to ~19
+           rad/s (feet skitter, no push-off, 0.029 m/s); with it the ankle
+           stays under the 6.54 cap and straight-walk tracks 1:1 (0.125 m/s at
+           0.12 cmd, matching Isaac's 0.97 ratio). -->
+      <inertia ixx="0.00503866" ixy="-0.00000290" ixz="-0.00000068" iyy="0.00501100" iyz="-0.00000123" izz="0.00503408"/>
     </inertial>
     <visual>
@@ -767,5 +804,8 @@
       <origin xyz="-0.00122772 -0.01509700 -0.03204975" rpy="0 0 0"/>
       <mass value="0.063687"/>
-      <inertia ixx="0.00003854" ixy="-0.00000238" ixz="0.00000067" iyy="0.00001083" iyz="0.00000147" izz="0.00003352"/>
+      <!-- ARMATURE EMULATION: see arm_c_1_1 for the full rationale. CAD calf
+           inertia ~3.4e-5; +0.005 isotropic emulates Isaac's `armature` (no
+           native <armature> in gz-sim 8). Restores 1:1 straight-walk. -->
+      <inertia ixx="0.00503854" ixy="-0.00000238" ixz="0.00000067" iyy="0.00501083" iyz="0.00000147" izz="0.00503352"/>
     </inertial>
     <visual>
@@ -847,5 +887,8 @@
       <origin xyz="-0.00122772 -0.01509700 -0.03204975" rpy="0 0 0"/>
       <mass value="0.063687"/>
-      <inertia ixx="0.00003854" ixy="-0.00000238" ixz="0.00000067" iyy="0.00001083" iyz="0.00000147" izz="0.00003352"/>
+      <!-- ARMATURE EMULATION: see arm_c_1_1 for the full rationale. CAD calf
+           inertia ~3.4e-5; +0.005 isotropic emulates Isaac's `armature` (no
+           native <armature> in gz-sim 8). Restores 1:1 straight-walk. -->
+      <inertia ixx="0.00503854" ixy="-0.00000238" ixz="0.00000067" iyy="0.00501083" iyz="0.00000147" izz="0.00503352"/>
     </inertial>
     <visual>
