Commit message: revert: roll back to the MPU-6500 IMU, drop hardcoded device report
What:
- Revert 22fda7a (BNO055 swap) and baf06c8 (BNO address probing), restoring
  the MPU-6500 firmware, node parsing, EKF config and the external madgwick
  filter the MPU needs for orientation.
- Keep ef9a66d: MPU_9265.stl and its URDF references stay.
- upload_firmware.sh no longer prints a hardcoded I2C device list.

Why:
- The BNO055 does not respond on the bus. A full sweep of 0x03 to 0x77 on the
  M33 Wire bus, run from firmware independent of the two-address probe, finds
  exactly one device: 0x40, the PCA9685. Nothing at 0x28, 0x29, 0x4A or 0x4B.
- That rules out both the scan logic and a mis-identified part at another
  address, and it proves the bus is healthy since the PCA9685 enumerates in
  the same pass. All five module pins measure correct: VCC 3.3 V, SDA/SCL
  continuity, ADDR high, RST high, BOOT high.
- The remaining candidate is the connection to the module itself, which is
  also what the history suggests: it streamed at 98 Hz with chip_id 0xa0, went
  intermittent, then stopped.
- The policy observation includes projected_gravity_b and root_ang_vel_b, both
  IMU-derived, so no IMU means no walking at all. The MPU-6500 path is a
  known-good state at /imu ~122 Hz and unblocks hardware work now.
- upload_firmware.sh printed "I2C devices: PCA9685 @ 0x40, MPU9250 @ 0x68"
  unconditionally. It scanned nothing, so it reported the IMU present whether
  or not it was, and it cost real time during this investigation. Replaced
  with a pointer to the status service that reads the MCU's actual scan.

How:
- colcon build + colcon test on big_bertha_bringup: 174 tests, 0 failures.

File: big_bertha_description/urdf/big_bertha.urdf.xacro (robot description, xacro)
@@ -46,10 +46,10 @@
   <link name="base_link">
     <inertial>
-      <origin xyz="0.06489606 -0.06499993 0.02039469" rpy="0 0 0"/>
+      <origin xyz="0 0 0.02039469" rpy="0 0 0"/>
       <mass value="0.263885"/>
       <inertia ixx="0.00116595" ixy="-0.00000226" ixz="0.00000001" iyy="0.00116867" iyz="0.00000004" izz="0.00226074"/>
     </inertial>
     <visual>
-      <origin xyz="0 -0 0.005" rpy="3.140796 -0 0"/>
+      <origin xyz="-0.06489606 0.06499993 0.005" rpy="3.140796 -0 0"/>
       <geometry>
         <mesh filename="${mesh_pkg}/central_perforated_plate.stl" scale="0.001 0.001 0.001"/>
@@ -58,5 +58,5 @@
     </visual>
     <collision>
-      <origin xyz="0 -0 0.005" rpy="3.140796 -0 0"/>
+      <origin xyz="-0.06489606 0.06499993 0.005" rpy="3.140796 -0 0"/>
       <geometry>
         <mesh filename="${mesh_pkg}/central_perforated_plate.stl" scale="0.001 0.001 0.001"/>
@@ -64,5 +64,5 @@
     </collision>
     <visual>
-      <origin xyz="0 -0 0.035" rpy="3.140796 -0 0"/>
+      <origin xyz="-0.06489606 0.06499993 0.035" rpy="3.140796 -0 0"/>
       <geometry>
         <mesh filename="${mesh_pkg}/central_perforated_plate.stl" scale="0.001 0.001 0.001"/>
@@ -71,5 +71,5 @@
     </visual>
     <collision>
-      <origin xyz="0 -0 0.035" rpy="3.140796 -0 0"/>
+      <origin xyz="-0.06489606 0.06499993 0.035" rpy="3.140796 -0 0"/>
       <geometry>
         <mesh filename="${mesh_pkg}/central_perforated_plate.stl" scale="0.001 0.001 0.001"/>
@@ -77,57 +77,57 @@
     </collision>
     <visual>
-      <origin xyz="0.001 -0.061 0.03" rpy="3.140796 -0 0"/>
-      <geometry>
-        <mesh filename="${mesh_pkg}/body_standoffs.stl" scale="0.001 0.001 0.001"/>
-      </geometry>
-      <material name="silver"/>
-    </visual>
-    <collision>
-      <origin xyz="0.001 -0.061 0.03" rpy="3.140796 -0 0"/>
-      <geometry>
-        <mesh filename="${mesh_pkg}/body_standoffs.stl" scale="0.001 0.001 0.001"/>
-      </geometry>
-    </collision>
-    <visual>
-      <origin xyz="0.069 -0.001 0.03" rpy="3.140796 -0 -1.57"/>
-      <geometry>
-        <mesh filename="${mesh_pkg}/body_standoffs.stl" scale="0.001 0.001 0.001"/>
-      </geometry>
-      <material name="silver"/>
-    </visual>
-    <collision>
-      <origin xyz="0.069 -0.001 0.03" rpy="3.140796 -0 -1.57"/>
-      <geometry>
-        <mesh filename="${mesh_pkg}/body_standoffs.stl" scale="0.001 0.001 0.001"/>
-      </geometry>
-    </collision>
-    <visual>
-      <origin xyz="0.127 -0.069 0.03" rpy="3.140796 -0 3.14"/>
-      <geometry>
-        <mesh filename="${mesh_pkg}/body_standoffs.stl" scale="0.001 0.001 0.001"/>
-      </geometry>
-      <material name="silver"/>
-    </visual>
-    <collision>
-      <origin xyz="0.127 -0.069 0.03" rpy="3.140796 -0 3.14"/>
-      <geometry>
-        <mesh filename="${mesh_pkg}/body_standoffs.stl" scale="0.001 0.001 0.001"/>
-      </geometry>
-    </collision>
-    <visual>
-      <origin xyz="0.068 -0.127 0.03" rpy="3.140796 -0 1.57"/>
-      <geometry>
-        <mesh filename="${mesh_pkg}/body_standoffs.stl" scale="0.001 0.001 0.001"/>
-      </geometry>
-      <material name="silver"/>
-    </visual>
-    <collision>
-      <origin xyz="0.068 -0.127 0.03" rpy="3.140796 -0 1.57"/>
-      <geometry>
-        <mesh filename="${mesh_pkg}/body_standoffs.stl" scale="0.001 0.001 0.001"/>
-      </geometry>
-    </collision>
-    <visual>
-      <origin xyz="0.0325 0.007 0" rpy="3.140796 -0 -1.57"/>
+      <origin xyz="-0.06389606 0.00399993 0.03" rpy="3.140796 -0 0"/>
+      <geometry>
+        <mesh filename="${mesh_pkg}/body_standoffs.stl" scale="0.001 0.001 0.001"/>
+      </geometry>
+      <material name="silver"/>
+    </visual>
+    <collision>
+      <origin xyz="-0.06389606 0.00399993 0.03" rpy="3.140796 -0 0"/>
+      <geometry>
+        <mesh filename="${mesh_pkg}/body_standoffs.stl" scale="0.001 0.001 0.001"/>
+      </geometry>
+    </collision>
+    <visual>
+      <origin xyz="0.00410394 0.06399993 0.03" rpy="3.140796 -0 -1.57"/>
+      <geometry>
+        <mesh filename="${mesh_pkg}/body_standoffs.stl" scale="0.001 0.001 0.001"/>
+      </geometry>
+      <material name="silver"/>
+    </visual>
+    <collision>
+      <origin xyz="0.00410394 0.06399993 0.03" rpy="3.140796 -0 -1.57"/>
+      <geometry>
+        <mesh filename="${mesh_pkg}/body_standoffs.stl" scale="0.001 0.001 0.001"/>
+      </geometry>
+    </collision>
+    <visual>
+      <origin xyz="0.06210394 -0.00400007 0.03" rpy="3.140796 -0 3.14"/>
+      <geometry>
+        <mesh filename="${mesh_pkg}/body_standoffs.stl" scale="0.001 0.001 0.001"/>
+      </geometry>
+      <material name="silver"/>
+    </visual>
+    <collision>
+      <origin xyz="0.06210394 -0.00400007 0.03" rpy="3.140796 -0 3.14"/>
+      <geometry>
+        <mesh filename="${mesh_pkg}/body_standoffs.stl" scale="0.001 0.001 0.001"/>
+      </geometry>
+    </collision>
+    <visual>
+      <origin xyz="0.00310394 -0.06200007 0.03" rpy="3.140796 -0 1.57"/>
+      <geometry>
+        <mesh filename="${mesh_pkg}/body_standoffs.stl" scale="0.001 0.001 0.001"/>
+      </geometry>
+      <material name="silver"/>
+    </visual>
+    <collision>
+      <origin xyz="0.00310394 -0.06200007 0.03" rpy="3.140796 -0 1.57"/>
+      <geometry>
+        <mesh filename="${mesh_pkg}/body_standoffs.stl" scale="0.001 0.001 0.001"/>
+      </geometry>
+    </collision>
+    <visual>
+      <origin xyz="-0.03239606 0.07199993 0" rpy="3.140796 -0 -1.57"/>
       <geometry>
         <mesh filename="${mesh_pkg}/arm_perforated_plate_bottom.stl" scale="0.001 0.001 0.001"/>
@@ -136,5 +136,5 @@
     </visual>
     <collision>
-      <origin xyz="0.0325 0.007 0" rpy="3.140796 -0 -1.57"/>
+      <origin xyz="-0.03239606 0.07199993 0" rpy="3.140796 -0 -1.57"/>
       <geometry>
         <mesh filename="${mesh_pkg}/arm_perforated_plate_bottom.stl" scale="0.001 0.001 0.001"/>
@@ -142,5 +142,5 @@
     </collision>
     <visual>
-      <origin xyz="0.137 -0.032 0" rpy="3.140796 -0 3.14"/>
+      <origin xyz="0.07210394 0.03299993 0" rpy="3.140796 -0 3.14"/>
       <geometry>
         <mesh filename="${mesh_pkg}/arm_perforated_plate_bottom.stl" scale="0.001 0.001 0.001"/>
@@ -149,5 +149,5 @@
     </visual>
     <collision>
-      <origin xyz="0.137 -0.032 0" rpy="3.140796 -0 3.14"/>
+      <origin xyz="0.07210394 0.03299993 0" rpy="3.140796 -0 3.14"/>
       <geometry>
         <mesh filename="${mesh_pkg}/arm_perforated_plate_bottom.stl" scale="0.001 0.001 0.001"/>
@@ -155,5 +155,5 @@
     </collision>
     <visual>
-      <origin xyz="-0.007 -0.098 0" rpy="3.140796 -0 0"/>
+      <origin xyz="-0.07189606 -0.03300007 0" rpy="3.140796 -0 0"/>
       <geometry>
         <mesh filename="${mesh_pkg}/arm_perforated_plate_bottom.stl" scale="0.001 0.001 0.001"/>
@@ -162,5 +162,5 @@
     </visual>
     <collision>
-      <origin xyz="-0.007 -0.098 0" rpy="3.140796 -0 0"/>
+      <origin xyz="-0.07189606 -0.03300007 0" rpy="3.140796 -0 0"/>
       <geometry>
         <mesh filename="${mesh_pkg}/arm_perforated_plate_bottom.stl" scale="0.001 0.001 0.001"/>
@@ -168,5 +168,5 @@
     </collision>
     <visual>
-      <origin xyz="0.097 -0.137 0" rpy="3.140796 -0 1.57"/>
+      <origin xyz="0.03210394 -0.07200007 0" rpy="3.140796 -0 1.57"/>
       <geometry>
         <mesh filename="${mesh_pkg}/arm_perforated_plate_bottom.stl" scale="0.001 0.001 0.001"/>
@@ -175,5 +175,5 @@
     </visual>
     <collision>
-      <origin xyz="0.097 -0.137 0" rpy="3.140796 -0 1.57"/>
+      <origin xyz="0.03210394 -0.07200007 0" rpy="3.140796 -0 1.57"/>
       <geometry>
         <mesh filename="${mesh_pkg}/arm_perforated_plate_bottom.stl" scale="0.001 0.001 0.001"/>
@@ -181,5 +181,5 @@
     </collision>
     <visual>
-      <origin xyz="0.155 -0.078 0.03" rpy="3.140796 -0 -1.57"/>
+      <origin xyz="0.09010394 -0.01300007 0.03" rpy="3.140796 -0 -1.57"/>
       <geometry>
         <mesh filename="${mesh_pkg}/arm_perforated_plate_top.stl" scale="0.001 0.001 0.001"/>
@@ -188,5 +188,5 @@
     </visual>
     <collision>
-      <origin xyz="0.155 -0.078 0.03" rpy="3.140796 -0 -1.57"/>
+      <origin xyz="0.09010394 -0.01300007 0.03" rpy="3.140796 -0 -1.57"/>
       <geometry>
         <mesh filename="${mesh_pkg}/arm_perforated_plate_top.stl" scale="0.001 0.001 0.001"/>
@@ -194,5 +194,5 @@
     </collision>
     <visual>
-      <origin xyz="0.052 -0.155 0.03" rpy="3.140796 -0 -3.14"/>
+      <origin xyz="-0.01289606 -0.09000007 0.03" rpy="3.140796 -0 -3.14"/>
       <geometry>
         <mesh filename="${mesh_pkg}/arm_perforated_plate_top.stl" scale="0.001 0.001 0.001"/>
@@ -201,5 +201,5 @@
     </visual>
     <collision>
-      <origin xyz="0.052 -0.155 0.03" rpy="3.140796 -0 -3.14"/>
+      <origin xyz="-0.01289606 -0.09000007 0.03" rpy="3.140796 -0 -3.14"/>
       <geometry>
         <mesh filename="${mesh_pkg}/arm_perforated_plate_top.stl" scale="0.001 0.001 0.001"/>
@@ -207,5 +207,5 @@
     </collision>
     <visual>
-      <origin xyz="0.078 0.025 0.03" rpy="3.140796 -0 0"/>
+      <origin xyz="0.01310394 0.08999993 0.03" rpy="3.140796 -0 0"/>
       <geometry>
         <mesh filename="${mesh_pkg}/arm_perforated_plate_top.stl" scale="0.001 0.001 0.001"/>
@@ -214,5 +214,5 @@
     </visual>
     <collision>
-      <origin xyz="0.078 0.025 0.03" rpy="3.140796 -0 0"/>
+      <origin xyz="0.01310394 0.08999993 0.03" rpy="3.140796 -0 0"/>
       <geometry>
         <mesh filename="${mesh_pkg}/arm_perforated_plate_top.stl" scale="0.001 0.001 0.001"/>
@@ -220,5 +220,5 @@
     </collision>
     <visual>
-      <origin xyz="-0.025 -0.052 0.03" rpy="3.140796 -0 1.57"/>
+      <origin xyz="-0.08989606 0.01299993 0.03" rpy="3.140796 -0 1.57"/>
       <geometry>
         <mesh filename="${mesh_pkg}/arm_perforated_plate_top.stl" scale="0.001 0.001 0.001"/>
@@ -227,5 +227,5 @@
     </visual>
     <collision>
-      <origin xyz="-0.025 -0.052 0.03" rpy="3.140796 -0 1.57"/>
+      <origin xyz="-0.08989606 0.01299993 0.03" rpy="3.140796 -0 1.57"/>
       <geometry>
         <mesh filename="${mesh_pkg}/arm_perforated_plate_top.stl" scale="0.001 0.001 0.001"/>
@@ -233,51 +233,51 @@
     </collision>
     <visual>
-      <origin xyz="-0.015 -0.0115 0.002" rpy="0.0007963268 -0 0"/>
-      <geometry>
-        <mesh filename="${mesh_pkg}/servo_mg995.stl" scale="0.001 0.001 0.001"/>
-      </geometry>
-      <material name="silver"/>
-    </visual>
-    <collision>
-      <origin xyz="-0.015 -0.0115 0.002" rpy="0.0007963268 -0 0"/>
-      <geometry>
-        <mesh filename="${mesh_pkg}/servo_mg995.stl" scale="0.001 0.001 0.001"/>
-      </geometry>
-    </collision>
-    <visual>
-      <origin xyz="0.011 -0.145 0.002" rpy="0.0007963268 -0 1.57"/>
-      <geometry>
-        <mesh filename="${mesh_pkg}/servo_mg995.stl" scale="0.001 0.001 0.001"/>
-      </geometry>
-      <material name="silver"/>
-    </visual>
-    <collision>
-      <origin xyz="0.011 -0.145 0.002" rpy="0.0007963268 -0 1.57"/>
-      <geometry>
-        <mesh filename="${mesh_pkg}/servo_mg995.stl" scale="0.001 0.001 0.001"/>
-      </geometry>
-    </collision>
-    <visual>
-      <origin xyz="0.145 -0.1185 0.002" rpy="0.0007963268 -0 -3.14"/>
-      <geometry>
-        <mesh filename="${mesh_pkg}/servo_mg995.stl" scale="0.001 0.001 0.001"/>
-      </geometry>
-      <material name="silver"/>
-    </visual>
-    <collision>
-      <origin xyz="0.145 -0.1185 0.002" rpy="0.0007963268 -0 -3.14"/>
-      <geometry>
-        <mesh filename="${mesh_pkg}/servo_mg995.stl" scale="0.001 0.001 0.001"/>
-      </geometry>
-    </collision>
-    <visual>
-      <origin xyz="0.1185 0.015 0.002" rpy="0.0007963268 -0 -1.57"/>
-      <geometry>
-        <mesh filename="${mesh_pkg}/servo_mg995.stl" scale="0.001 0.001 0.001"/>
-      </geometry>
-      <material name="silver"/>
-    </visual>
-    <collision>
-      <origin xyz="0.1185 0.015 0.002" rpy="0.0007963268 -0 -1.57"/>
+      <origin xyz="-0.07989606 0.05349993 0.002" rpy="0.0007963268 -0 0"/>
+      <geometry>
+        <mesh filename="${mesh_pkg}/servo_mg995.stl" scale="0.001 0.001 0.001"/>
+      </geometry>
+      <material name="silver"/>
+    </visual>
+    <collision>
+      <origin xyz="-0.07989606 0.05349993 0.002" rpy="0.0007963268 -0 0"/>
+      <geometry>
+        <mesh filename="${mesh_pkg}/servo_mg995.stl" scale="0.001 0.001 0.001"/>
+      </geometry>
+    </collision>
+    <visual>
+      <origin xyz="-0.05389606 -0.08000007 0.002" rpy="0.0007963268 -0 1.57"/>
+      <geometry>
+        <mesh filename="${mesh_pkg}/servo_mg995.stl" scale="0.001 0.001 0.001"/>
+      </geometry>
+      <material name="silver"/>
+    </visual>
+    <collision>
+      <origin xyz="-0.05389606 -0.08000007 0.002" rpy="0.0007963268 -0 1.57"/>
+      <geometry>
+        <mesh filename="${mesh_pkg}/servo_mg995.stl" scale="0.001 0.001 0.001"/>
+      </geometry>
+    </collision>
+    <visual>
+      <origin xyz="0.08010394 -0.05350007 0.002" rpy="0.0007963268 -0 -3.14"/>
+      <geometry>
+        <mesh filename="${mesh_pkg}/servo_mg995.stl" scale="0.001 0.001 0.001"/>
+      </geometry>
+      <material name="silver"/>
+    </visual>
+    <collision>
+      <origin xyz="0.08010394 -0.05350007 0.002" rpy="0.0007963268 -0 -3.14"/>
+      <geometry>
+        <mesh filename="${mesh_pkg}/servo_mg995.stl" scale="0.001 0.001 0.001"/>
+      </geometry>
+    </collision>
+    <visual>
+      <origin xyz="0.05360394 0.07999993 0.002" rpy="0.0007963268 -0 -1.57"/>
+      <geometry>
+        <mesh filename="${mesh_pkg}/servo_mg995.stl" scale="0.001 0.001 0.001"/>
+      </geometry>
+      <material name="silver"/>
+    </visual>
+    <collision>
+      <origin xyz="0.05360394 0.07999993 0.002" rpy="0.0007963268 -0 -1.57"/>
       <geometry>
         <mesh filename="${mesh_pkg}/servo_mg995.stl" scale="0.001 0.001 0.001"/>
@@ -925,5 +925,5 @@
   <!-- Leg 4 (back-left): Revolute_110/111/112 -->
   <joint name="Revolute_110" type="revolute">
-    <origin xyz="0.129 0.015 0.04" rpy="1.570796 -0 -0.785"/>
+    <origin xyz="0.06410394 0.07999993 0.04" rpy="1.570796 -0 -0.785"/>
     <parent link="base_link"/>
     <child link="arm_a_4_1"/>
@@ -950,5 +950,5 @@
   <!-- Leg 1 (front-left): Revolute_113/114/115 -->
   <joint name="Revolute_113" type="revolute">
-    <origin xyz="-0.015 -0.002 0.04" rpy="1.570796 -0 0.785"/>
+    <origin xyz="-0.07989606 0.06299993 0.04" rpy="1.570796 -0 0.785"/>
     <parent link="base_link"/>
     <child link="arm_a_1_1"/>
@@ -975,5 +975,5 @@
   <!-- Leg 2 (front-right): Revolute_116/117/118 -->
   <joint name="Revolute_116" type="revolute">
-    <origin xyz="0.0027 -0.145 0.04" rpy="1.570796 -0 2.355"/>
+    <origin xyz="-0.06219606 -0.08000007 0.04" rpy="1.570796 -0 2.355"/>
     <parent link="base_link"/>
     <child link="arm_a_2_1"/>
@@ -1000,5 +1000,5 @@
   <!-- Leg 3 (back-right): Revolute_119/120/121 -->
   <joint name="Revolute_119" type="revolute">
-    <origin xyz="0.145 -0.128 0.04" rpy="1.570796 -0 -2.355"/>
+    <origin xyz="0.08010394 -0.06300007 0.04" rpy="1.570796 -0 -2.355"/>
     <parent link="base_link"/>
     <child link="arm_a_3_1"/>
@@ -1030,5 +1030,5 @@
        stale URDF). -->
   <joint name="battery_joint" type="fixed">
-    <origin xyz="0.0657 -0.0657 0.0585" rpy="3.140796 -0 0"/>
+    <origin xyz="0.00080394 -0.00070007 0.0585" rpy="3.140796 -0 0"/>
     <parent link="base_link"/>
     <child link="battery_link"/>
@@ -1057,5 +1057,5 @@
        cosmetic mount rotation inside circuit_box_link. -->
   <joint name="imu_joint" type="fixed">
-    <origin xyz="0.0657 -0.0657 0.0614" rpy="0 0 0"/>
+    <origin xyz="0.00080394 -0.00070007 0.0614" rpy="0 0 0"/>
     <parent link="base_link"/>
     <child link="imu_link"/>
