Commit message: fix: match the trained plant mass and joint armature
Two divergences between the Gazebo model and the robot the policy was
actually trained on, both found by diffing the deployed URDF against
assets/URDF/big_bertha/Spyder_mg995_description.urdf.

battery_link carried 0.18 kg against training's 0.5 kg, making the
deployed robot ~1.13 kg instead of ~1.45 kg. Friction is mu*N, so a 22%
lighter body has 22% less normal force and the feet skid rather than push
off. Restoring the trained mass and inertia: 0.079 -> 0.086 m/s.

Training adds armature to Revolute_.* (all twelve joints, pinned at 0.005
in clean eval) but only the calf links carried it, so the hips and knees
ran with none and the legs decoupled. That asymmetry is the visible one:
ankle amplitude on legs 1&4 against legs 2&3 measured 1.30 where Isaac is
1.00, with two feet barely leaving the ground. Adding it to the hip and
knee links takes that to 1.07.

Folding armature into link inertia is an approximation: true joint
armature does not add inertia to the rest of the chain, this does, and it
costs speed (0.086 -> 0.072 m/s at 0.002, 0.055 at training's 0.005).
0.002 is the better trade. The correct fix is joint-level armature, which
neither sdformat14 nor the dartsim plugin exposes.

Forward tracking is still ~25% of command against Isaac's ~97%. 189 tests
pass.

File: big_bertha_description/urdf/big_bertha.urdf.xacro (robot description, xacro)
@@ -312,6 +312,10 @@
     <inertial>
       <origin xyz="0 0 0.0105" rpy="0 0 0"/>
-      <mass value="0.18"/>
-      <inertia ixx="0.00002775" ixy="0.0" ixz="0.0" iyy="0.00018111" iyz="0.0" izz="0.00019011"/>
+      <!-- 0.5 kg, matching the training URDF. This carried 0.18 kg, which made
+           the deployed robot ~1.13 kg against the ~1.45 kg the policy trained
+           on. Friction is mu*N, so a 22% lighter body has 22% less normal force
+           and the feet skid instead of pushing off. -->
+      <mass value="0.5"/>
+      <inertia ixx="0.00034198" ixy="0.0" ixz="0.0" iyy="0.00058075" iyz="0.0" izz="0.00073864"/>
     </inertial>
     <visual>
@@ -559,5 +563,5 @@
       <origin xyz="-0.00051903 -0.01742240 -0.04805902" rpy="0 0 0"/>
       <mass value="0.061703"/>
-      <inertia ixx="0.00001630" ixy="-0.00000008" ixz="-0.00000046" iyy="0.00001265" iyz="0.00000033" izz="0.00001841"/>
+      <inertia ixx="0.00201630" ixy="-0.00000008" ixz="-0.00000046" iyy="0.00201265" iyz="0.00000033" izz="0.00201841"/>
     </inertial>
     <visual>
@@ -592,5 +596,5 @@
       <origin xyz="0.04154098 -0.00048149 0.00107965" rpy="0 0 0"/>
       <mass value="0.008137"/>
-      <inertia ixx="0.00000479" ixy="-0.00000000" ixz="-0.00000001" iyy="0.00000378" iyz="0.00000000" izz="0.00000801"/>
+      <inertia ixx="0.00200479" ixy="-0.00000000" ixz="-0.00000001" iyy="0.00200378" iyz="0.00000000" izz="0.00200801"/>
     </inertial>
     <visual>
@@ -655,9 +659,19 @@
     </collision>
   </link>
+  <!-- ARMATURE ON HIPS AND KNEES. Training adds armature to Revolute_.* (ALL
+       twelve joints, 0.005 pinned in clean eval); only the calf links carried
+       it here, so hips and knees ran with none and the legs decoupled. Folding
+       it into link inertia is an approximation: unlike true joint armature it
+       also adds parasitic inertia to the chain, which costs forward speed, so
+       the value here is 0.002 rather than training's 0.005. Measured: ankle
+       amplitude asymmetry (legs 1&4 vs 2&3, Isaac = 1.00) 1.30 -> 1.07 at
+       0.002 and 1.13 at 0.005, with speed 0.086 -> 0.072 and 0.055 m/s.
+       A proper fix needs joint-level armature, which sdformat14 and the
+       dartsim plugin do not expose; that wants a custom gz-sim system plugin. -->
   <link name="arm_a_1_1">
     <inertial>
       <origin xyz="-0.00089507 -0.01742240 -0.05050470" rpy="0 0 0"/>
       <mass value="0.061703"/>
-      <inertia ixx="0.00001640" ixy="-0.00000009" ixz="-0.00000040" iyy="0.00001271" iyz="0.00000034" izz="0.00001836"/>
+      <inertia ixx="0.00201640" ixy="-0.00000009" ixz="-0.00000040" iyy="0.00201271" iyz="0.00000034" izz="0.00201836"/>
     </inertial>
     <visual>
@@ -692,5 +706,5 @@
       <origin xyz="0.04154098 -0.00048149 0.00107965" rpy="0 0 0"/>
       <mass value="0.008137"/>
-      <inertia ixx="0.00000479" ixy="-0.00000000" ixz="-0.00000001" iyy="0.00000378" iyz="0.00000000" izz="0.00000801"/>
+      <inertia ixx="0.00200479" ixy="-0.00000000" ixz="-0.00000001" iyy="0.00200378" iyz="0.00000000" izz="0.00200801"/>
     </inertial>
     <visual>
@@ -751,5 +765,5 @@
       <origin xyz="0.00261850 -0.01742175 -0.04806032" rpy="0 0 0"/>
       <mass value="0.061703"/>
-      <inertia ixx="0.00001629" ixy="0.00000010" ixz="0.00000036" iyy="0.00001259" iyz="0.00000033" izz="0.00001835"/>
+      <inertia ixx="0.00201629" ixy="0.00000010" ixz="0.00000036" iyy="0.00201259" iyz="0.00000033" izz="0.00201835"/>
     </inertial>
     <visual>
@@ -784,5 +798,5 @@
       <origin xyz="0.03797490 0.00049744 0.00094975" rpy="0 0 0"/>
       <mass value="0.008137"/>
-      <inertia ixx="0.00000479" ixy="-0.00000000" ixz="-0.00000000" iyy="0.00000378" iyz="-0.00000001" izz="0.00000801"/>
+      <inertia ixx="0.00200479" ixy="-0.00000000" ixz="-0.00000000" iyy="0.00200378" iyz="-0.00000001" izz="0.00200801"/>
     </inertial>
     <visual>
@@ -834,5 +848,5 @@
       <origin xyz="0.00261850 -0.01742175 -0.04806032" rpy="0 0 0"/>
       <mass value="0.061703"/>
-      <inertia ixx="0.00001629" ixy="0.00000010" ixz="0.00000036" iyy="0.00001259" iyz="0.00000033" izz="0.00001835"/>
+      <inertia ixx="0.00201629" ixy="0.00000010" ixz="0.00000036" iyy="0.00201259" iyz="0.00000033" izz="0.00201835"/>
     </inertial>
     <visual>
@@ -867,5 +881,5 @@
       <origin xyz="0.03797490 0.00049744 0.00094975" rpy="0 0 0"/>
       <mass value="0.008137"/>
-      <inertia ixx="0.00000479" ixy="-0.00000000" ixz="-0.00000000" iyy="0.00000378" iyz="-0.00000001" izz="0.00000801"/>
+      <inertia ixx="0.00200479" ixy="-0.00000000" ixz="-0.00000000" iyy="0.00200378" iyz="-0.00000001" izz="0.00200801"/>
     </inertial>
     <visual>

Commit message: fix: raise joint damping to match Isaac ankle amplitude
Measured against an Isaac reference run of the same policy and command
(vx 0.29): Isaac holds ankle amplitude at 0.47-0.50 rad, Gazebo at the
0.02 URDF damping overshot to 0.79, so the foot arrived fast and skidded.

Swept joint damping on the straight walk:
  0.02  0.081 m/s (28%)  ankle 0.79/0.56/0.53/0.79  pitch 9.3 deg
  0.08  0.082 m/s (28%)  ankle 0.59/0.43/0.41/0.59  pitch 9.2
  0.15  0.100 m/s (35%)  ankle 0.47/0.38/0.38/0.53  pitch 8.1
  0.25  0.101 m/s (35%)  ankle 0.49/0.46/0.38/0.58  pitch 7.9

0.25 lifts forward tracking 28% -> 35% of command and drops body pitch to
7.9 deg against Isaac's 8.0 deg tilt p95. The isaac reference is a 3-min
headless play run (BB_EVAL_STEPS gates the gait dump AND loop exit).

189 tests pass.

File: big_bertha_description/urdf/big_bertha.urdf.xacro (robot description, xacro)
@@ -930,5 +930,11 @@
     <axis xyz="0 1.0 0"/>
     <limit lower="-1.57" upper="1.57" effort="1000.0" velocity="1000.0"/>
-    <dynamics damping="0.02" friction="0.0"/>
+    <!-- damping 0.25, not 0.02: measured against an Isaac reference run of
+         the same policy and command. Isaac holds ankle amplitude at
+         0.47-0.50 rad; at 0.02 Gazebo overshot to 0.79, so the foot
+         arrived fast and skidded. 0.25 brings it to 0.49/0.46/0.38/0.58,
+         lifts forward tracking 28% -> 35% of command, and drops body
+         pitch 9.3 -> 7.9 deg against Isaac's 8.0 deg tilt p95. -->
+    <dynamics damping="0.25" friction="0.0"/>
   </joint>
   <joint name="Revolute_111" type="revolute">
@@ -938,5 +944,5 @@
     <axis xyz="0 1.0 0"/>
     <limit lower="-1.57" upper="0.96" effort="1000.0" velocity="1000.0"/>
-    <dynamics damping="0.02" friction="0.0"/>
+    <dynamics damping="0.25" friction="0.0"/>
   </joint>
   <joint name="Revolute_112" type="revolute">
@@ -946,5 +952,5 @@
     <axis xyz="0 0 1"/>
     <limit lower="0" upper="2.355" effort="1000.0" velocity="1000.0"/>
-    <dynamics damping="0.02" friction="0.0"/>
+    <dynamics damping="0.25" friction="0.0"/>
   </joint>
   <!-- Leg 1 (front-left): Revolute_113/114/115 -->
@@ -955,5 +961,5 @@
     <axis xyz="0 1.0 0"/>
     <limit lower="-1.57" upper="1.57" effort="1000.0" velocity="1000.0"/>
-    <dynamics damping="0.02" friction="0.0"/>
+    <dynamics damping="0.25" friction="0.0"/>
   </joint>
   <joint name="Revolute_114" type="revolute">
@@ -963,5 +969,5 @@
     <axis xyz="0 1.0 0"/>
     <limit lower="-1.57" upper="0.96" effort="1000.0" velocity="1000.0"/>
-    <dynamics damping="0.02" friction="0.0"/>
+    <dynamics damping="0.25" friction="0.0"/>
   </joint>
   <joint name="Revolute_115" type="revolute">
@@ -971,5 +977,5 @@
     <axis xyz="0 0 1"/>
     <limit lower="0" upper="2.355" effort="1000.0" velocity="1000.0"/>
-    <dynamics damping="0.02" friction="0.0"/>
+    <dynamics damping="0.25" friction="0.0"/>
   </joint>
   <!-- Leg 2 (front-right): Revolute_116/117/118 -->
@@ -980,5 +986,5 @@
     <axis xyz="0 1.0 0"/>
     <limit lower="-1.57" upper="1.57" effort="1000.0" velocity="1000.0"/>
-    <dynamics damping="0.02" friction="0.0"/>
+    <dynamics damping="0.25" friction="0.0"/>
   </joint>
   <joint name="Revolute_117" type="revolute">
@@ -988,5 +994,5 @@
     <axis xyz="0 1.0 0"/>
     <limit lower="-1.57" upper="0.96" effort="1000.0" velocity="1000.0"/>
-    <dynamics damping="0.02" friction="0.0"/>
+    <dynamics damping="0.25" friction="0.0"/>
   </joint>
   <joint name="Revolute_118" type="revolute">
@@ -996,5 +1002,5 @@
     <axis xyz="0 0 1"/>
     <limit lower="0" upper="2.355" effort="1000.0" velocity="1000.0"/>
-    <dynamics damping="0.02" friction="0.0"/>
+    <dynamics damping="0.25" friction="0.0"/>
   </joint>
   <!-- Leg 3 (back-right): Revolute_119/120/121 -->
@@ -1005,5 +1011,5 @@
     <axis xyz="0 1.0 0"/>
     <limit lower="-1.57" upper="1.57" effort="1000.0" velocity="1000.0"/>
-    <dynamics damping="0.02" friction="0.0"/>
+    <dynamics damping="0.25" friction="0.0"/>
   </joint>
   <joint name="Revolute_120" type="revolute">
@@ -1013,5 +1019,5 @@
     <axis xyz="0 1.0 0"/>
     <limit lower="-1.57" upper="0.96" effort="1000.0" velocity="1000.0"/>
-    <dynamics damping="0.02" friction="0.0"/>
+    <dynamics damping="0.25" friction="0.0"/>
   </joint>
   <joint name="Revolute_121" type="revolute">
@@ -1021,5 +1027,5 @@
     <axis xyz="0 0 1"/>
     <limit lower="0" upper="2.355" effort="1000.0" velocity="1000.0"/>
-    <dynamics damping="0.02" friction="0.0"/>
+    <dynamics damping="0.25" friction="0.0"/>
   </joint>
   <!-- Fixed sensor / payload frames. Chain and origins copied verbatim from

Commit message: feat: urdf fix and sim bringup verified here

File: big_bertha_description/urdf/big_bertha.urdf.xacro (robot description, xacro)
@@ -174,5 +174,5 @@
     </collision>
     <visual>
-      <origin xyz="-0.03239606 0.07199993 0" rpy="3.140796 -0 -1.57"/>
+      <origin xyz="-0.07228187 0.03297877 -0.00495642" rpy="0 0.00079665 0.00079633"/>
       <geometry>
         <mesh filename="${mesh_pkg}/arm_perforated_plate_bottom.stl" scale="0.001 0.001 0.001"/>
@@ -181,5 +181,5 @@
     </visual>
     <collision>
-      <origin xyz="-0.03239606 0.07199993 0" rpy="3.140796 -0 -1.57"/>
+      <origin xyz="-0.07228187 0.03297877 -0.00495642" rpy="0 0.00079665 0.00079633"/>
       <geometry>
         <mesh filename="${mesh_pkg}/arm_perforated_plate_bottom.stl" scale="0.001 0.001 0.001"/>
@@ -187,5 +187,5 @@
     </collision>
     <visual>
-      <origin xyz="0.07210394 0.03299993 0" rpy="3.140796 -0 3.14"/>
+      <origin xyz="0.03313434 0.07242838 -0.00495642" rpy="0 0.00079665 -1.57238898"/>
       <geometry>
         <mesh filename="${mesh_pkg}/arm_perforated_plate_bottom.stl" scale="0.001 0.001 0.001"/>
@@ -194,5 +194,5 @@
     </visual>
     <collision>
-      <origin xyz="0.07210394 0.03299993 0" rpy="3.140796 -0 3.14"/>
+      <origin xyz="0.03313434 0.07242838 -0.00495642" rpy="0 0.00079665 -1.57238898"/>
       <geometry>
         <mesh filename="${mesh_pkg}/arm_perforated_plate_bottom.stl" scale="0.001 0.001 0.001"/>
@@ -200,5 +200,5 @@
     </collision>
     <visual>
-      <origin xyz="-0.07189606 -0.03300007 0" rpy="3.140796 -0 0"/>
+      <origin xyz="-0.03289610 -0.07240807 -0.00495642" rpy="0 0.00079665 1.57079633"/>
       <geometry>
         <mesh filename="${mesh_pkg}/arm_perforated_plate_bottom.stl" scale="0.001 0.001 0.001"/>
@@ -207,5 +207,5 @@
     </visual>
     <collision>
-      <origin xyz="-0.07189606 -0.03300007 0" rpy="3.140796 -0 0"/>
+      <origin xyz="-0.03289610 -0.07240807 -0.00495642" rpy="0 0.00079665 1.57079633"/>
       <geometry>
         <mesh filename="${mesh_pkg}/arm_perforated_plate_bottom.stl" scale="0.001 0.001 0.001"/>
@@ -213,5 +213,5 @@
     </collision>
     <visual>
-      <origin xyz="0.03210394 -0.07200007 0" rpy="3.140796 -0 1.57"/>
+      <origin xyz="0.07252212 -0.03302123 -0.00495642" rpy="0 0.00079665 3.14079633"/>
       <geometry>
         <mesh filename="${mesh_pkg}/arm_perforated_plate_bottom.stl" scale="0.001 0.001 0.001"/>
@@ -220,5 +220,5 @@
     </visual>
     <collision>
-      <origin xyz="0.03210394 -0.07200007 0" rpy="3.140796 -0 1.57"/>
+      <origin xyz="0.07252212 -0.03302123 -0.00495642" rpy="0 0.00079665 3.14079633"/>
       <geometry>
         <mesh filename="${mesh_pkg}/arm_perforated_plate_bottom.stl" scale="0.001 0.001 0.001"/>
@@ -226,5 +226,5 @@
     </collision>
     <visual>
-      <origin xyz="0.09010394 -0.01300007 0.03" rpy="3.140796 -0 -1.57"/>
+      <origin xyz="0.01313118 -0.09003815 0.02504051" rpy="-0 0.00079665 0.00079633"/>
       <geometry>
         <mesh filename="${mesh_pkg}/arm_perforated_plate_top.stl" scale="0.001 0.001 0.001"/>
@@ -233,5 +233,5 @@
     </visual>
     <collision>
-      <origin xyz="0.09010394 -0.01300007 0.03" rpy="3.140796 -0 -1.57"/>
+      <origin xyz="0.01313118 -0.09003815 0.02504051" rpy="-0 0.00079665 0.00079633"/>
       <geometry>
         <mesh filename="${mesh_pkg}/arm_perforated_plate_top.stl" scale="0.001 0.001 0.001"/>
@@ -239,5 +239,5 @@
     </collision>
     <visual>
-      <origin xyz="-0.01289606 -0.09000007 0.03" rpy="3.140796 -0 -3.14"/>
+      <origin xyz="-0.08996029 -0.01306255 0.02504051" rpy="-0 0.00079665 -1.56920367"/>
       <geometry>
         <mesh filename="${mesh_pkg}/arm_perforated_plate_top.stl" scale="0.001 0.001 0.001"/>
@@ -246,5 +246,5 @@
     </visual>
     <collision>
-      <origin xyz="-0.01289606 -0.09000007 0.03" rpy="3.140796 -0 -3.14"/>
+      <origin xyz="-0.08996029 -0.01306255 0.02504051" rpy="-0 0.00079665 -1.56920367"/>
       <geometry>
         <mesh filename="${mesh_pkg}/arm_perforated_plate_top.stl" scale="0.001 0.001 0.001"/>
@@ -252,5 +252,5 @@
     </collision>
     <visual>
-      <origin xyz="0.01310394 0.08999993 0.03" rpy="3.140796 -0 0"/>
+      <origin xyz="0.09010394 0.01299206 0.02504051" rpy="-0 0.00079665 1.57079633"/>
       <geometry>
         <mesh filename="${mesh_pkg}/arm_perforated_plate_top.stl" scale="0.001 0.001 0.001"/>
@@ -259,5 +259,5 @@
     </visual>
     <collision>
-      <origin xyz="0.01310394 0.08999993 0.03" rpy="3.140796 -0 0"/>
+      <origin xyz="0.09010394 0.01299206 0.02504051" rpy="-0 0.00079665 1.57079633"/>
       <geometry>
         <mesh filename="${mesh_pkg}/arm_perforated_plate_top.stl" scale="0.001 0.001 0.001"/>
@@ -265,5 +265,5 @@
     </collision>
     <visual>
-      <origin xyz="-0.08989606 0.01299993 0.03" rpy="3.140796 -0 1.57"/>
+      <origin xyz="-0.01286492 0.08996182 0.02504051" rpy="-0 0.00079665 3.14079633"/>
       <geometry>
         <mesh filename="${mesh_pkg}/arm_perforated_plate_top.stl" scale="0.001 0.001 0.001"/>
@@ -272,5 +272,5 @@
     </visual>
     <collision>
-      <origin xyz="-0.08989606 0.01299993 0.03" rpy="3.140796 -0 1.57"/>
+      <origin xyz="-0.01286492 0.08996182 0.02504051" rpy="-0 0.00079665 3.14079633"/>
       <geometry>
         <mesh filename="${mesh_pkg}/arm_perforated_plate_top.stl" scale="0.001 0.001 0.001"/>
@@ -278,51 +278,51 @@
     </collision>
     <visual>
-      <origin xyz="-0.07989606 0.05349993 0.002" rpy="0.0007963268 -0 0"/>
-      <geometry>
-        <mesh filename="${mesh_pkg}/servo_mg995.stl" scale="0.001 0.001 0.001"/>
-      </geometry>
-      <material name="silver"/>
-    </visual>
-    <collision>
-      <origin xyz="-0.07989606 0.05349993 0.002" rpy="0.0007963268 -0 0"/>
-      <geometry>
-        <mesh filename="${mesh_pkg}/servo_mg995.stl" scale="0.001 0.001 0.001"/>
-      </geometry>
-    </collision>
-    <visual>
-      <origin xyz="-0.05389606 -0.08000007 0.002" rpy="0.0007963268 -0 1.57"/>
-      <geometry>
-        <mesh filename="${mesh_pkg}/servo_mg995.stl" scale="0.001 0.001 0.001"/>
-      </geometry>
-      <material name="silver"/>
-    </visual>
-    <collision>
-      <origin xyz="-0.05389606 -0.08000007 0.002" rpy="0.0007963268 -0 1.57"/>
-      <geometry>
-        <mesh filename="${mesh_pkg}/servo_mg995.stl" scale="0.001 0.001 0.001"/>
-      </geometry>
-    </collision>
-    <visual>
-      <origin xyz="0.08010394 -0.05350007 0.002" rpy="0.0007963268 -0 -3.14"/>
-      <geometry>
-        <mesh filename="${mesh_pkg}/servo_mg995.stl" scale="0.001 0.001 0.001"/>
-      </geometry>
-      <material name="silver"/>
-    </visual>
-    <collision>
-      <origin xyz="0.08010394 -0.05350007 0.002" rpy="0.0007963268 -0 -3.14"/>
-      <geometry>
-        <mesh filename="${mesh_pkg}/servo_mg995.stl" scale="0.001 0.001 0.001"/>
-      </geometry>
-    </collision>
-    <visual>
-      <origin xyz="0.05360394 0.07999993 0.002" rpy="0.0007963268 -0 -1.57"/>
-      <geometry>
-        <mesh filename="${mesh_pkg}/servo_mg995.stl" scale="0.001 0.001 0.001"/>
-      </geometry>
-      <material name="silver"/>
-    </visual>
-    <collision>
-      <origin xyz="0.05360394 0.07999993 0.002" rpy="0.0007963268 -0 -1.57"/>
+      <origin xyz="-0.05357497 0.07986813 0.00250810" rpy="0 -0.00079633 1.57079633"/>
+      <geometry>
+        <mesh filename="${mesh_pkg}/servo_mg995.stl" scale="0.001 0.001 0.001"/>
+      </geometry>
+      <material name="silver"/>
+    </visual>
+    <collision>
+      <origin xyz="-0.05357497 0.07986813 0.00250810" rpy="0 -0.00079633 1.57079633"/>
+      <geometry>
+        <mesh filename="${mesh_pkg}/servo_mg995.stl" scale="0.001 0.001 0.001"/>
+      </geometry>
+    </collision>
+    <visual>
+      <origin xyz="-0.07976937 -0.05374829 0.00250810" rpy="0 -0.00079633 3.14079633"/>
+      <geometry>
+        <mesh filename="${mesh_pkg}/servo_mg995.stl" scale="0.001 0.001 0.001"/>
+      </geometry>
+      <material name="silver"/>
+    </visual>
+    <collision>
+      <origin xyz="-0.07976937 -0.05374829 0.00250810" rpy="0 -0.00079633 3.14079633"/>
+      <geometry>
+        <mesh filename="${mesh_pkg}/servo_mg995.stl" scale="0.001 0.001 0.001"/>
+      </geometry>
+    </collision>
+    <visual>
+      <origin xyz="0.05382510 -0.07987963 0.00250810" rpy="0 -0.00079633 -1.56920367"/>
+      <geometry>
+        <mesh filename="${mesh_pkg}/servo_mg995.stl" scale="0.001 0.001 0.001"/>
+      </geometry>
+      <material name="silver"/>
+    </visual>
+    <collision>
+      <origin xyz="0.05382510 -0.07987963 0.00250810" rpy="0 -0.00079633 -1.56920367"/>
+      <geometry>
+        <mesh filename="${mesh_pkg}/servo_mg995.stl" scale="0.001 0.001 0.001"/>
+      </geometry>
+    </collision>
+    <visual>
+      <origin xyz="0.07997783 0.05369406 0.00250810" rpy="0 -0.00079633 0.00079633"/>
+      <geometry>
+        <mesh filename="${mesh_pkg}/servo_mg995.stl" scale="0.001 0.001 0.001"/>
+      </geometry>
+      <material name="silver"/>
+    </visual>
+    <collision>
+      <origin xyz="0.07997783 0.05369406 0.00250810" rpy="0 -0.00079633 0.00079633"/>
       <geometry>
         <mesh filename="${mesh_pkg}/servo_mg995.stl" scale="0.001 0.001 0.001"/>
@@ -988,5 +988,5 @@
   <!-- Leg 4 (back-left): Revolute_110/111/112 -->
   <joint name="Revolute_110" type="revolute">
-    <origin xyz="0.06410394 0.07999993 0.04" rpy="1.570796 -0 -0.785"/>
+    <origin xyz="0.07993523 0.06369403 0.04" rpy="1.570796 -0 -0.785"/>
     <parent link="base_link"/>
     <child link="arm_a_4_1"/>
@@ -1013,5 +1013,5 @@
   <!-- Leg 1 (front-left): Revolute_113/114/115 -->
   <joint name="Revolute_113" type="revolute">
-    <origin xyz="-0.07989606 0.06299993 0.04" rpy="1.570796 -0 0.785"/>
+    <origin xyz="-0.06357497 0.07983349 0.04" rpy="1.570796 -0 0.785"/>
     <parent link="base_link"/>
     <child link="arm_a_1_1"/>
@@ -1038,5 +1038,5 @@
   <!-- Leg 2 (front-right): Revolute_116/117/118 -->
   <joint name="Revolute_116" type="revolute">
-    <origin xyz="-0.06219606 -0.08000007 0.04" rpy="1.570796 -0 2.355"/>
+    <origin xyz="-0.07974269 -0.06374831 0.04" rpy="1.570796 -0 2.355"/>
     <parent link="base_link"/>
     <child link="arm_a_2_1"/>
@@ -1063,5 +1063,5 @@
   <!-- Leg 3 (back-right): Revolute_119/120/121 -->
   <joint name="Revolute_119" type="revolute">
-    <origin xyz="0.08010394 -0.06300007 0.04" rpy="1.570796 -0 -2.355"/>
+    <origin xyz="0.06382503 -0.07982906 0.04" rpy="1.570796 -0 -2.355"/>
     <parent link="base_link"/>
     <child link="arm_a_3_1"/>
